Commit message: Scale to 150cm withers: bovine body shape, front/rear leg differentiation, carriage wheel fix
- Body: multi-box bovine silhouette (barrel + withers + brisket + rump), 107kg
- Front hips LOW (0.93m, scapula position), rear hips HIGH (1.20m, pelvis)
- Front legs: thigh 0.38m, shank 0.34m, cannon 0.18m
- Rear legs: thigh 0.50m, shank 0.45m, cannon 0.22m
- Carriage: track 205cm (was 140), wheelbase 140cm (was 205)
- Updated kinematics, force analysis, gaits, URDFs, build plan
- All integration tests pass (FK/IK, forces, gaits)

Co-authored-by: Copilot <223556219+Copilot@users.noreply.github.com>

File: robot/urdf/robotic_horse.urdf (robot description, URDF)
Before this commit: robot robotic_horse, 32 links, 31 joints
Links:
- link base_link: mass 86.0 -> 107.0; geometry collision box size=1.80 0.80 0.65; visual box size=0.40 0.65 0.10
- link fl_cannon_link: mass 1.2 -> 1.0; geometry collision cylinder length=0.18 radius=0.025; visual cylinder length=0.18 radius=0.025
- link fl_foot_link: geometry collision sphere radius=0.05; visual sphere radius=0.05
- link fl_shank_link: mass 5.0 -> 3.5; geometry collision cylinder length=0.34 radius=0.035; visual cylinder length=0.34 radius=0.035
- link fl_thigh_link: mass 6.0 -> 4.0; geometry collision cylinder length=0.38 radius=0.04; visual cylinder length=0.38 radius=0.04
- link fr_cannon_link: mass 1.2 -> 1.0; geometry collision cylinder length=0.18 radius=0.025; visual cylinder length=0.18 radius=0.025
- link fr_foot_link: geometry collision sphere radius=0.05; visual sphere radius=0.05
- link fr_shank_link: mass 5.0 -> 3.5; geometry collision cylinder length=0.34 radius=0.035; visual cylinder length=0.34 radius=0.035
- link fr_thigh_link: mass 6.0 -> 4.0; geometry collision cylinder length=0.38 radius=0.04; visual cylinder length=0.38 radius=0.04
- link front_axle_link: geometry collision box size=0.06 2.00 0.06; visual box size=0.06 2.00 0.06
- link rear_axle_link: geometry collision box size=0.06 2.00 0.06; visual box size=0.06 2.00 0.06
- link rl_cannon_link: geometry collision cylinder length=0.22 radius=0.03; visual cylinder length=0.22 radius=0.03
- link rl_foot_link: mass 0.4 -> 0.5; geometry collision sphere radius=0.06; visual sphere radius=0.06
- link rl_shank_link: mass 5.0 -> 4.0; geometry collision cylinder length=0.45 radius=0.04; visual cylinder length=0.45 radius=0.04
- link rl_thigh_link: mass 6.0 -> 5.0; geometry collision cylinder length=0.50 radius=0.045; visual cylinder length=0.50 radius=0.045
- link rr_cannon_link: geometry collision cylinder length=0.22 radius=0.03; visual cylinder length=0.22 radius=0.03
- link rr_foot_link: mass 0.4 -> 0.5; geometry collision sphere radius=0.06; visual sphere radius=0.06
- link rr_shank_link: mass 5.0 -> 4.0; geometry collision cylinder length=0.45 radius=0.04; visual cylinder length=0.45 radius=0.04
- link rr_thigh_link: mass 6.0 -> 5.0; geometry collision cylinder length=0.50 radius=0.045; visual cylinder length=0.50 radius=0.045
Joints:
- joint cart_fl_wheel_joint: origin xyz=0 0.70 0 rpy=0 0 0 -> xyz=0 1.025 0 rpy=0 0 0
- joint cart_fr_wheel_joint: origin xyz=0 -0.70 0 rpy=0 0 0 -> xyz=0 -1.025 0 rpy=0 0 0
- joint cart_rl_wheel_joint: origin xyz=0 0.70 0 rpy=0 0 0 -> xyz=0 1.025 0 rpy=0 0 0
- joint cart_rr_wheel_joint: origin xyz=0 -0.70 0 rpy=0 0 0 -> xyz=0 -1.025 0 rpy=0 0 0
- joint fl_cannon_joint: origin xyz=0 0 -0.18 rpy=0 0 0 -> xyz=0 0 -0.34 rpy=0 0 0
- joint fl_foot_joint: origin xyz=0 0 -0.10 rpy=0 0 0 -> xyz=0 0 -0.18 rpy=0 0 0
- joint fl_hip_joint: origin xyz=0.48 0.24 -0.16 rpy=0 0 0 -> xyz=0.65 0.40 -0.15 rpy=0 0 0
- joint fl_knee_joint: limit lower=-1.8 upper=2.0 effort=800 velocity=5.0 -> lower=-1.80 upper=-0.10 effort=800 velocity=5.0; origin xyz=0 0 -0.20 rpy=0 0 0 -> xyz=0 0 -0.38 rpy=0 0 0
- joint fl_thigh_joint: limit lower=-1.8 upper=1.8 effort=500 velocity=3.0 -> lower=-0.30 upper=1.20 effort=500 velocity=3.0
- joint fr_cannon_joint: origin xyz=0 0 -0.18 rpy=0 0 0 -> xyz=0 0 -0.34 rpy=0 0 0
- joint fr_foot_joint: origin xyz=0 0 -0.10 rpy=0 0 0 -> xyz=0 0 -0.18 rpy=0 0 0
- joint fr_hip_joint: origin xyz=0.48 -0.24 -0.16 rpy=0 0 0 -> xyz=0.65 -0.40 -0.15 rpy=0 0 0
- joint fr_knee_joint: limit lower=-1.8 upper=2.0 effort=800 velocity=5.0 -> lower=-1.80 upper=-0.10 effort=800 velocity=5.0; origin xyz=0 0 -0.20 rpy=0 0 0 -> xyz=0 0 -0.38 rpy=0 0 0
- joint fr_thigh_joint: limit lower=-1.8 upper=1.8 effort=500 velocity=3.0 -> lower=-0.30 upper=1.20 effort=500 velocity=3.0
- joint neck_joint: origin xyz=0.68 0 0.12 rpy=0 -0.10 0 -> xyz=0.85 0 0.30 rpy=0 -0.10 0
- joint rear_axle_joint: origin xyz=-1.15 0 -0.05 rpy=0 0 0 -> xyz=-0.90 0 -0.05 rpy=0 0 0
- joint rl_cannon_joint: origin xyz=0 0 -0.18 rpy=0 0 0 -> xyz=0 0 -0.45 rpy=0 0 0
- joint rl_foot_joint: origin xyz=0 0 -0.10 rpy=0 0 0 -> xyz=0 0 -0.22 rpy=0 0 0
- joint rl_hip_joint: origin xyz=-0.48 0.24 -0.16 rpy=0 0 0 -> xyz=-0.65 0.36 0.12 rpy=0 0 0
- joint rl_knee_joint: limit lower=-1.8 upper=2.0 effort=800 velocity=5.0 -> lower=0.10 upper=1.80 effort=800 velocity=5.0; origin xyz=0 0 -0.20 rpy=0 0 0 -> xyz=0 0 -0.50 rpy=0 0 0
- joint rl_thigh_joint: limit lower=-1.8 upper=1.8 effort=500 velocity=3.0 -> lower=-1.20 upper=0.30 effort=500 velocity=3.0
- joint rr_cannon_joint: origin xyz=0 0 -0.18 rpy=0 0 0 -> xyz=0 0 -0.45 rpy=0 0 0
- joint rr_foot_joint: origin xyz=0 0 -0.10 rpy=0 0 0 -> xyz=0 0 -0.22 rpy=0 0 0
- joint rr_hip_joint: origin xyz=-0.48 -0.24 -0.16 rpy=0 0 0 -> xyz=-0.65 -0.36 0.12 rpy=0 0 0
- joint rr_knee_joint: limit lower=-1.8 upper=2.0 effort=800 velocity=5.0 -> lower=0.10 upper=1.80 effort=800 velocity=5.0; origin xyz=0 0 -0.20 rpy=0 0 0 -> xyz=0 0 -0.50 rpy=0 0 0
- joint rr_thigh_joint: limit lower=-1.8 upper=1.8 effort=500 velocity=3.0 -> lower=-1.20 upper=0.30 effort=500 velocity=3.0
