Commit message: Scale to 150cm withers: bovine body shape, front/rear leg differentiation, carriage wheel fix
- Body: multi-box bovine silhouette (barrel + withers + brisket + rump), 107kg
- Front hips LOW (0.93m, scapula position), rear hips HIGH (1.20m, pelvis)
- Front legs: thigh 0.38m, shank 0.34m, cannon 0.18m
- Rear legs: thigh 0.50m, shank 0.45m, cannon 0.22m
- Carriage: track 205cm (was 140), wheelbase 140cm (was 205)
- Updated kinematics, force analysis, gaits, URDFs, build plan
- All integration tests pass (FK/IK, forces, gaits)

Co-authored-by: Copilot <223556219+Copilot@users.noreply.github.com>

File: ros2_ws/src/robotic_horse_description/urdf/robotic_horse.urdf.xacro (robot description, xacro)
@@ -18,9 +18,9 @@
       {fl,fr,rl,rr}_cannon_joint  — hock/fetlock (coupled)   (position ctrl)
   Physical parameters (edit here and in ros2_control.yaml):
-    Body mass  : 86 kg (QDD motors + frame + decoration)
-    Thigh      : 0.20 m,  3.5 kg
-    Shank      : 0.18 m,  3.0 kg
-    Cannon     : 0.10 m,  1.0 kg
-    Foot sphere: r=0.04 m, 0.3 kg
+    Body mass  : 107 kg (QDD motors + frame + decoration)
+    Front thigh: 0.38 m,  4.0 kg  /  Rear thigh: 0.50 m,  5.0 kg
+    Front shank: 0.34 m,  3.5 kg  /  Rear shank: 0.45 m,  4.0 kg
+    Front cannon: 0.18 m, 1.0 kg  /  Rear cannon: 0.22 m, 1.2 kg
+    Front foot: r=0.05 m, 0.4 kg  /  Rear foot: r=0.06 m, 0.5 kg
 -->
 <robot name="robotic_horse" xmlns:xacro="http://www.ros.org/wiki/xacro">
@@ -65,21 +65,39 @@
        BASE LINK
   ═══════════════════════════════════════════════════════ -->
-  <!-- Body mass ~86 kg: motors(48)+frame(24)+electronics(8)+decoration(1)+legs(5).
-       Inertia (86 kg, 1.40x0.60x0.40 m box): Ixx=3.73, Iyy=15.19, Izz=16.63 kg·m² -->
+  <!-- Body mass ~107 kg: motors(48)+frame(38)+electronics(8)+decoration(8)+legs(5).
+       Inertia (107 kg, 1.80x0.80x0.65 m box): Ixx=9.47, Iyy=32.63, Izz=34.58 kg·m² -->
   <link name="base_link">
     <inertial>
-      <mass value="86.0"/>
+      <mass value="107.0"/>
       <origin xyz="0 0 0" rpy="0 0 0"/>
-      <inertia ixx="3.73" iyy="15.19" izz="16.63" ixy="0" ixz="0" iyz="0"/>
+      <inertia ixx="9.47" iyy="32.63" izz="34.58" ixy="0" ixz="0" iyz="0"/>
     </inertial>
-    <!-- Main body panel -->
+    <!-- Main barrel (ribcage/abdomen) -->
     <visual>
       <origin xyz="0 0 0" rpy="0 0 0"/>
-      <geometry><box size="1.40 0.60 0.40"/></geometry>
+      <geometry><box size="1.80 0.80 0.55"/></geometry>
+      <material name="body_panel"/>
+    </visual>
+    <!-- Withers rise (front-top) -->
+    <visual>
+      <origin xyz="0.50 0 0.365" rpy="0 0 0"/>
+      <geometry><box size="0.55 0.70 0.18"/></geometry>
+      <material name="body_panel"/>
+    </visual>
+    <!-- Chest extension (brisket, front-bottom) -->
+    <visual>
+      <origin xyz="0.55 0 -0.325" rpy="0 0 0"/>
+      <geometry><box size="0.40 0.65 0.10"/></geometry>
+      <material name="body_panel"/>
+    </visual>
+    <!-- Rump (back-top, slight rise) -->
+    <visual>
+      <origin xyz="-0.55 0 0.315" rpy="0 0 0"/>
+      <geometry><box size="0.40 0.68 0.08"/></geometry>
       <material name="body_panel"/>
     </visual>
     <collision>
       <origin xyz="0 0 0" rpy="0 0 0"/>
-      <geometry><box size="1.40 0.68 0.40"/></geometry>
+      <geometry><box size="1.80 0.80 0.65"/></geometry>
     </collision>
   </link>
@@ -98,5 +116,5 @@
   <joint name="neck_yaw_joint" type="revolute">
     <parent link="base_link"/><child link="neck_yaw_link"/>
-    <origin xyz="0.68 0 0.12" rpy="0 0 0"/>
+    <origin xyz="0.85 0 0.30" rpy="0 0 0"/>
     <axis xyz="0 0 1"/>
     <limit lower="-0.6" upper="0.6" effort="15.0" velocity="2.0"/>
@@ -241,5 +259,5 @@
   <joint name="fl_hip_joint" type="revolute">
     <parent link="base_link"/><child link="fl_hip_link"/>
-    <origin xyz="0.48 0.24 -0.16" rpy="0 0 0"/>
+    <origin xyz="0.65 0.40 -0.15" rpy="0 0 0"/>
     <axis xyz="0 0 1"/>
     <limit lower="-0.35" upper="0.35" effort="200" velocity="2.0"/>
@@ -248,33 +266,30 @@
   <gazebo reference="fl_hip_link"><material>Gazebo/Grey</material></gazebo>
   <link name="fl_thigh_link">
-    <inertial><mass value="6.0"/><origin xyz="0 0 -0.10" rpy="0 0 0"/>
-      <inertia ixx="0.022" iyy="0.022" izz="0.005" ixy="0" ixz="0" iyz="0"/></inertial>
-    <visual><origin xyz="0 0 -0.10" rpy="0 0 0"/>
-      <geometry><box size="0.070 0.070 0.20"/></geometry><material name="orange"/></visual>
-    <!-- Ballscrew actuator tube -->
-    <visual><origin xyz="0.040 0 -0.10" rpy="0 0 0"/>
-      <geometry><cylinder radius="0.018" length="0.13"/></geometry><material name="silver"/></visual>
-    <collision><origin xyz="0 0 -0.10" rpy="0 0 0">
-      </origin><geometry><box size="0.070 0.070 0.20"/></geometry></collision>
+    <inertial><mass value="4.0"/><origin xyz="0 0 -0.19" rpy="0 0 0"/>
+      <inertia ixx="0.0496" iyy="0.0496" izz="0.0032" ixy="0" ixz="0" iyz="0"/></inertial>
+    <visual><origin xyz="0 0 -0.19" rpy="0 0 0"/>
+      <geometry><cylinder radius="0.04" length="0.38"/></geometry><material name="orange"/></visual>
+    <collision><origin xyz="0 0 -0.19" rpy="0 0 0">
+      </origin><geometry><cylinder radius="0.04" length="0.38"/></geometry></collision>
   </link>
   <joint name="fl_thigh_joint" type="revolute">
     <parent link="fl_hip_link"/><child link="fl_thigh_link"/>
     <origin xyz="0 0 -0.10" rpy="0 0 0"/><axis xyz="0 1 0"/>
-    <limit lower="-1.8" upper="1.8" effort="500" velocity="3.0"/>
+    <limit lower="-0.30" upper="1.20" effort="500" velocity="3.0"/>
     <dynamics damping="2.5" friction="0.3"/>
   </joint>
   <gazebo reference="fl_thigh_link"><material>Gazebo/Orange</material></gazebo>
   <link name="fl_shank_link">
-    <inertial><mass value="5.0"/><origin xyz="0 0 -0.09" rpy="0 0 0"/>
-      <inertia ixx="0.015" iyy="0.015" izz="0.003" ixy="0" ixz="0" iyz="0"/></inertial>
-    <visual><origin xyz="0 0 -0.09" rpy="0 0 0">
-      </origin><geometry><box size="0.050 0.050 0.18"/></geometry><material name="dark_grey"/></visual>
-    <collision><origin xyz="0 0 -0.09" rpy="0 0 0">
-      </origin><geometry><box size="0.050 0.050 0.18"/></geometry></collision>
+    <inertial><mass value="3.5"/><origin xyz="0 0 -0.17" rpy="0 0 0"/>
+      <inertia ixx="0.0348" iyy="0.0348" izz="0.0021" ixy="0" ixz="0" iyz="0"/></inertial>
+    <visual><origin xyz="0 0 -0.17" rpy="0 0 0">
+      </origin><geometry><cylinder radius="0.035" length="0.34"/></geometry><material name="dark_grey"/></visual>
+    <collision><origin xyz="0 0 -0.17" rpy="0 0 0">
+      </origin><geometry><cylinder radius="0.035" length="0.34"/></geometry></collision>
   </link>
   <joint name="fl_knee_joint" type="revolute">
     <parent link="fl_thigh_link"/><child link="fl_shank_link"/>
-    <origin xyz="0 0 -0.20" rpy="0 0 0"/><axis xyz="0 1 0"/>
-    <limit lower="-1.8" upper="2.0" effort="800" velocity="5.0"/>
+    <origin xyz="0 0 -0.38" rpy="0 0 0"/><axis xyz="0 1 0"/>
+    <limit lower="-1.80" upper="-0.10" effort="800" velocity="5.0"/>
     <dynamics damping="3.5" friction="0.3"/>
   </joint>
@@ -282,14 +297,14 @@
   <!-- Cannon bone (metatarsal/metacarpal): pantograph-kept near vertical -->
   <link name="fl_cannon_link">
-    <inertial><mass value="1.2"/><origin xyz="0 0 -0.05" rpy="0 0 0"/>
-      <inertia ixx="0.0011" iyy="0.0011" izz="0.0002" ixy="0" ixz="0" iyz="0"/></inertial>
-    <visual><origin xyz="0 0 -0.05" rpy="0 0 0"/>
-      <geometry><cylinder radius="0.018" length="0.10"/></geometry><material name="dark_grey"/></visual>
-    <collision><origin xyz="0 0 -0.05" rpy="0 0 0"/>
-      <geometry><cylinder radius="0.016" length="0.10"/></geometry></collision>
+    <inertial><mass value="1.0"/><origin xyz="0 0 -0.09" rpy="0 0 0"/>
+      <inertia ixx="0.0028" iyy="0.0028" izz="0.0003" ixy="0" ixz="0" iyz="0"/></inertial>
+    <visual><origin xyz="0 0 -0.09" rpy="0 0 0"/>
+      <geometry><cylinder radius="0.025" length="0.18"/></geometry><material name="dark_grey"/></visual>
+    <collision><origin xyz="0 0 -0.09" rpy="0 0 0"/>
+      <geometry><cylinder radius="0.025" length="0.18"/></geometry></collision>
   </link>
   <joint name="fl_cannon_joint" type="revolute">
     <parent link="fl_shank_link"/><child link="fl_cannon_link"/>
-    <origin xyz="0 0 -0.18" rpy="0 0 0"/><axis xyz="0 1 0"/>
+    <origin xyz="0 0 -0.34" rpy="0 0 0"/><axis xyz="0 1 0"/>
     <limit lower="-2.0" upper="2.0" effort="100" velocity="6.0"/>
     <dynamics damping="1.0" friction="0.1"/>
@@ -298,13 +313,13 @@
     <link name="fl_foot_link">
     <inertial><mass value="0.4"/><origin xyz="0 0 0" rpy="0 0 0"/>
-      <inertia ixx="0.00026" iyy="0.00026" izz="0.00026" ixy="0" ixz="0" iyz="0"/></inertial>
+      <inertia ixx="0.00040" iyy="0.00040" izz="0.00040" ixy="0" ixz="0" iyz="0"/></inertial>
     <visual><origin xyz="0 0 0" rpy="0 0 0"/>
-      <geometry><sphere radius="0.04"/></geometry><material name="black"/></visual>
+      <geometry><sphere radius="0.05"/></geometry><material name="black"/></visual>
     <collision><origin xyz="0 0 0" rpy="0 0 0"/>
-      <geometry><sphere radius="0.04"/></geometry></collision>
+      <geometry><sphere radius="0.05"/></geometry></collision>
   </link>
   <joint name="fl_foot_joint" type="fixed">
     <parent link="fl_cannon_link"/><child link="fl_foot_link"/>
-    <origin xyz="0 0 -0.10" rpy="0 0 0"/>
+    <origin xyz="0 0 -0.18" rpy="0 0 0"/>
   </joint>
   <gazebo reference="fl_foot_link">
@@ -324,5 +339,5 @@
   <joint name="fr_hip_joint" type="revolute">
     <parent link="base_link"/><child link="fr_hip_link"/>
-    <origin xyz="0.48 -0.24 -0.16" rpy="0 0 0"/>
+    <origin xyz="0.65 -0.40 -0.15" rpy="0 0 0"/>
     <axis xyz="0 0 1"/>
     <limit lower="-0.35" upper="0.35" effort="200" velocity="2.0"/>
@@ -331,33 +346,30 @@
   <gazebo reference="fr_hip_link"><material>Gazebo/Grey</material></gazebo>
   <link name="fr_thigh_link">
-    <inertial><mass value="6.0"/><origin xyz="0 0 -0.10" rpy="0 0 0"/>
-      <inertia ixx="0.022" iyy="0.022" izz="0.005" ixy="0" ixz="0" iyz="0"/></inertial>
-    <visual><origin xyz="0 0 -0.10" rpy="0 0 0">
-      </origin><geometry><box size="0.070 0.070 0.20"/></geometry><material name="orange"/></visual>
-    <!-- Ballscrew actuator tube -->
-    <visual><origin xyz="0.040 0 -0.10" rpy="0 0 0"/>
-      <geometry><cylinder radius="0.018" length="0.13"/></geometry><material name="silver"/></visual>
-    <collision><origin xyz="0 0 -0.10" rpy="0 0 0">
-      </origin><geometry><box size="0.070 0.070 0.20"/></geometry></collision>
+    <inertial><mass value="4.0"/><origin xyz="0 0 -0.19" rpy="0 0 0"/>
+      <inertia ixx="0.0496" iyy="0.0496" izz="0.0032" ixy="0" ixz="0" iyz="0"/></inertial>
+    <visual><origin xyz="0 0 -0.19" rpy="0 0 0"/>
+      <geometry><cylinder radius="0.04" length="0.38"/></geometry><material name="orange"/></visual>
+    <collision><origin xyz="0 0 -0.19" rpy="0 0 0">
+      </origin><geometry><cylinder radius="0.04" length="0.38"/></geometry></collision>
   </link>
   <joint name="fr_thigh_joint" type="revolute">
     <parent link="fr_hip_link"/><child link="fr_thigh_link"/>
     <origin xyz="0 0 -0.10" rpy="0 0 0"/><axis xyz="0 1 0"/>
-    <limit lower="-1.8" upper="1.8" effort="500" velocity="3.0"/>
+    <limit lower="-0.30" upper="1.20" effort="500" velocity="3.0"/>
     <dynamics damping="2.5" friction="0.3"/>
   </joint>
   <gazebo reference="fr_thigh_link"><material>Gazebo/Orange</material></gazebo>
   <link name="fr_shank_link">
-    <inertial><mass value="5.0"/><origin xyz="0 0 -0.09" rpy="0 0 0"/>
-      <inertia ixx="0.015" iyy="0.015" izz="0.003" ixy="0" ixz="0" iyz="0"/></inertial>
-    <visual><origin xyz="0 0 -0.09" rpy="0 0 0">
-      </origin><geometry><box size="0.050 0.050 0.18"/></geometry><material name="dark_grey"/></visual>
-    <collision><origin xyz="0 0 -0.09" rpy="0 0 0">
-      </origin><geometry><box size="0.050 0.050 0.18"/></geometry></collision>
+    <inertial><mass value="3.5"/><origin xyz="0 0 -0.17" rpy="0 0 0"/>
+      <inertia ixx="0.0348" iyy="0.0348" izz="0.0021" ixy="0" ixz="0" iyz="0"/></inertial>
+    <visual><origin xyz="0 0 -0.17" rpy="0 0 0">
+      </origin><geometry><cylinder radius="0.035" length="0.34"/></geometry><material name="dark_grey"/></visual>
+    <collision><origin xyz="0 0 -0.17" rpy="0 0 0">
+      </origin><geometry><cylinder radius="0.035" length="0.34"/></geometry></collision>
   </link>
   <joint name="fr_knee_joint" type="revolute">
     <parent link="fr_thigh_link"/><child link="fr_shank_link"/>
-    <origin xyz="0 0 -0.20" rpy="0 0 0"/><axis xyz="0 1 0"/>
-    <limit lower="-1.8" upper="2.0" effort="800" velocity="5.0"/>
+    <origin xyz="0 0 -0.38" rpy="0 0 0"/><axis xyz="0 1 0"/>
+    <limit lower="-1.80" upper="-0.10" effort="800" velocity="5.0"/>
     <dynamics damping="3.5" friction="0.3"/>
   </joint>
@@ -365,14 +377,14 @@
   <!-- Cannon bone (metatarsal/metacarpal): pantograph-kept near vertical -->
   <link name="fr_cannon_link">
-    <inertial><mass value="1.2"/><origin xyz="0 0 -0.05" rpy="0 0 0"/>
-      <inertia ixx="0.0011" iyy="0.0011" izz="0.0002" ixy="0" ixz="0" iyz="0"/></inertial>
-    <visual><origin xyz="0 0 -0.05" rpy="0 0 0"/>
-      <geometry><cylinder radius="0.018" length="0.10"/></geometry><material name="dark_grey"/></visual>
-    <collision><origin xyz="0 0 -0.05" rpy="0 0 0"/>
-      <geometry><cylinder radius="0.016" length="0.10"/></geometry></collision>
+    <inertial><mass value="1.0"/><origin xyz="0 0 -0.09" rpy="0 0 0"/>
+      <inertia ixx="0.0028" iyy="0.0028" izz="0.0003" ixy="0" ixz="0" iyz="0"/></inertial>
+    <visual><origin xyz="0 0 -0.09" rpy="0 0 0"/>
+      <geometry><cylinder radius="0.025" length="0.18"/></geometry><material name="dark_grey"/></visual>
+    <collision><origin xyz="0 0 -0.09" rpy="0 0 0"/>
+      <geometry><cylinder radius="0.025" length="0.18"/></geometry></collision>
   </link>
   <joint name="fr_cannon_joint" type="revolute">
     <parent link="fr_shank_link"/><child link="fr_cannon_link"/>
-    <origin xyz="0 0 -0.18" rpy="0 0 0"/><axis xyz="0 1 0"/>
+    <origin xyz="0 0 -0.34" rpy="0 0 0"/><axis xyz="0 1 0"/>
     <limit lower="-2.0" upper="2.0" effort="100" velocity="6.0"/>
     <dynamics damping="1.0" friction="0.1"/>
@@ -381,13 +393,13 @@
     <link name="fr_foot_link">
     <inertial><mass value="0.4"/><origin xyz="0 0 0" rpy="0 0 0"/>
-      <inertia ixx="0.00026" iyy="0.00026" izz="0.00026" ixy="0" ixz="0" iyz="0"/></inertial>
+      <inertia ixx="0.00040" iyy="0.00040" izz="0.00040" ixy="0" ixz="0" iyz="0"/></inertial>
     <visual><origin xyz="0 0 0" rpy="0 0 0"/>
-      <geometry><sphere radius="0.04"/></geometry><material name="black"/></visual>
+      <geometry><sphere radius="0.05"/></geometry><material name="black"/></visual>
     <collision><origin xyz="0 0 0" rpy="0 0 0"/>
-      <geometry><sphere radius="0.04"/></geometry></collision>
+      <geometry><sphere radius="0.05"/></geometry></collision>
   </link>
   <joint name="fr_foot_joint" type="fixed">
     <parent link="fr_cannon_link"/><child link="fr_foot_link"/>
-    <origin xyz="0 0 -0.10" rpy="0 0 0"/>
+    <origin xyz="0 0 -0.18" rpy="0 0 0"/>
   </joint>
   <gazebo reference="fr_foot_link">
@@ -406,5 +418,5 @@
   <joint name="rl_hip_joint" type="revolute">
     <parent link="base_link"/><child link="rl_hip_link"/>
-    <origin xyz="-0.48 0.24 -0.16" rpy="0 0 0"/>
+    <origin xyz="-0.65 0.36 0.12" rpy="0 0 0"/>
     <axis xyz="0 0 1"/>
     <limit lower="-0.35" upper="0.35" effort="200" velocity="2.0"/>
@@ -413,33 +425,30 @@
   <gazebo reference="rl_hip_link"><material>Gazebo/Grey</material></gazebo>
   <link name="rl_thigh_link">
-    <inertial><mass value="6.0"/><origin xyz="0 0 -0.10" rpy="0 0 0"/>
-      <inertia ixx="0.022" iyy="0.022" izz="0.005" ixy="0" ixz="0" iyz="0"/></inertial>
-    <visual><origin xyz="0 0 -0.10" rpy="0 0 0">
-      </origin><geometry><box size="0.070 0.070 0.20"/></geometry><material name="orange"/></visual>
-    <!-- Ballscrew actuator tube -->
-    <visual><origin xyz="0.040 0 -0.10" rpy="0 0 0"/>
-      <geometry><cylinder radius="0.018" length="0.13"/></geometry><material name="silver"/></visual>
-    <collision><origin xyz="0 0 -0.10" rpy="0 0 0">
-      </origin><geometry><box size="0.070 0.070 0.20"/></geometry></collision>
+    <inertial><mass value="5.0"/><origin xyz="0 0 -0.25" rpy="0 0 0"/>
+      <inertia ixx="0.1068" iyy="0.1068" izz="0.0051" ixy="0" ixz="0" iyz="0"/></inertial>
+    <visual><origin xyz="0 0 -0.25" rpy="0 0 0">
+      </origin><geometry><cylinder radius="0.045" length="0.50"/></geometry><material name="orange"/></visual>
+    <collision><origin xyz="0 0 -0.25" rpy="0 0 0">
+      </origin><geometry><cylinder radius="0.045" length="0.50"/></geometry></collision>
   </link>
   <joint name="rl_thigh_joint" type="revolute">
     <parent link="rl_hip_link"/><child link="rl_thigh_link"/>
     <origin xyz="0 0 -0.10" rpy="0 0 0"/><axis xyz="0 1 0"/>
-    <limit lower="-1.8" upper="1.8" effort="500" velocity="3.0"/>
+    <limit lower="-1.20" upper="0.30" effort="500" velocity="3.0"/>
     <dynamics damping="2.5" friction="0.3"/>
   </joint>
   <gazebo reference="rl_thigh_link"><material>Gazebo/Orange</material></gazebo>
   <link name="rl_shank_link">
-    <inertial><mass value="5.0"/><origin xyz="0 0 -0.09" rpy="0 0 0"/>
-      <inertia ixx="0.015" iyy="0.015" izz="0.003" ixy="0" ixz="0" iyz="0"/></inertial>
-    <visual><origin xyz="0 0 -0.09" rpy="0 0 0">
-      </origin><geometry><box size="0.050 0.050 0.18"/></geometry><material name="dark_grey"/></visual>
-    <collision><origin xyz="0 0 -0.09" rpy="0 0 0">
-      </origin><geometry><box size="0.050 0.050 0.18"/></geometry></collision>
+    <inertial><mass value="4.0"/><origin xyz="0 0 -0.225" rpy="0 0 0"/>
+      <inertia ixx="0.0695" iyy="0.0695" izz="0.0032" ixy="0" ixz="0" iyz="0"/></inertial>
+    <visual><origin xyz="0 0 -0.225" rpy="0 0 0">
+      </origin><geometry><cylinder radius="0.04" length="0.45"/></geometry><material name="dark_grey"/></visual>
+    <collision><origin xyz="0 0 -0.225" rpy="0 0 0">
+      </origin><geometry><cylinder radius="0.04" length="0.45"/></geometry></collision>
   </link>
   <joint name="rl_knee_joint" type="revolute">
     <parent link="rl_thigh_link"/><child link="rl_shank_link"/>
-    <origin xyz="0 0 -0.20" rpy="0 0 0"/><axis xyz="0 1 0"/>
-    <limit lower="-1.8" upper="2.0" effort="800" velocity="5.0"/>
+    <origin xyz="0 0 -0.50" rpy="0 0 0"/><axis xyz="0 1 0"/>
+    <limit lower="0.10" upper="1.80" effort="800" velocity="5.0"/>
     <dynamics damping="3.5" friction="0.3"/>
   </joint>
@@ -447,14 +456,14 @@
   <!-- Cannon bone (metatarsal/metacarpal): pantograph-kept near vertical -->
   <link name="rl_cannon_link">
-    <inertial><mass value="1.2"/><origin xyz="0 0 -0.05" rpy="0 0 0"/>
-      <inertia ixx="0.0011" iyy="0.0011" izz="0.0002" ixy="0" ixz="0" iyz="0"/></inertial>
-    <visual><origin xyz="0 0 -0.05" rpy="0 0 0"/>
-      <geometry><cylinder radius="0.018" length="0.10"/></geometry><material name="dark_grey"/></visual>
-    <collision><origin xyz="0 0 -0.05" rpy="0 0 0"/>
-      <geometry><cylinder radius="0.016" length="0.10"/></geometry></collision>
+    <inertial><mass value="1.2"/><origin xyz="0 0 -0.11" rpy="0 0 0"/>
+      <inertia ixx="0.0049" iyy="0.0049" izz="0.0005" ixy="0" ixz="0" iyz="0"/></inertial>
+    <visual><origin xyz="0 0 -0.11" rpy="0 0 0"/>
+      <geometry><cylinder radius="0.03" length="0.22"/></geometry><material name="dark_grey"/></visual>
+    <collision><origin xyz="0 0 -0.11" rpy="0 0 0"/>
+      <geometry><cylinder radius="0.03" length="0.22"/></geometry></collision>
   </link>
   <joint name="rl_cannon_joint" type="revolute">
     <parent link="rl_shank_link"/><child link="rl_cannon_link"/>
-    <origin xyz="0 0 -0.18" rpy="0 0 0"/><axis xyz="0 1 0"/>
+    <origin xyz="0 0 -0.45" rpy="0 0 0"/><axis xyz="0 1 0"/>
     <limit lower="-2.0" upper="2.0" effort="100" velocity="6.0"/>
     <dynamics damping="1.0" friction="0.1"/>
@@ -462,14 +471,14 @@
   <gazebo reference="rl_cannon_link"><material>Gazebo/DarkGrey</material></gazebo>
     <link name="rl_foot_link">
-    <inertial><mass value="0.4"/><origin xyz="0 0 0" rpy="0 0 0"/>
-      <inertia ixx="0.00026" iyy="0.00026" izz="0.00026" ixy="0" ixz="0" iyz="0"/></inertial>
+    <inertial><mass value="0.5"/><origin xyz="0 0 0" rpy="0 0 0"/>
+      <inertia ixx="0.00072" iyy="0.00072" izz="0.00072" ixy="0" ixz="0" iyz="0"/></inertial>
     <visual><origin xyz="0 0 0" rpy="0 0 0"/>
-      <geometry><sphere radius="0.04"/></geometry><material name="black"/></visual>
+      <geometry><sphere radius="0.06"/></geometry><material name="black"/></visual>
     <collision><origin xyz="0 0 0" rpy="0 0 0"/>
-      <geometry><sphere radius="0.04"/></geometry></collision>
+      <geometry><sphere radius="0.06"/></geometry></collision>
   </link>
   <joint name="rl_foot_joint" type="fixed">
     <parent link="rl_cannon_link"/><child link="rl_foot_link"/>
-    <origin xyz="0 0 -0.10" rpy="0 0 0"/>
+    <origin xyz="0 0 -0.22" rpy="0 0 0"/>
   </joint>
   <gazebo reference="rl_foot_link">
@@ -488,5 +497,5 @@
   <joint name="rr_hip_joint" type="revolute">
     <parent link="base_link"/><child link="rr_hip_link"/>
-    <origin xyz="-0.48 -0.24 -0.16" rpy="0 0 0"/>
+    <origin xyz="-0.65 -0.36 0.12" rpy="0 0 0"/>
     <axis xyz="0 0 1"/>
     <limit lower="-0.35" upper="0.35" effort="200" velocity="2.0"/>
@@ -495,33 +504,30 @@
   <gazebo reference="rr_hip_link"><material>Gazebo/Grey</material></gazebo>
   <link name="rr_thigh_link">
-    <inertial><mass value="6.0"/><origin xyz="0 0 -0.10" rpy="0 0 0"/>
-      <inertia ixx="0.022" iyy="0.022" izz="0.005" ixy="0" ixz="0" iyz="0"/></inertial>
-    <visual><origin xyz="0 0 -0.10" rpy="0 0 0">
-      </origin><geometry><box size="0.070 0.070 0.20"/></geometry><material name="orange"/></visual>
-    <!-- Ballscrew actuator tube -->
-    <visual><origin xyz="0.040 0 -0.10" rpy="0 0 0"/>
-      <geometry><cylinder radius="0.018" length="0.13"/></geometry><material name="silver"/></visual>
-    <collision><origin xyz="0 0 -0.10" rpy="0 0 0">
-      </origin><geometry><box size="0.070 0.070 0.20"/></geometry></collision>
+    <inertial><mass value="5.0"/><origin xyz="0 0 -0.25" rpy="0 0 0"/>
+      <inertia ixx="0.1068" iyy="0.1068" izz="0.0051" ixy="0" ixz="0" iyz="0"/></inertial>
+    <visual><origin xyz="0 0 -0.25" rpy="0 0 0">
+      </origin><geometry><cylinder radius="0.045" length="0.50"/></geometry><material name="orange"/></visual>
+    <collision><origin xyz="0 0 -0.25" rpy="0 0 0">
+      </origin><geometry><cylinder radius="0.045" length="0.50"/></geometry></collision>
   </link>
   <joint name="rr_thigh_joint" type="revolute">
     <parent link="rr_hip_link"/><child link="rr_thigh_link"/>
     <origin xyz="0 0 -0.10" rpy="0 0 0"/><axis xyz="0 1 0"/>
-    <limit lower="-1.8" upper="1.8" effort="500" velocity="3.0"/>
+    <limit lower="-1.20" upper="0.30" effort="500" velocity="3.0"/>
     <dynamics damping="2.5" friction="0.3"/>
   </joint>
   <gazebo reference="rr_thigh_link"><material>Gazebo/Orange</material></gazebo>
   <link name="rr_shank_link">
-    <inertial><mass value="5.0"/><origin xyz="0 0 -0.09" rpy="0 0 0"/>
-      <inertia ixx="0.015" iyy="0.015" izz="0.003" ixy="0" ixz="0" iyz="0"/></inertial>
-    <visual><origin xyz="0 0 -0.09" rpy="0 0 0">
-      </origin><geometry><box size="0.050 0.050 0.18"/></geometry><material name="dark_grey"/></visual>
-    <collision><origin xyz="0 0 -0.09" rpy="0 0 0">
-      </origin><geometry><box size="0.050 0.050 0.18"/></geometry></collision>
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