Commit message: Elk animatronic: realistic mass + 3-gait elk locomotion
Body mass: 20kg -> 28kg (62kg total horse)
- hip: 0.5->2.0kg, thigh: 1.5->3.5kg, shank: 1.0->2.5kg, foot: 0.2->0.4kg
- All inertia tensors recomputed from cylinder/box geometry
- Leg joint damping increased (hip:2.5, knee:3.5)
- PID gains scaled for 62kg (hip:250/15, thigh:500/30, knee:800/50)

Elk-accurate gaits (blendspace_node.py):
- WALK: 4-beat lateral sequence RL->FL->RR->FR, period=1.6s, swing=35%
- TROT: diagonal pairs with suspension, period=0.90s, swing=50%
- GALLOP: rotary gallop FL->RL->FR->RR, period=0.50s, swing=55%

Elk step profile: sin(pi*p^0.7) height (peaks at 40% swing),
p^1.3 forward extension (leg lifts before swinging forward)

Q key now cycles: WALK -> TROT -> GALLOP -> WALK
INSTRUCTIONS2.0.md: Section 11 added

Co-authored-by: Copilot <223556219+Copilot@users.noreply.github.com>

File: ros2_ws/src/robotic_horse_description/urdf/robotic_horse.urdf.xacro (robot description, xacro)
@@ -234,9 +234,10 @@
        BASE LINK
   ═══════════════════════════════════════════════════════ -->
+  <!-- Elk animatronic body: 28kg (frame 12kg + main motors 10kg + costume 6kg) -->
   <link name="base_link">
     <inertial>
-      <mass value="20.0"/>
+      <mass value="28.0"/>
       <origin xyz="0 0 0" rpy="0 0 0"/>
-      <inertia ixx="0.138" iyy="1.075" izz="1.140" ixy="0" ixz="0" iyz="0"/>
+      <inertia ixx="0.356" iyy="1.289" izz="1.353" ixy="0" ixz="0" iyz="0"/>
     </inertial>
     <!-- Main body panel -->
@@ -271,6 +272,6 @@
   <!-- ── FRONT-LEFT ── -->
   <link name="fl_hip_link">
-    <inertial><mass value="0.5"/><origin xyz="0 0 0" rpy="0 0 0"/>
-      <inertia ixx="0.001" iyy="0.001" izz="0.001" ixy="0" ixz="0" iyz="0"/></inertial>
+    <inertial><mass value="2.0"/><origin xyz="0 0 0" rpy="0 0 0"/>
+      <inertia ixx="0.003" iyy="0.003" izz="0.004" ixy="0" ixz="0" iyz="0"/></inertial>
     <visual><origin xyz="0 0 -0.05" rpy="0 0 0"/>
       <geometry><cylinder radius="0.04" length="0.10"/></geometry><material name="silver"/></visual>
@@ -283,10 +284,10 @@
     <axis xyz="0 0 1"/>
     <limit lower="-0.35" upper="0.35" effort="200" velocity="2.0"/>
-    <dynamics damping="0.5" friction="0.1"/>
+    <dynamics damping="2.5" friction="0.3"/>
   </joint>
   <gazebo reference="fl_hip_link"><material>Gazebo/Grey</material></gazebo>
   <link name="fl_thigh_link">
-    <inertial><mass value="1.5"/><origin xyz="0 0 -0.225" rpy="0 0 0"/>
-      <inertia ixx="0.025" iyy="0.025" izz="0.002" ixy="0" ixz="0" iyz="0"/></inertial>
+    <inertial><mass value="3.5"/><origin xyz="0 0 -0.225" rpy="0 0 0"/>
+      <inertia ixx="0.061" iyy="0.061" izz="0.004" ixy="0" ixz="0" iyz="0"/></inertial>
     <visual><origin xyz="0 0 -0.225" rpy="0 0 0"/>
       <geometry><box size="0.04 0.04 0.45"/></geometry><material name="orange"/></visual>
@@ -301,10 +302,10 @@
     <origin xyz="0 0 -0.08" rpy="0 0 0"/><axis xyz="0 1 0"/>
     <limit lower="-1.2" upper="0.5" effort="500" velocity="3.0"/>
-    <dynamics damping="0.5" friction="0.1"/>
+    <dynamics damping="2.5" friction="0.3"/>
   </joint>
   <gazebo reference="fl_thigh_link"><material>Gazebo/Orange</material></gazebo>
   <link name="fl_shank_link">
-    <inertial><mass value="1.0"/><origin xyz="0 0 -0.25" rpy="0 0 0"/>
-      <inertia ixx="0.021" iyy="0.021" izz="0.001" ixy="0" ixz="0" iyz="0"/></inertial>
+    <inertial><mass value="2.5"/><origin xyz="0 0 -0.25" rpy="0 0 0"/>
+      <inertia ixx="0.053" iyy="0.053" izz="0.002" ixy="0" ixz="0" iyz="0"/></inertial>
     <visual><origin xyz="0 0 -0.25" rpy="0 0 0">
       </origin><geometry><box size="0.035 0.035 0.50"/></geometry><material name="dark_grey"/></visual>
@@ -316,10 +317,10 @@
     <origin xyz="0 0 -0.45" rpy="0 0 0"/><axis xyz="0 1 0"/>
     <limit lower="-0.1" upper="2.0" effort="800" velocity="5.0"/>
-    <dynamics damping="0.8" friction="0.1"/>
+    <dynamics damping="3.5" friction="0.3"/>
   </joint>
   <gazebo reference="fl_shank_link"><material>Gazebo/DarkGrey</material></gazebo>
   <link name="fl_foot_link">
-    <inertial><mass value="0.2"/><origin xyz="0 0 0" rpy="0 0 0"/>
-      <inertia ixx="0.0001" iyy="0.0001" izz="0.0001" ixy="0" ixz="0" iyz="0"/></inertial>
+    <inertial><mass value="0.4"/><origin xyz="0 0 0" rpy="0 0 0"/>
+      <inertia ixx="0.00026" iyy="0.00026" izz="0.00026" ixy="0" ixz="0" iyz="0"/></inertial>
     <visual><origin xyz="0 0 0" rpy="0 0 0"/>
       <geometry><sphere radius="0.04"/></geometry><material name="black"/></visual>
@@ -338,6 +339,6 @@
   <!-- ── FRONT-RIGHT ── -->
   <link name="fr_hip_link">
-    <inertial><mass value="0.5"/><origin xyz="0 0 0" rpy="0 0 0"/>
-      <inertia ixx="0.001" iyy="0.001" izz="0.001" ixy="0" ixz="0" iyz="0"/></inertial>
+    <inertial><mass value="2.0"/><origin xyz="0 0 0" rpy="0 0 0"/>
+      <inertia ixx="0.003" iyy="0.003" izz="0.004" ixy="0" ixz="0" iyz="0"/></inertial>
     <visual><origin xyz="0 0 -0.05" rpy="0 0 0"/>
       <geometry><cylinder radius="0.04" length="0.10"/></geometry><material name="silver"/></visual>
@@ -350,10 +351,10 @@
     <axis xyz="0 0 1"/>
     <limit lower="-0.35" upper="0.35" effort="200" velocity="2.0"/>
-    <dynamics damping="0.5" friction="0.1"/>
+    <dynamics damping="2.5" friction="0.3"/>
   </joint>
   <gazebo reference="fr_hip_link"><material>Gazebo/Grey</material></gazebo>
   <link name="fr_thigh_link">
-    <inertial><mass value="1.5"/><origin xyz="0 0 -0.225" rpy="0 0 0"/>
-      <inertia ixx="0.025" iyy="0.025" izz="0.002" ixy="0" ixz="0" iyz="0"/></inertial>
+    <inertial><mass value="3.5"/><origin xyz="0 0 -0.225" rpy="0 0 0"/>
+      <inertia ixx="0.061" iyy="0.061" izz="0.004" ixy="0" ixz="0" iyz="0"/></inertial>
     <visual><origin xyz="0 0 -0.225" rpy="0 0 0">
       </origin><geometry><box size="0.04 0.04 0.45"/></geometry><material name="orange"/></visual>
@@ -368,10 +369,10 @@
     <origin xyz="0 0 -0.08" rpy="0 0 0"/><axis xyz="0 1 0"/>
     <limit lower="-1.2" upper="0.5" effort="500" velocity="3.0"/>
-    <dynamics damping="0.5" friction="0.1"/>
+    <dynamics damping="2.5" friction="0.3"/>
   </joint>
   <gazebo reference="fr_thigh_link"><material>Gazebo/Orange</material></gazebo>
   <link name="fr_shank_link">
-    <inertial><mass value="1.0"/><origin xyz="0 0 -0.25" rpy="0 0 0"/>
-      <inertia ixx="0.021" iyy="0.021" izz="0.001" ixy="0" ixz="0" iyz="0"/></inertial>
+    <inertial><mass value="2.5"/><origin xyz="0 0 -0.25" rpy="0 0 0"/>
+      <inertia ixx="0.053" iyy="0.053" izz="0.002" ixy="0" ixz="0" iyz="0"/></inertial>
     <visual><origin xyz="0 0 -0.25" rpy="0 0 0">
       </origin><geometry><box size="0.035 0.035 0.50"/></geometry><material name="dark_grey"/></visual>
@@ -383,10 +384,10 @@
     <origin xyz="0 0 -0.45" rpy="0 0 0"/><axis xyz="0 1 0"/>
     <limit lower="-0.1" upper="2.0" effort="800" velocity="5.0"/>
-    <dynamics damping="0.8" friction="0.1"/>
+    <dynamics damping="3.5" friction="0.3"/>
   </joint>
   <gazebo reference="fr_shank_link"><material>Gazebo/DarkGrey</material></gazebo>
   <link name="fr_foot_link">
-    <inertial><mass value="0.2"/><origin xyz="0 0 0" rpy="0 0 0"/>
-      <inertia ixx="0.0001" iyy="0.0001" izz="0.0001" ixy="0" ixz="0" iyz="0"/></inertial>
+    <inertial><mass value="0.4"/><origin xyz="0 0 0" rpy="0 0 0"/>
+      <inertia ixx="0.00026" iyy="0.00026" izz="0.00026" ixy="0" ixz="0" iyz="0"/></inertial>
     <visual><origin xyz="0 0 0" rpy="0 0 0"/>
       <geometry><sphere radius="0.04"/></geometry><material name="black"/></visual>
@@ -404,6 +405,6 @@
   <!-- ── REAR-LEFT ── -->
   <link name="rl_hip_link">
-    <inertial><mass value="0.5"/><origin xyz="0 0 0" rpy="0 0 0"/>
-      <inertia ixx="0.001" iyy="0.001" izz="0.001" ixy="0" ixz="0" iyz="0"/></inertial>
+    <inertial><mass value="2.0"/><origin xyz="0 0 0" rpy="0 0 0"/>
+      <inertia ixx="0.003" iyy="0.003" izz="0.004" ixy="0" ixz="0" iyz="0"/></inertial>
     <visual><origin xyz="0 0 -0.05" rpy="0 0 0"/>
       <geometry><cylinder radius="0.04" length="0.10"/></geometry><material name="silver"/></visual>
@@ -416,10 +417,10 @@
     <axis xyz="0 0 1"/>
     <limit lower="-0.35" upper="0.35" effort="200" velocity="2.0"/>
-    <dynamics damping="0.5" friction="0.1"/>
+    <dynamics damping="2.5" friction="0.3"/>
   </joint>
   <gazebo reference="rl_hip_link"><material>Gazebo/Grey</material></gazebo>
   <link name="rl_thigh_link">
-    <inertial><mass value="1.5"/><origin xyz="0 0 -0.225" rpy="0 0 0"/>
-      <inertia ixx="0.025" iyy="0.025" izz="0.002" ixy="0" ixz="0" iyz="0"/></inertial>
+    <inertial><mass value="3.5"/><origin xyz="0 0 -0.225" rpy="0 0 0"/>
+      <inertia ixx="0.061" iyy="0.061" izz="0.004" ixy="0" ixz="0" iyz="0"/></inertial>
     <visual><origin xyz="0 0 -0.225" rpy="0 0 0">
       </origin><geometry><box size="0.04 0.04 0.45"/></geometry><material name="orange"/></visual>
@@ -434,10 +435,10 @@
     <origin xyz="0 0 -0.08" rpy="0 0 0"/><axis xyz="0 1 0"/>
     <limit lower="-1.2" upper="0.5" effort="500" velocity="3.0"/>
-    <dynamics damping="0.5" friction="0.1"/>
+    <dynamics damping="2.5" friction="0.3"/>
   </joint>
   <gazebo reference="rl_thigh_link"><material>Gazebo/Orange</material></gazebo>
   <link name="rl_shank_link">
-    <inertial><mass value="1.0"/><origin xyz="0 0 -0.25" rpy="0 0 0"/>
-      <inertia ixx="0.021" iyy="0.021" izz="0.001" ixy="0" ixz="0" iyz="0"/></inertial>
+    <inertial><mass value="2.5"/><origin xyz="0 0 -0.25" rpy="0 0 0"/>
+      <inertia ixx="0.053" iyy="0.053" izz="0.002" ixy="0" ixz="0" iyz="0"/></inertial>
     <visual><origin xyz="0 0 -0.25" rpy="0 0 0">
       </origin><geometry><box size="0.035 0.035 0.50"/></geometry><material name="dark_grey"/></visual>
@@ -449,10 +450,10 @@
     <origin xyz="0 0 -0.45" rpy="0 0 0"/><axis xyz="0 1 0"/>
     <limit lower="-0.1" upper="2.0" effort="800" velocity="5.0"/>
-    <dynamics damping="0.8" friction="0.1"/>
+    <dynamics damping="3.5" friction="0.3"/>
   </joint>
   <gazebo reference="rl_shank_link"><material>Gazebo/DarkGrey</material></gazebo>
   <link name="rl_foot_link">
-    <inertial><mass value="0.2"/><origin xyz="0 0 0" rpy="0 0 0"/>
-      <inertia ixx="0.0001" iyy="0.0001" izz="0.0001" ixy="0" ixz="0" iyz="0"/></inertial>
+    <inertial><mass value="0.4"/><origin xyz="0 0 0" rpy="0 0 0"/>
+      <inertia ixx="0.00026" iyy="0.00026" izz="0.00026" ixy="0" ixz="0" iyz="0"/></inertial>
     <visual><origin xyz="0 0 0" rpy="0 0 0"/>
       <geometry><sphere radius="0.04"/></geometry><material name="black"/></visual>
@@ -470,6 +471,6 @@
   <!-- ── REAR-RIGHT ── -->
   <link name="rr_hip_link">
-    <inertial><mass value="0.5"/><origin xyz="0 0 0" rpy="0 0 0"/>
-      <inertia ixx="0.001" iyy="0.001" izz="0.001" ixy="0" ixz="0" iyz="0"/></inertial>
+    <inertial><mass value="2.0"/><origin xyz="0 0 0" rpy="0 0 0"/>
+      <inertia ixx="0.003" iyy="0.003" izz="0.004" ixy="0" ixz="0" iyz="0"/></inertial>
     <visual><origin xyz="0 0 -0.05" rpy="0 0 0"/>
       <geometry><cylinder radius="0.04" length="0.10"/></geometry><material name="silver"/></visual>
@@ -482,10 +483,10 @@
     <axis xyz="0 0 1"/>
     <limit lower="-0.35" upper="0.35" effort="200" velocity="2.0"/>
-    <dynamics damping="0.5" friction="0.1"/>
+    <dynamics damping="2.5" friction="0.3"/>
   </joint>
   <gazebo reference="rr_hip_link"><material>Gazebo/Grey</material></gazebo>
   <link name="rr_thigh_link">
-    <inertial><mass value="1.5"/><origin xyz="0 0 -0.225" rpy="0 0 0"/>
-      <inertia ixx="0.025" iyy="0.025" izz="0.002" ixy="0" ixz="0" iyz="0"/></inertial>
+    <inertial><mass value="3.5"/><origin xyz="0 0 -0.225" rpy="0 0 0"/>
+      <inertia ixx="0.061" iyy="0.061" izz="0.004" ixy="0" ixz="0" iyz="0"/></inertial>
     <visual><origin xyz="0 0 -0.225" rpy="0 0 0">
       </origin><geometry><box size="0.04 0.04 0.45"/></geometry><material name="orange"/></visual>
@@ -500,10 +501,10 @@
     <origin xyz="0 0 -0.08" rpy="0 0 0"/><axis xyz="0 1 0"/>
     <limit lower="-1.2" upper="0.5" effort="500" velocity="3.0"/>
-    <dynamics damping="0.5" friction="0.1"/>
+    <dynamics damping="2.5" friction="0.3"/>
   </joint>
   <gazebo reference="rr_thigh_link"><material>Gazebo/Orange</material></gazebo>
   <link name="rr_shank_link">
-    <inertial><mass value="1.0"/><origin xyz="0 0 -0.25" rpy="0 0 0"/>
-      <inertia ixx="0.021" iyy="0.021" izz="0.001" ixy="0" ixz="0" iyz="0"/></inertial>
+    <inertial><mass value="2.5"/><origin xyz="0 0 -0.25" rpy="0 0 0"/>
+      <inertia ixx="0.053" iyy="0.053" izz="0.002" ixy="0" ixz="0" iyz="0"/></inertial>
     <visual><origin xyz="0 0 -0.25" rpy="0 0 0">
       </origin><geometry><box size="0.035 0.035 0.50"/></geometry><material name="dark_grey"/></visual>
@@ -515,10 +516,10 @@
     <origin xyz="0 0 -0.45" rpy="0 0 0"/><axis xyz="0 1 0"/>
     <limit lower="-0.1" upper="2.0" effort="800" velocity="5.0"/>
-    <dynamics damping="0.8" friction="0.1"/>
+    <dynamics damping="3.5" friction="0.3"/>
   </joint>
   <gazebo reference="rr_shank_link"><material>Gazebo/DarkGrey</material></gazebo>
   <link name="rr_foot_link">
-    <inertial><mass value="0.2"/><origin xyz="0 0 0" rpy="0 0 0"/>
-      <inertia ixx="0.0001" iyy="0.0001" izz="0.0001" ixy="0" ixz="0" iyz="0"/></inertial>
+    <inertial><mass value="0.4"/><origin xyz="0 0 0" rpy="0 0 0"/>
+      <inertia ixx="0.00026" iyy="0.00026" izz="0.00026" ixy="0" ixz="0" iyz="0"/></inertial>
     <visual><origin xyz="0 0 0" rpy="0 0 0"/>
       <geometry><sphere radius="0.04"/></geometry><material name="black"/></visual>
