Commit message: Deer leg anatomy: 3-segment legs, front/rear elbow config, cannon bone
- URDF: Shortened thigh 0.45→0.38m and shank 0.50→0.38m (deer proportions)
- URDF: Added cannon bone link+joint (0.22m) per leg — metatarsal/metacarpal
- URDF: Foot reparented from shank to cannon_link
- URDF: Front legs (FL/FR) initial pose: elbow-DOWN
    thigh=+0.564, knee=-1.127, cannon=+0.714
    Carpal (wrist) bends FORWARD (away from cart) — correct for horse forelimbs
- URDF: Rear legs (RL/RR) initial pose: elbow-UP
    thigh=-0.564, knee=+1.127, cannon=-0.414
    Hock bends BACKWARD (toward cart) — correct for horse hindlimbs
- URDF: Widened joint limits to ±1.8 rad for thigh, -1.8/+2.0 for knee
- URDF: Added cannon joints to ros2_control block (position-controlled)
- ros2_control.yaml: 17-joint list, cannon PIDs p=400/d=20
- blendspace_node.py v3: split IK into _ik_3d_front (elbow-down) and
    _ik_3d_rear (elbow-up); added cannon pantograph formula per leg;
    ANKLE_HEIGHT=0.643m IK target (not foot); 17-joint JOINT_ORDER;
    correct front/rear neutral poses in idle publisher
- All geometry verified: ankle at (0,0,-0.643), cannon world angle=8.6°

Cannon bone pantograph: cannon = CANNON_LEAN - (thigh + knee)
Keeps cannon near-vertical (8.6° forward) regardless of leg pose,
simulating red deer check-ligament passive mechanics — zero extra motors.

Co-authored-by: Copilot <223556219+Copilot@users.noreply.github.com>

File: ros2_ws/src/robotic_horse_description/urdf/robotic_horse.urdf.xacro (robot description, xacro)
@@ -288,37 +288,53 @@
   <gazebo reference="fl_hip_link"><material>Gazebo/Grey</material></gazebo>
   <link name="fl_thigh_link">
-    <inertial><mass value="3.5"/><origin xyz="0 0 -0.225" rpy="0 0 0"/>
-      <inertia ixx="0.061" iyy="0.061" izz="0.004" ixy="0" ixz="0" iyz="0"/></inertial>
-    <visual><origin xyz="0 0 -0.225" rpy="0 0 0"/>
-      <geometry><box size="0.04 0.04 0.45"/></geometry><material name="orange"/></visual>
+    <inertial><mass value="3.5"/><origin xyz="0 0 -0.19" rpy="0 0 0"/>
+      <inertia ixx="0.044" iyy="0.044" izz="0.004" ixy="0" ixz="0" iyz="0"/></inertial>
+    <visual><origin xyz="0 0 -0.19" rpy="0 0 0"/>
+      <geometry><box size="0.04 0.04 0.38"/></geometry><material name="orange"/></visual>
     <!-- Ballscrew actuator tube -->
-    <visual><origin xyz="0.025 0 -0.28" rpy="0 0 0"/>
-      <geometry><cylinder radius="0.015" length="0.32"/></geometry><material name="silver"/></visual>
-    <collision><origin xyz="0 0 -0.225" rpy="0 0 0">
-      </origin><geometry><box size="0.04 0.04 0.45"/></geometry></collision>
+    <visual><origin xyz="0.025 0 -0.19" rpy="0 0 0"/>
+      <geometry><cylinder radius="0.015" length="0.25"/></geometry><material name="silver"/></visual>
+    <collision><origin xyz="0 0 -0.19" rpy="0 0 0">
+      </origin><geometry><box size="0.04 0.04 0.38"/></geometry></collision>
   </link>
   <joint name="fl_thigh_joint" type="revolute">
     <parent link="fl_hip_link"/><child link="fl_thigh_link"/>
     <origin xyz="0 0 -0.08" rpy="0 0 0"/><axis xyz="0 1 0"/>
-    <limit lower="-1.2" upper="0.5" effort="500" velocity="3.0"/>
+    <limit lower="-1.8" upper="1.8" effort="500" velocity="3.0"/>
     <dynamics damping="2.5" friction="0.3"/>
   </joint>
   <gazebo reference="fl_thigh_link"><material>Gazebo/Orange</material></gazebo>
   <link name="fl_shank_link">
-    <inertial><mass value="2.5"/><origin xyz="0 0 -0.25" rpy="0 0 0"/>
-      <inertia ixx="0.053" iyy="0.053" izz="0.002" ixy="0" ixz="0" iyz="0"/></inertial>
-    <visual><origin xyz="0 0 -0.25" rpy="0 0 0">
-      </origin><geometry><box size="0.035 0.035 0.50"/></geometry><material name="dark_grey"/></visual>
-    <collision><origin xyz="0 0 -0.25" rpy="0 0 0">
-      </origin><geometry><box size="0.03 0.03 0.50"/></geometry></collision>
+    <inertial><mass value="2.5"/><origin xyz="0 0 -0.19" rpy="0 0 0"/>
+      <inertia ixx="0.031" iyy="0.031" izz="0.002" ixy="0" ixz="0" iyz="0"/></inertial>
+    <visual><origin xyz="0 0 -0.19" rpy="0 0 0">
+      </origin><geometry><box size="0.035 0.035 0.38"/></geometry><material name="dark_grey"/></visual>
+    <collision><origin xyz="0 0 -0.19" rpy="0 0 0">
+      </origin><geometry><box size="0.03 0.03 0.38"/></geometry></collision>
   </link>
   <joint name="fl_knee_joint" type="revolute">
     <parent link="fl_thigh_link"/><child link="fl_shank_link"/>
-    <origin xyz="0 0 -0.45" rpy="0 0 0"/><axis xyz="0 1 0"/>
-    <limit lower="-0.1" upper="2.0" effort="800" velocity="5.0"/>
+    <origin xyz="0 0 -0.38" rpy="0 0 0"/><axis xyz="0 1 0"/>
+    <limit lower="-1.8" upper="2.0" effort="800" velocity="5.0"/>
     <dynamics damping="3.5" friction="0.3"/>
   </joint>
   <gazebo reference="fl_shank_link"><material>Gazebo/DarkGrey</material></gazebo>
-  <link name="fl_foot_link">
+  <!-- Cannon bone (metatarsal/metacarpal): pantograph-kept near vertical -->
+  <link name="fl_cannon_link">
+    <inertial><mass value="0.8"/><origin xyz="0 0 -0.11" rpy="0 0 0"/>
+      <inertia ixx="0.0033" iyy="0.0033" izz="0.0001" ixy="0" ixz="0" iyz="0"/></inertial>
+    <visual><origin xyz="0 0 -0.11" rpy="0 0 0"/>
+      <geometry><cylinder radius="0.012" length="0.22"/></geometry><material name="dark_grey"/></visual>
+    <collision><origin xyz="0 0 -0.11" rpy="0 0 0"/>
+      <geometry><cylinder radius="0.010" length="0.22"/></geometry></collision>
+  </link>
+  <joint name="fl_cannon_joint" type="revolute">
+    <parent link="fl_shank_link"/><child link="fl_cannon_link"/>
+    <origin xyz="0 0 -0.38" rpy="0 0 0"/><axis xyz="0 1 0"/>
+    <limit lower="-2.0" upper="2.0" effort="100" velocity="6.0"/>
+    <dynamics damping="1.0" friction="0.1"/>
+  </joint>
+  <gazebo reference="fl_cannon_link"><material>Gazebo/DarkGrey</material></gazebo>
+    <link name="fl_foot_link">
     <inertial><mass value="0.4"/><origin xyz="0 0 0" rpy="0 0 0"/>
       <inertia ixx="0.00026" iyy="0.00026" izz="0.00026" ixy="0" ixz="0" iyz="0"/></inertial>
@@ -329,6 +345,6 @@
   </link>
   <joint name="fl_foot_joint" type="fixed">
-    <parent link="fl_shank_link"/><child link="fl_foot_link"/>
-    <origin xyz="0 0 -0.50" rpy="0 0 0"/>
+    <parent link="fl_cannon_link"/><child link="fl_foot_link"/>
+    <origin xyz="0 0 -0.22" rpy="0 0 0"/>
   </joint>
   <gazebo reference="fl_foot_link">
@@ -355,37 +371,53 @@
   <gazebo reference="fr_hip_link"><material>Gazebo/Grey</material></gazebo>
   <link name="fr_thigh_link">
-    <inertial><mass value="3.5"/><origin xyz="0 0 -0.225" rpy="0 0 0"/>
-      <inertia ixx="0.061" iyy="0.061" izz="0.004" ixy="0" ixz="0" iyz="0"/></inertial>
-    <visual><origin xyz="0 0 -0.225" rpy="0 0 0">
-      </origin><geometry><box size="0.04 0.04 0.45"/></geometry><material name="orange"/></visual>
+    <inertial><mass value="3.5"/><origin xyz="0 0 -0.19" rpy="0 0 0"/>
+      <inertia ixx="0.044" iyy="0.044" izz="0.004" ixy="0" ixz="0" iyz="0"/></inertial>
+    <visual><origin xyz="0 0 -0.19" rpy="0 0 0">
+      </origin><geometry><box size="0.04 0.04 0.38"/></geometry><material name="orange"/></visual>
     <!-- Ballscrew actuator tube -->
-    <visual><origin xyz="0.025 0 -0.28" rpy="0 0 0"/>
-      <geometry><cylinder radius="0.015" length="0.32"/></geometry><material name="silver"/></visual>
-    <collision><origin xyz="0 0 -0.225" rpy="0 0 0">
-      </origin><geometry><box size="0.04 0.04 0.45"/></geometry></collision>
+    <visual><origin xyz="0.025 0 -0.19" rpy="0 0 0"/>
+      <geometry><cylinder radius="0.015" length="0.25"/></geometry><material name="silver"/></visual>
+    <collision><origin xyz="0 0 -0.19" rpy="0 0 0">
+      </origin><geometry><box size="0.04 0.04 0.38"/></geometry></collision>
   </link>
   <joint name="fr_thigh_joint" type="revolute">
     <parent link="fr_hip_link"/><child link="fr_thigh_link"/>
     <origin xyz="0 0 -0.08" rpy="0 0 0"/><axis xyz="0 1 0"/>
-    <limit lower="-1.2" upper="0.5" effort="500" velocity="3.0"/>
+    <limit lower="-1.8" upper="1.8" effort="500" velocity="3.0"/>
     <dynamics damping="2.5" friction="0.3"/>
   </joint>
   <gazebo reference="fr_thigh_link"><material>Gazebo/Orange</material></gazebo>
   <link name="fr_shank_link">
-    <inertial><mass value="2.5"/><origin xyz="0 0 -0.25" rpy="0 0 0"/>
-      <inertia ixx="0.053" iyy="0.053" izz="0.002" ixy="0" ixz="0" iyz="0"/></inertial>
-    <visual><origin xyz="0 0 -0.25" rpy="0 0 0">
-      </origin><geometry><box size="0.035 0.035 0.50"/></geometry><material name="dark_grey"/></visual>
-    <collision><origin xyz="0 0 -0.25" rpy="0 0 0">
-      </origin><geometry><box size="0.03 0.03 0.50"/></geometry></collision>
+    <inertial><mass value="2.5"/><origin xyz="0 0 -0.19" rpy="0 0 0"/>
+      <inertia ixx="0.031" iyy="0.031" izz="0.002" ixy="0" ixz="0" iyz="0"/></inertial>
+    <visual><origin xyz="0 0 -0.19" rpy="0 0 0">
+      </origin><geometry><box size="0.035 0.035 0.38"/></geometry><material name="dark_grey"/></visual>
+    <collision><origin xyz="0 0 -0.19" rpy="0 0 0">
+      </origin><geometry><box size="0.03 0.03 0.38"/></geometry></collision>
   </link>
   <joint name="fr_knee_joint" type="revolute">
     <parent link="fr_thigh_link"/><child link="fr_shank_link"/>
-    <origin xyz="0 0 -0.45" rpy="0 0 0"/><axis xyz="0 1 0"/>
-    <limit lower="-0.1" upper="2.0" effort="800" velocity="5.0"/>
+    <origin xyz="0 0 -0.38" rpy="0 0 0"/><axis xyz="0 1 0"/>
+    <limit lower="-1.8" upper="2.0" effort="800" velocity="5.0"/>
     <dynamics damping="3.5" friction="0.3"/>
   </joint>
   <gazebo reference="fr_shank_link"><material>Gazebo/DarkGrey</material></gazebo>
-  <link name="fr_foot_link">
+  <!-- Cannon bone (metatarsal/metacarpal): pantograph-kept near vertical -->
+  <link name="fr_cannon_link">
+    <inertial><mass value="0.8"/><origin xyz="0 0 -0.11" rpy="0 0 0"/>
+      <inertia ixx="0.0033" iyy="0.0033" izz="0.0001" ixy="0" ixz="0" iyz="0"/></inertial>
+    <visual><origin xyz="0 0 -0.11" rpy="0 0 0"/>
+      <geometry><cylinder radius="0.012" length="0.22"/></geometry><material name="dark_grey"/></visual>
+    <collision><origin xyz="0 0 -0.11" rpy="0 0 0"/>
+      <geometry><cylinder radius="0.010" length="0.22"/></geometry></collision>
+  </link>
+  <joint name="fr_cannon_joint" type="revolute">
+    <parent link="fr_shank_link"/><child link="fr_cannon_link"/>
+    <origin xyz="0 0 -0.38" rpy="0 0 0"/><axis xyz="0 1 0"/>
+    <limit lower="-2.0" upper="2.0" effort="100" velocity="6.0"/>
+    <dynamics damping="1.0" friction="0.1"/>
+  </joint>
+  <gazebo reference="fr_cannon_link"><material>Gazebo/DarkGrey</material></gazebo>
+    <link name="fr_foot_link">
     <inertial><mass value="0.4"/><origin xyz="0 0 0" rpy="0 0 0"/>
       <inertia ixx="0.00026" iyy="0.00026" izz="0.00026" ixy="0" ixz="0" iyz="0"/></inertial>
@@ -396,6 +428,6 @@
   </link>
   <joint name="fr_foot_joint" type="fixed">
-    <parent link="fr_shank_link"/><child link="fr_foot_link"/>
-    <origin xyz="0 0 -0.50" rpy="0 0 0"/>
+    <parent link="fr_cannon_link"/><child link="fr_foot_link"/>
+    <origin xyz="0 0 -0.22" rpy="0 0 0"/>
   </joint>
   <gazebo reference="fr_foot_link">
@@ -421,37 +453,53 @@
   <gazebo reference="rl_hip_link"><material>Gazebo/Grey</material></gazebo>
   <link name="rl_thigh_link">
-    <inertial><mass value="3.5"/><origin xyz="0 0 -0.225" rpy="0 0 0"/>
-      <inertia ixx="0.061" iyy="0.061" izz="0.004" ixy="0" ixz="0" iyz="0"/></inertial>
-    <visual><origin xyz="0 0 -0.225" rpy="0 0 0">
-      </origin><geometry><box size="0.04 0.04 0.45"/></geometry><material name="orange"/></visual>
+    <inertial><mass value="3.5"/><origin xyz="0 0 -0.19" rpy="0 0 0"/>
+      <inertia ixx="0.044" iyy="0.044" izz="0.004" ixy="0" ixz="0" iyz="0"/></inertial>
+    <visual><origin xyz="0 0 -0.19" rpy="0 0 0">
+      </origin><geometry><box size="0.04 0.04 0.38"/></geometry><material name="orange"/></visual>
     <!-- Ballscrew actuator tube -->
-    <visual><origin xyz="0.025 0 -0.28" rpy="0 0 0"/>
-      <geometry><cylinder radius="0.015" length="0.32"/></geometry><material name="silver"/></visual>
-    <collision><origin xyz="0 0 -0.225" rpy="0 0 0">
-      </origin><geometry><box size="0.04 0.04 0.45"/></geometry></collision>
+    <visual><origin xyz="0.025 0 -0.19" rpy="0 0 0"/>
+      <geometry><cylinder radius="0.015" length="0.25"/></geometry><material name="silver"/></visual>
+    <collision><origin xyz="0 0 -0.19" rpy="0 0 0">
+      </origin><geometry><box size="0.04 0.04 0.38"/></geometry></collision>
   </link>
   <joint name="rl_thigh_joint" type="revolute">
     <parent link="rl_hip_link"/><child link="rl_thigh_link"/>
     <origin xyz="0 0 -0.08" rpy="0 0 0"/><axis xyz="0 1 0"/>
-    <limit lower="-1.2" upper="0.5" effort="500" velocity="3.0"/>
+    <limit lower="-1.8" upper="1.8" effort="500" velocity="3.0"/>
     <dynamics damping="2.5" friction="0.3"/>
   </joint>
   <gazebo reference="rl_thigh_link"><material>Gazebo/Orange</material></gazebo>
   <link name="rl_shank_link">
-    <inertial><mass value="2.5"/><origin xyz="0 0 -0.25" rpy="0 0 0"/>
-      <inertia ixx="0.053" iyy="0.053" izz="0.002" ixy="0" ixz="0" iyz="0"/></inertial>
-    <visual><origin xyz="0 0 -0.25" rpy="0 0 0">
-      </origin><geometry><box size="0.035 0.035 0.50"/></geometry><material name="dark_grey"/></visual>
-    <collision><origin xyz="0 0 -0.25" rpy="0 0 0">
-      </origin><geometry><box size="0.03 0.03 0.50"/></geometry></collision>
+    <inertial><mass value="2.5"/><origin xyz="0 0 -0.19" rpy="0 0 0"/>
+      <inertia ixx="0.031" iyy="0.031" izz="0.002" ixy="0" ixz="0" iyz="0"/></inertial>
+    <visual><origin xyz="0 0 -0.19" rpy="0 0 0">
+      </origin><geometry><box size="0.035 0.035 0.38"/></geometry><material name="dark_grey"/></visual>
+    <collision><origin xyz="0 0 -0.19" rpy="0 0 0">
+      </origin><geometry><box size="0.03 0.03 0.38"/></geometry></collision>
   </link>
   <joint name="rl_knee_joint" type="revolute">
     <parent link="rl_thigh_link"/><child link="rl_shank_link"/>
-    <origin xyz="0 0 -0.45" rpy="0 0 0"/><axis xyz="0 1 0"/>
-    <limit lower="-0.1" upper="2.0" effort="800" velocity="5.0"/>
+    <origin xyz="0 0 -0.38" rpy="0 0 0"/><axis xyz="0 1 0"/>
+    <limit lower="-1.8" upper="2.0" effort="800" velocity="5.0"/>
     <dynamics damping="3.5" friction="0.3"/>
   </joint>
   <gazebo reference="rl_shank_link"><material>Gazebo/DarkGrey</material></gazebo>
-  <link name="rl_foot_link">
+  <!-- Cannon bone (metatarsal/metacarpal): pantograph-kept near vertical -->
+  <link name="rl_cannon_link">
+    <inertial><mass value="0.8"/><origin xyz="0 0 -0.11" rpy="0 0 0"/>
+      <inertia ixx="0.0033" iyy="0.0033" izz="0.0001" ixy="0" ixz="0" iyz="0"/></inertial>
+    <visual><origin xyz="0 0 -0.11" rpy="0 0 0"/>
+      <geometry><cylinder radius="0.012" length="0.22"/></geometry><material name="dark_grey"/></visual>
+    <collision><origin xyz="0 0 -0.11" rpy="0 0 0"/>
+      <geometry><cylinder radius="0.010" length="0.22"/></geometry></collision>
+  </link>
+  <joint name="rl_cannon_joint" type="revolute">
+    <parent link="rl_shank_link"/><child link="rl_cannon_link"/>
+    <origin xyz="0 0 -0.38" rpy="0 0 0"/><axis xyz="0 1 0"/>
+    <limit lower="-2.0" upper="2.0" effort="100" velocity="6.0"/>
+    <dynamics damping="1.0" friction="0.1"/>
+  </joint>
+  <gazebo reference="rl_cannon_link"><material>Gazebo/DarkGrey</material></gazebo>
+    <link name="rl_foot_link">
     <inertial><mass value="0.4"/><origin xyz="0 0 0" rpy="0 0 0"/>
       <inertia ixx="0.00026" iyy="0.00026" izz="0.00026" ixy="0" ixz="0" iyz="0"/></inertial>
@@ -462,6 +510,6 @@
   </link>
   <joint name="rl_foot_joint" type="fixed">
-    <parent link="rl_shank_link"/><child link="rl_foot_link"/>
-    <origin xyz="0 0 -0.50" rpy="0 0 0"/>
+    <parent link="rl_cannon_link"/><child link="rl_foot_link"/>
+    <origin xyz="0 0 -0.22" rpy="0 0 0"/>
   </joint>
   <gazebo reference="rl_foot_link">
@@ -487,37 +535,53 @@
   <gazebo reference="rr_hip_link"><material>Gazebo/Grey</material></gazebo>
   <link name="rr_thigh_link">
-    <inertial><mass value="3.5"/><origin xyz="0 0 -0.225" rpy="0 0 0"/>
-      <inertia ixx="0.061" iyy="0.061" izz="0.004" ixy="0" ixz="0" iyz="0"/></inertial>
-    <visual><origin xyz="0 0 -0.225" rpy="0 0 0">
-      </origin><geometry><box size="0.04 0.04 0.45"/></geometry><material name="orange"/></visual>
+    <inertial><mass value="3.5"/><origin xyz="0 0 -0.19" rpy="0 0 0"/>
+      <inertia ixx="0.044" iyy="0.044" izz="0.004" ixy="0" ixz="0" iyz="0"/></inertial>
+    <visual><origin xyz="0 0 -0.19" rpy="0 0 0">
+      </origin><geometry><box size="0.04 0.04 0.38"/></geometry><material name="orange"/></visual>
     <!-- Ballscrew actuator tube -->
-    <visual><origin xyz="0.025 0 -0.28" rpy="0 0 0"/>
-      <geometry><cylinder radius="0.015" length="0.32"/></geometry><material name="silver"/></visual>
-    <collision><origin xyz="0 0 -0.225" rpy="0 0 0">
-      </origin><geometry><box size="0.04 0.04 0.45"/></geometry></collision>
+    <visual><origin xyz="0.025 0 -0.19" rpy="0 0 0"/>
+      <geometry><cylinder radius="0.015" length="0.25"/></geometry><material name="silver"/></visual>
+    <collision><origin xyz="0 0 -0.19" rpy="0 0 0">
+      </origin><geometry><box size="0.04 0.04 0.38"/></geometry></collision>
   </link>
   <joint name="rr_thigh_joint" type="revolute">
     <parent link="rr_hip_link"/><child link="rr_thigh_link"/>
     <origin xyz="0 0 -0.08" rpy="0 0 0"/><axis xyz="0 1 0"/>
-    <limit lower="-1.2" upper="0.5" effort="500" velocity="3.0"/>
+    <limit lower="-1.8" upper="1.8" effort="500" velocity="3.0"/>
     <dynamics damping="2.5" friction="0.3"/>
   </joint>
   <gazebo reference="rr_thigh_link"><material>Gazebo/Orange</material></gazebo>
   <link name="rr_shank_link">
-    <inertial><mass value="2.5"/><origin xyz="0 0 -0.25" rpy="0 0 0"/>
-      <inertia ixx="0.053" iyy="0.053" izz="0.002" ixy="0" ixz="0" iyz="0"/></inertial>
-    <visual><origin xyz="0 0 -0.25" rpy="0 0 0">
-      </origin><geometry><box size="0.035 0.035 0.50"/></geometry><material name="dark_grey"/></visual>
-    <collision><origin xyz="0 0 -0.25" rpy="0 0 0">
-      </origin><geometry><box size="0.03 0.03 0.50"/></geometry></collision>
+    <inertial><mass value="2.5"/><origin xyz="0 0 -0.19" rpy="0 0 0"/>
+      <inertia ixx="0.031" iyy="0.031" izz="0.002" ixy="0" ixz="0" iyz="0"/></inertial>
+    <visual><origin xyz="0 0 -0.19" rpy="0 0 0">
+      </origin><geometry><box size="0.035 0.035 0.38"/></geometry><material name="dark_grey"/></visual>
+    <collision><origin xyz="0 0 -0.19" rpy="0 0 0">
+      </origin><geometry><box size="0.03 0.03 0.38"/></geometry></collision>
   </link>
   <joint name="rr_knee_joint" type="revolute">
     <parent link="rr_thigh_link"/><child link="rr_shank_link"/>
-    <origin xyz="0 0 -0.45" rpy="0 0 0"/><axis xyz="0 1 0"/>
-    <limit lower="-0.1" upper="2.0" effort="800" velocity="5.0"/>
+    <origin xyz="0 0 -0.38" rpy="0 0 0"/><axis xyz="0 1 0"/>
+    <limit lower="-1.8" upper="2.0" effort="800" velocity="5.0"/>
     <dynamics damping="3.5" friction="0.3"/>
   </joint>
   <gazebo reference="rr_shank_link"><material>Gazebo/DarkGrey</material></gazebo>
-  <link name="rr_foot_link">
+  <!-- Cannon bone (metatarsal/metacarpal): pantograph-kept near vertical -->
+  <link name="rr_cannon_link">
+    <inertial><mass value="0.8"/><origin xyz="0 0 -0.11" rpy="0 0 0"/>
+      <inertia ixx="0.0033" iyy="0.0033" izz="0.0001" ixy="0" ixz="0" iyz="0"/></inertial>
+    <visual><origin xyz="0 0 -0.11" rpy="0 0 0"/>
+      <geometry><cylinder radius="0.012" length="0.22"/></geometry><material name="dark_grey"/></visual>
+    <collision><origin xyz="0 0 -0.11" rpy="0 0 0"/>
+      <geometry><cylinder radius="0.010" length="0.22"/></geometry></collision>
+  </link>
+  <joint name="rr_cannon_joint" type="revolute">
+    <parent link="rr_shank_link"/><child link="rr_cannon_link"/>
+    <origin xyz="0 0 -0.38" rpy="0 0 0"/><axis xyz="0 1 0"/>
+    <limit lower="-2.0" upper="2.0" effort="100" velocity="6.0"/>
+    <dynamics damping="1.0" friction="0.1"/>
+  </joint>
+  <gazebo reference="rr_cannon_link"><material>Gazebo/DarkGrey</material></gazebo>
+    <link name="rr_foot_link">
     <inertial><mass value="0.4"/><origin xyz="0 0 0" rpy="0 0 0"/>
       <inertia ixx="0.00026" iyy="0.00026" izz="0.00026" ixy="0" ixz="0" iyz="0"/></inertial>
@@ -528,6 +592,6 @@
   </link>
   <joint name="rr_foot_joint" type="fixed">
-    <parent link="rr_shank_link"/><child link="rr_foot_link"/>
-    <origin xyz="0 0 -0.50" rpy="0 0 0"/>
+    <parent link="rr_cannon_link"/><child link="rr_foot_link"/>
+    <origin xyz="0 0 -0.22" rpy="0 0 0"/>
   </joint>
   <gazebo reference="rr_foot_link">
@@ -574,8 +638,8 @@
     <joint name="fl_thigh_joint">
       <command_interface name="position">
-        <param name="min">-1.2</param><param name="max">0.5</param>
-      </command_interface>
-      <state_interface name="position">
-        <param name="initial_value">-0.344</param>
+        <param name="min">-1.8</param><param name="max">1.8</param>
+      </command_interface>
+      <state_interface name="position">
+        <param name="initial_value">0.564</param>
       </state_interface>
       <state_interface name="velocity"/>
@@ -584,8 +648,18 @@
     <joint name="fl_knee_joint">
       <command_interface name="position">
-        <param name="min">-0.1</param><param name="max">2.0</param>
-      </command_interface>
-      <state_interface name="position">
-        <param name="initial_value">0.651</param>
+        <param name="min">-1.8</param><param name="max">2.0</param>
+      </command_interface>
+      <state_interface name="position">
+        <param name="initial_value">-1.127</param>
+      </state_interface>
+      <state_interface name="velocity"/>
+      <state_interface name="effort"/>
+    </joint>
+    <joint name="fl_cannon_joint">
+      <command_interface name="position">
+        <param name="min">-2.0</param><param name="max">2.0</param>
+      </command_interface>
+      <state_interface name="position">
+        <param name="initial_value">0.714</param>
       </state_interface>
       <state_interface name="velocity"/>
@@ -605,8 +679,8 @@
     <joint name="fr_thigh_joint">
       <command_interface name="position">
-        <param name="min">-1.2</param><param name="max">0.5</param>
-      </command_interface>
-      <state_interface name="position">
-        <param name="initial_value">-0.344</param>
+        <param name="min">-1.8</param><param name="max">1.8</param>
+      </command_interface>
+      <state_interface name="position">
+        <param name="initial_value">0.564</param>
       </state_interface>
       <state_interface name="velocity"/>
@@ -615,8 +689,18 @@
     <joint name="fr_knee_joint">
       <command_interface name="position">
-        <param name="min">-0.1</param><param name="max">2.0</param>
-      </command_interface>
-      <state_interface name="position">
-        <param name="initial_value">0.651</param>
+        <param name="min">-1.8</param><param name="max">2.0</param>
+      </command_interface>
+      <state_interface name="position">
+        <param name="initial_value">-1.127</param>
+      </state_interface>
+      <state_interface name="velocity"/>
+      <state_interface name="effort"/>
+    </joint>
+    <joint name="fr_cannon_joint">
+      <command_interface name="position">
+        <param name="min">-2.0</param><param name="max">2.0</param>
+      </command_interface>
+      <state_interface name="position">
+        <param name="initial_value">0.714</param>
       </state_interface>
       <state_interface name="velocity"/>
@@ -636,8 +720,8 @@
     <joint name="rl_thigh_joint">
       <command_interface name="position">
-        <param name="min">-1.2</param><param name="max">0.5</param>
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