Commit message: Fix falling forward and bouncy gait
Balance:
- base_link CoM shifted -0.15m rearward to counterbalance head/neck
- neck mass 4.0->2.5kg, head mass 2.0->1.2kg (realistic elk head)
- shaft_to_horse: limits tightened +-0.35->+-0.15 rad, damping 15->40,
  friction 3->10 — cart now firmly holds horse upright

Gait stability (remove bounce):
- WALK: swing_frac 0.35->0.22, step_height 0.20->0.06m (grounded steps)
- TROT: swing_frac 0.50->0.32, step_height 0.30->0.12m
- GALLOP: swing_frac 0.55->0.42, step_height 0.40->0.22m
- Stance feet now press 2cm into ground (fz -= 0.02) for firm contact

Co-authored-by: Copilot <223556219+Copilot@users.noreply.github.com>

File: ros2_ws/src/robotic_horse_description/urdf/robotic_horse.urdf.xacro (robot description, xacro)
@@ -228,6 +228,6 @@
     <origin xyz="3.40 0 1.05" rpy="0 0 0"/>
     <axis xyz="0 1 0"/>
-    <limit lower="-0.35" upper="0.35" effort="2000" velocity="1.0"/>
-    <dynamics damping="15.0" friction="3.0"/>
+    <limit lower="-0.15" upper="0.15" effort="3000" velocity="0.5"/>
+    <dynamics damping="40.0" friction="10.0"/>
   </joint>
   <!-- Collar link: massless pivot point where shaft meets horse.
@@ -249,9 +249,10 @@
        BASE LINK
   ═══════════════════════════════════════════════════════ -->
-  <!-- Elk animatronic body: 45kg (frame 18kg + motors 15kg + costume 12kg) -->
+  <!-- Elk animatronic body: 45kg (frame 18kg + motors 15kg + costume 12kg)
+       CoM shifted -0.15m rear to counterbalance neck/head forward mass. -->
   <link name="base_link">
     <inertial>
       <mass value="45.0"/>
-      <origin xyz="0 0 0" rpy="0 0 0"/>
+      <origin xyz="-0.15 0 0" rpy="0 0 0"/>
       <inertia ixx="1.202" iyy="4.875" izz="5.402" ixy="0" ixz="0" iyz="0"/>
     </inertial>
@@ -282,6 +283,6 @@
        Joint origin at front-top of body (withers area). -->
   <link name="neck_link">
-    <inertial><mass value="4.0"/><origin xyz="0 0 0.275" rpy="0 0 0"/>
-      <inertia ixx="0.111" iyy="0.111" izz="0.020" ixy="0" ixz="0" iyz="0"/></inertial>
+    <inertial><mass value="2.5"/><origin xyz="0 0 0.275" rpy="0 0 0"/>
+      <inertia ixx="0.080" iyy="0.080" izz="0.015" ixy="0" ixz="0" iyz="0"/></inertial>
     <visual><origin xyz="0 0 0.275" rpy="0 0 0"/>
       <geometry><cylinder radius="0.12" length="0.55"/></geometry><material name="body_panel"/></visual>
@@ -296,6 +297,6 @@
   <!-- Head: skull box + snout extension -->
   <link name="head_link">
-    <inertial><mass value="2.0"/><origin xyz="0.10 0 0" rpy="0 0 0"/>
-      <inertia ixx="0.016" iyy="0.031" izz="0.026" ixy="0" ixz="0" iyz="0"/></inertial>
+    <inertial><mass value="1.2"/><origin xyz="0.10 0 0" rpy="0 0 0"/>
+      <inertia ixx="0.010" iyy="0.020" izz="0.016" ixy="0" ixz="0" iyz="0"/></inertial>
     <!-- Skull -->
     <visual><origin xyz="0 0 0" rpy="0 0 0"/>

Commit message: Remove cart, add IMU self-balance, bidirectional adaptive steps
- URDF: Remove entire wagon assembly (cart, wheels, shaft, collar joints)
  base_link is now root link; IMU sensor added on base_link at /imu/data
- ros2_control.yaml: 16 joints (4 legs x 4 each), no cart steer
- blendspace_node.py v5:
  * Subscribe to /imu/data; extract body pitch + roll from quaternion
  * Bidirectional pitch-adaptive step heights: front legs lift more when
    leaning forward, rear legs reduce clearance accordingly
  * Minimum stride enforced per gait (walk 50cm, trot 70cm, gallop 100cm)
    so slow walking still takes large steps at low cadence
  * Balance foot offset: lean forward shifts foot targets backward
  * IMU-corrected idle pose: pitch/roll corrections to thigh/hip angles
  * Removed cart_to_shaft_steer from JOINT_ORDER and all trajectory logic
- gazebo.launch.py: spawn at x=0 y=0 z=1.55 (freestanding); bridge IMU topic

Co-authored-by: Copilot <223556219+Copilot@users.noreply.github.com>

File: ros2_ws/src/robotic_horse_description/urdf/robotic_horse.urdf.xacro (robot description, xacro)
@@ -36,214 +36,29 @@
   <material name="iron">       <color rgba="0.28 0.28 0.28 1"/></material>
   <!-- ═══════════════════════════════════════════════════════
-       WAGON ASSEMBLY
-       cart_base is the physics root spawned at (-2.50, 0, 0.55).
-       Front wheels steer via cart_to_shaft_steer revolute-Z joint.
-       Shaft poles slope up from front axle to horse collar.
-       shaft_to_horse is revolute-Y so horse can pitch on hills.
-       World-frame positions (spawn: x=-2.50, z=0.55):
-         Cart centre    : (-2.50,  0,  0.55)
-         Front axle     : (-1.80,  0,  0.35)  xyz="0.70 0 -0.20" in cart
-         Horse base_link: ( 0.30,  0,  1.00)  xyz="2.10 0 0.65" in shaft_steer
+       IMU SENSOR  — provides body orientation for self-balance
+       Published on /imu/data (bridged from gz transport).
+       Pitch (Y) used to adapt foot step heights per leg.
+       Roll  (X) used to adapt hip Z splay at idle.
   ═══════════════════════════════════════════════════════ -->
-  <!-- ── WAGON BODY (root link) ─────────────────────────────── -->
-  <link name="cart_base">
-    <inertial>
-      <mass value="120.0"/>
-      <origin xyz="0 0 0" rpy="0 0 0"/>
-      <inertia ixx="11.6" iyy="21.2" izz="29.6" ixy="0" ixz="0" iyz="0"/>
-    </inertial>
-    <!-- Main wagon box -->
-    <visual>
-      <origin xyz="0 0 0" rpy="0 0 0"/>
-      <geometry><box size="1.40 1.00 0.40"/></geometry>
-      <material name="wood"/>
-    </visual>
-    <!-- Front footboard -->
-    <visual>
-      <origin xyz="0.73 0 0.25" rpy="0 0 0"/>
-      <geometry><box size="0.06 1.00 0.10"/></geometry>
-      <material name="iron"/>
-    </visual>
-    <!-- Rear board -->
-    <visual>
-      <origin xyz="-0.73 0 0.25" rpy="0 0 0"/>
-      <geometry><box size="0.06 1.00 0.10"/></geometry>
-      <material name="iron"/>
-    </visual>
-    <collision>
-      <origin xyz="0 0 0" rpy="0 0 0"/>
-      <geometry><box size="1.40 1.00 0.40"/></geometry>
-    </collision>
-  </link>
-  <gazebo reference="cart_base"><material>Gazebo/DarkGrey</material></gazebo>
-  <!-- ── REAR-LEFT WHEEL ────────────────────────────────── -->
-  <link name="cart_wheel_rl">
-    <inertial><mass value="5.0"/><origin xyz="0 0 0" rpy="0 0 0"/>
-      <inertia ixx="0.157" iyy="0.306" izz="0.157" ixy="0" ixz="0" iyz="0"/>
-    </inertial>
-    <visual><origin xyz="0 0 0" rpy="1.5708 0 0"/>
-      <geometry><cylinder radius="0.35" length="0.10"/></geometry>
-      <material name="dark_grey"/>
-    </visual>
-    <collision><origin xyz="0 0 0" rpy="1.5708 0 0"/>
-      <geometry><cylinder radius="0.35" length="0.10"/></geometry>
-    </collision>
-  </link>
-  <joint name="cart_to_wheel_rl" type="continuous">
-    <parent link="cart_base"/><child link="cart_wheel_rl"/>
-    <origin xyz="-0.50  0.55 -0.20" rpy="0 0 0"/>
-    <axis xyz="0 1 0"/>
-    <dynamics damping="2.0" friction="1.0"/>
-  </joint>
-  <gazebo reference="cart_wheel_rl">
-    <material>Gazebo/FlatBlack</material>
-    <kp>500000.0</kp><kd>50.0</kd><mu1>0.9</mu1><mu2>0.9</mu2>
+  <!-- IMU sensor on base_link — publishes body orientation for balance -->
+  <gazebo reference="base_link">
+    <sensor name="imu_sensor" type="imu">
+      <always_on>true</always_on>
+      <update_rate>100</update_rate>
+      <topic>/imu/data</topic>
+      <imu>
+        <angular_velocity>
+          <x><noise type="gaussian"><mean>0</mean><stddev>0.001</stddev></noise></x>
+          <y><noise type="gaussian"><mean>0</mean><stddev>0.001</stddev></noise></y>
+          <z><noise type="gaussian"><mean>0</mean><stddev>0.001</stddev></noise></z>
+        </angular_velocity>
+        <linear_acceleration>
+          <x><noise type="gaussian"><mean>0</mean><stddev>0.01</stddev></noise></x>
+          <y><noise type="gaussian"><mean>0</mean><stddev>0.01</stddev></noise></y>
+          <z><noise type="gaussian"><mean>0</mean><stddev>0.01</stddev></noise></z>
+        </linear_acceleration>
+      </imu>
+    </sensor>
   </gazebo>
-  <!-- ── REAR-RIGHT WHEEL ───────────────────────────────── -->
-  <link name="cart_wheel_rr">
-    <inertial><mass value="5.0"/><origin xyz="0 0 0" rpy="0 0 0"/>
-      <inertia ixx="0.157" iyy="0.306" izz="0.157" ixy="0" ixz="0" iyz="0"/>
-    </inertial>
-    <visual><origin xyz="0 0 0" rpy="1.5708 0 0"/>
-      <geometry><cylinder radius="0.35" length="0.10"/></geometry>
-      <material name="dark_grey"/>
-    </visual>
-    <collision><origin xyz="0 0 0" rpy="1.5708 0 0"/>
-      <geometry><cylinder radius="0.35" length="0.10"/></geometry>
-    </collision>
-  </link>
-  <joint name="cart_to_wheel_rr" type="continuous">
-    <parent link="cart_base"/><child link="cart_wheel_rr"/>
-    <origin xyz="-0.50 -0.55 -0.20" rpy="0 0 0"/>
-    <axis xyz="0 1 0"/>
-    <dynamics damping="2.0" friction="1.0"/>
-  </joint>
-  <gazebo reference="cart_wheel_rr">
-    <material>Gazebo/FlatBlack</material>
-    <kp>500000.0</kp><kd>50.0</kd><mu1>0.9</mu1><mu2>0.9</mu2>
-  </gazebo>
-  <!-- ── STEERING JOINT (cart yaw -> front wheels + shaft turn together) ── -->
-  <!-- Revolute-Z at front axle position in cart_base frame.
-       Limits +-35 deg lets cart navigate corners without jackknifing. -->
-  <joint name="cart_to_shaft_steer" type="revolute">
-    <parent link="cart_base"/><child link="shaft_steer_link"/>
-    <origin xyz="0.70 0 -0.20" rpy="0 0 0"/>
-    <axis xyz="0 0 1"/>
-    <limit lower="-0.61" upper="0.61" effort="5000" velocity="1.0"/>
-    <dynamics damping="10.0" friction="2.0"/>
-  </joint>
-  <!-- ── SHAFT + FRONT WHEELS ──────────────────────────────── -->
-  <!-- Origin = front axle centre.  Poles run from (0,+/-0.25,0)
-       up to horse collar at (2.10,+/-0.25,0.65), pitch=17 deg (0.299 rad). -->
-   <link name="shaft_steer_link">
-    <inertial>
-      <mass value="6.0"/>
-      <origin xyz="1.70 0 0.525" rpy="0 0 0"/>
-      <inertia ixx="0.30" iyy="6.50" izz="6.50" ixy="0" ixz="0" iyz="0"/>
-    </inertial>
-    <!-- Left shaft pole (slopes from cart front axle up to horse collar) -->
-    <visual>
-      <origin xyz="1.70 0.25 0.525" rpy="0 -0.299 0"/>
-      <geometry><box size="3.56 0.07 0.07"/></geometry>
-      <material name="wood"/>
-    </visual>
-    <!-- Right shaft pole -->
-    <visual>
-      <origin xyz="1.70 -0.25 0.525" rpy="0 -0.299 0"/>
-      <geometry><box size="3.56 0.07 0.07"/></geometry>
-      <material name="wood"/>
-    </visual>
-    <!-- Front axle crossbar at cart end -->
-    <visual>
-      <origin xyz="0 0 0" rpy="0 0 0"/>
-      <geometry><box size="0.10 0.62 0.10"/></geometry>
-      <material name="iron"/>
-    </visual>
-    <!-- Horse collar yoke at shaft tip -->
-    <visual>
-      <origin xyz="3.40 0 1.05" rpy="0 0 0"/>
-      <geometry><box size="0.10 0.62 0.10"/></geometry>
-      <material name="iron"/>
-    </visual>
-    <!-- Front axle cylinder (visual only) -->
-    <visual>
-      <origin xyz="0 0 0" rpy="1.5708 0 0"/>
-      <geometry><cylinder radius="0.04" length="1.20"/></geometry>
-      <material name="iron"/>
-    </visual>
-  </link>
-  <gazebo reference="shaft_steer_link"><material>Gazebo/Grey</material></gazebo>
-  <!-- ── FRONT-LEFT WHEEL ───────────────────────────────── -->
-  <link name="cart_wheel_fl">
-    <inertial><mass value="5.0"/><origin xyz="0 0 0" rpy="0 0 0"/>
-      <inertia ixx="0.157" iyy="0.306" izz="0.157" ixy="0" ixz="0" iyz="0"/>
-    </inertial>
-    <visual><origin xyz="0 0 0" rpy="1.5708 0 0"/>
-      <geometry><cylinder radius="0.35" length="0.10"/></geometry>
-      <material name="dark_grey"/>
-    </visual>
-    <collision><origin xyz="0 0 0" rpy="1.5708 0 0"/>
-      <geometry><cylinder radius="0.35" length="0.10"/></geometry>
-    </collision>
-  </link>
-  <joint name="shaft_to_wheel_fl" type="continuous">
-    <parent link="shaft_steer_link"/><child link="cart_wheel_fl"/>
-    <origin xyz="0  0.55 0" rpy="0 0 0"/>
-    <axis xyz="0 1 0"/>
-    <dynamics damping="2.0" friction="1.0"/>
-  </joint>
-  <gazebo reference="cart_wheel_fl">
-    <material>Gazebo/FlatBlack</material>
-    <kp>500000.0</kp><kd>50.0</kd><mu1>0.9</mu1><mu2>0.9</mu2>
-  </gazebo>
-  <!-- ── FRONT-RIGHT WHEEL ──────────────────────────────── -->
-  <link name="cart_wheel_fr">
-    <inertial><mass value="5.0"/><origin xyz="0 0 0" rpy="0 0 0"/>
-      <inertia ixx="0.157" iyy="0.306" izz="0.157" ixy="0" ixz="0" iyz="0"/>
-    </inertial>
-    <visual><origin xyz="0 0 0" rpy="1.5708 0 0"/>
-      <geometry><cylinder radius="0.35" length="0.10"/></geometry>
-      <material name="dark_grey"/>
-    </visual>
-    <collision><origin xyz="0 0 0" rpy="1.5708 0 0"/>
-      <geometry><cylinder radius="0.35" length="0.10"/></geometry>
-    </collision>
-  </link>
-  <joint name="shaft_to_wheel_fr" type="continuous">
-    <parent link="shaft_steer_link"/><child link="cart_wheel_fr"/>
-    <origin xyz="0 -0.55 0" rpy="0 0 0"/>
-    <axis xyz="0 1 0"/>
-    <dynamics damping="2.0" friction="1.0"/>
-  </joint>
-  <gazebo reference="cart_wheel_fr">
-    <material>Gazebo/FlatBlack</material>
-    <kp>500000.0</kp><kd>50.0</kd><mu1>0.9</mu1><mu2>0.9</mu2>
-  </gazebo>
-  <!-- ── HORSE PITCH JOINT ──────────────────────────────── -->
-  <!-- Revolute-Y: horse can pitch +/-15 deg on hills.
-       Damping prevents oscillation at the collar. -->
-  <joint name="shaft_to_horse" type="revolute">
-    <parent link="shaft_steer_link"/>
-    <child link="horse_collar_link"/>
-    <origin xyz="3.40 0 1.05" rpy="0 0 0"/>
-    <axis xyz="0 1 0"/>
-    <limit lower="-0.15" upper="0.15" effort="3000" velocity="0.5"/>
-    <dynamics damping="40.0" friction="10.0"/>
-  </joint>
-  <!-- Collar link: massless pivot point where shaft meets horse.
-       Allows the horse to yaw (turn) freely relative to the shaft,
-       simulating a rope-and-collar attachment rather than a rigid bar. -->
-  <link name="horse_collar_link">
-    <inertial><mass value="0.1"/><origin xyz="0 0 0" rpy="0 0 0"/>
-      <inertia ixx="0.001" iyy="0.001" izz="0.001" ixy="0" ixz="0" iyz="0"/></inertial>
-  </link>
-  <joint name="horse_yaw_joint" type="revolute">
-    <parent link="horse_collar_link"/>
-    <child link="base_link"/>
-    <origin xyz="0 0 0" rpy="0 0 0"/>
-    <axis xyz="0 0 1"/>
-    <limit lower="-1.57" upper="1.57" effort="0" velocity="3.0"/>
-    <dynamics damping="5.0" friction="0.5"/>
-  </joint>
   <!-- ═══════════════════════════════════════════════════════
        BASE LINK
@@ -655,7 +470,6 @@
   <!-- ═══════════════════════════════════════════════════════
        ROS2 CONTROL — hardware interface
-       (gazebo_ros2_control reads this at runtime)
-       12 commanded joints: 4x hip(Z) + 4x thigh(Y) + 4x knee(Y)
-       2 passive joints: cart_to_shaft_steer, shaft_to_horse
+       16 commanded joints: 4x hip(Z) + 4x thigh(Y) + 4x knee(Y) + 4x cannon(Y)
+       No passive joints (cart removed — robot is freestanding).
   ═══════════════════════════════════════════════════════ -->
   <ros2_control name="GazeboSystem" type="system">
@@ -663,20 +477,4 @@
       <plugin>gz_ros2_control/GazeboSimSystem</plugin>
     </hardware>
-    <!-- Steering joint — position commanded by blendspace_node -->
-    <joint name="cart_to_shaft_steer">
-      <command_interface name="position">
-        <param name="min">-0.61</param><param name="max">0.61</param>
-      </command_interface>
-      <state_interface name="position">
-        <param name="initial_value">0.0</param>
-      </state_interface>
-      <state_interface name="velocity"/>
-      <state_interface name="effort"/>
-    </joint>
-    <!-- Passive pitch joint — state only -->
-    <joint name="shaft_to_horse">
-      <state_interface name="position"/>
-      <state_interface name="velocity"/>
-    </joint>
     <!-- Front-left -->
     <joint name="fl_hip_joint">
