Commit message: Fix red deer proportions: accurate 1:1 scale
Before: body 1.10x0.48x0.30m, legs L1=L2=0.60m — 4:1 leg/body ratio (too long)
After:  body 1.10x0.38x0.55m, legs L1=0.38/L2=0.36/L3=0.25m — natural 1:1 ratio

Geometry (verified by FK):
  Withers ~1.54m, belly ~1.00m from ground
  Hip joints at (±0.43, ±0.19, -0.22) relative to body center
  Knee bend 56° at neutral — natural deer standing pose
  Body mass 60kg (up from 45kg for larger stag)

URDF: shorter leg segments, deeper body box (0.30→0.55m depth), recessed
  hip joints, scaled inertias/masses throughout all 4 legs
ros2_control.yaml: updated initial angles, PID gains scaled for lighter legs
blendspace_node.py: L1/L2/L3/FOOT_R/BODY_HEIGHT/LEG_POS/HALF_BODY_LENGTH/
  NEUTRAL_* all updated; step heights slightly reduced
gazebo.launch.py: spawn z=1.33m (was 1.55m)

Co-authored-by: Copilot <223556219+Copilot@users.noreply.github.com>

File: ros2_ws/src/robotic_horse_description/urdf/robotic_horse.urdf.xacro (robot description, xacro)
@@ -68,23 +68,23 @@
   <link name="base_link">
     <inertial>
-      <mass value="45.0"/>
-      <origin xyz="-0.15 0 0" rpy="0 0 0"/>
-      <inertia ixx="1.202" iyy="4.875" izz="5.402" ixy="0" ixz="0" iyz="0"/>
+      <mass value="60.0"/>
+      <origin xyz="-0.10 0 0" rpy="0 0 0"/>
+      <inertia ixx="2.234" iyy="7.563" izz="6.772" ixy="0" ixz="0" iyz="0"/>
     </inertial>
     <!-- Main body panel -->
     <visual>
       <origin xyz="0 0 0" rpy="0 0 0"/>
-      <geometry><box size="1.10 0.48 0.30"/></geometry>
+      <geometry><box size="1.10 0.38 0.55"/></geometry>
       <material name="body_panel"/>
     </visual>
     <!-- Top saddle plate -->
     <visual>
-      <origin xyz="-0.06 0 0.15" rpy="0 0 0"/>
-      <geometry><box size="0.70 0.35 0.04"/></geometry>
+      <origin xyz="-0.06 0 0.275" rpy="0 0 0"/>
+      <geometry><box size="0.70 0.32 0.04"/></geometry>
       <material name="silver"/>
     </visual>
     <collision>
       <origin xyz="0 0 0" rpy="0 0 0"/>
-      <geometry><box size="1.10 0.55 0.30"/></geometry>
+      <geometry><box size="1.10 0.45 0.55"/></geometry>
     </collision>
   </link>
@@ -107,5 +107,5 @@
   <joint name="neck_joint" type="fixed">
     <parent link="base_link"/><child link="neck_link"/>
-    <origin xyz="0.62 0 0.15" rpy="0 -0.698 0"/>
+    <origin xyz="0.52 0 0.265" rpy="0 -0.698 0"/>
   </joint>
   <gazebo reference="neck_link"><material>Gazebo/Brown</material></gazebo>
@@ -143,12 +143,12 @@
     <inertial><mass value="4.0"/><origin xyz="0 0 0" rpy="0 0 0"/>
       <inertia ixx="0.012" iyy="0.012" izz="0.007" ixy="0" ixz="0" iyz="0"/></inertial>
-    <visual><origin xyz="0 0 -0.08" rpy="0 0 0"/>
-      <geometry><cylinder radius="0.06" length="0.16"/></geometry><material name="silver"/></visual>
+    <visual><origin xyz="0 0 -0.06" rpy="0 0 0"/>
+      <geometry><cylinder radius="0.05" length="0.12"/></geometry><material name="silver"/></visual>
     <collision><origin xyz="0 0 -0.07" rpy="0 0 0"/>
-      <geometry><cylinder radius="0.04" length="0.14"/></geometry></collision>
+      <geometry><cylinder radius="0.04" length="0.10"/></geometry></collision>
   </link>
   <joint name="fl_hip_joint" type="revolute">
     <parent link="base_link"/><child link="fl_hip_link"/>
-    <origin xyz="0.55 0.28 -0.08" rpy="0 0 0"/>
+    <origin xyz="0.43 0.19 -0.22" rpy="0 0 0"/>
     <axis xyz="0 0 1"/>
     <limit lower="-0.35" upper="0.35" effort="200" velocity="2.0"/>
@@ -159,15 +159,15 @@
     <inertial><mass value="5.5"/><origin xyz="0 0 -0.30" rpy="0 0 0"/>
       <inertia ixx="0.170" iyy="0.170" izz="0.010" ixy="0" ixz="0" iyz="0"/></inertial>
-    <visual><origin xyz="0 0 -0.30" rpy="0 0 0"/>
-      <geometry><box size="0.06 0.06 0.60"/></geometry><material name="orange"/></visual>
+    <visual><origin xyz="0 0 -0.19" rpy="0 0 0"/>
+      <geometry><box size="0.055 0.055 0.38"/></geometry><material name="orange"/></visual>
     <!-- Ballscrew actuator tube -->
-    <visual><origin xyz="0.04 0 -0.30" rpy="0 0 0"/>
-      <geometry><cylinder radius="0.022" length="0.40"/></geometry><material name="silver"/></visual>
-    <collision><origin xyz="0 0 -0.30" rpy="0 0 0">
-      </origin><geometry><box size="0.06 0.06 0.60"/></geometry></collision>
+    <visual><origin xyz="0.035 0 -0.19" rpy="0 0 0"/>
+      <geometry><cylinder radius="0.018" length="0.25"/></geometry><material name="silver"/></visual>
+    <collision><origin xyz="0 0 -0.19" rpy="0 0 0">
+      </origin><geometry><box size="0.055 0.055 0.38"/></geometry></collision>
   </link>
   <joint name="fl_thigh_joint" type="revolute">
     <parent link="fl_hip_link"/><child link="fl_thigh_link"/>
-    <origin xyz="0 0 -0.13" rpy="0 0 0"/><axis xyz="0 1 0"/>
+    <origin xyz="0 0 -0.10" rpy="0 0 0"/><axis xyz="0 1 0"/>
     <limit lower="-1.8" upper="1.8" effort="500" velocity="3.0"/>
     <dynamics damping="2.5" friction="0.3"/>
@@ -177,12 +177,12 @@
     <inertial><mass value="4.0"/><origin xyz="0 0 -0.30" rpy="0 0 0"/>
       <inertia ixx="0.122" iyy="0.122" izz="0.004" ixy="0" ixz="0" iyz="0"/></inertial>
-    <visual><origin xyz="0 0 -0.30" rpy="0 0 0">
-      </origin><geometry><box size="0.050 0.050 0.60"/></geometry><material name="dark_grey"/></visual>
-    <collision><origin xyz="0 0 -0.19" rpy="0 0 0">
-      </origin><geometry><box size="0.04 0.04 0.60"/></geometry></collision>
+    <visual><origin xyz="0 0 -0.18" rpy="0 0 0">
+      </origin><geometry><box size="0.045 0.045 0.36"/></geometry><material name="dark_grey"/></visual>
+    <collision><origin xyz="0 0 -0.18" rpy="0 0 0">
+      </origin><geometry><box size="0.04 0.04 0.36"/></geometry></collision>
   </link>
   <joint name="fl_knee_joint" type="revolute">
     <parent link="fl_thigh_link"/><child link="fl_shank_link"/>
-    <origin xyz="0 0 -0.60" rpy="0 0 0"/><axis xyz="0 1 0"/>
+    <origin xyz="0 0 -0.38" rpy="0 0 0"/><axis xyz="0 1 0"/>
     <limit lower="-1.8" upper="2.0" effort="800" velocity="5.0"/>
     <dynamics damping="3.5" friction="0.3"/>
@@ -191,14 +191,14 @@
   <!-- Cannon bone (metatarsal/metacarpal): pantograph-kept near vertical -->
   <link name="fl_cannon_link">
-    <inertial><mass value="1.5"/><origin xyz="0 0 -0.175" rpy="0 0 0"/>
-      <inertia ixx="0.0155" iyy="0.0155" izz="0.0003" ixy="0" ixz="0" iyz="0"/></inertial>
-    <visual><origin xyz="0 0 -0.175" rpy="0 0 0"/>
-      <geometry><cylinder radius="0.018" length="0.35"/></geometry><material name="dark_grey"/></visual>
-    <collision><origin xyz="0 0 -0.175" rpy="0 0 0"/>
-      <geometry><cylinder radius="0.014" length="0.35"/></geometry></collision>
+    <inertial><mass value="1.0"/><origin xyz="0 0 -0.125" rpy="0 0 0"/>
+      <inertia ixx="0.0053" iyy="0.0053" izz="0.0001" ixy="0" ixz="0" iyz="0"/></inertial>
+    <visual><origin xyz="0 0 -0.125" rpy="0 0 0"/>
+      <geometry><cylinder radius="0.015" length="0.25"/></geometry><material name="dark_grey"/></visual>
+    <collision><origin xyz="0 0 -0.125" rpy="0 0 0"/>
+      <geometry><cylinder radius="0.012" length="0.25"/></geometry></collision>
   </link>
   <joint name="fl_cannon_joint" type="revolute">
     <parent link="fl_shank_link"/><child link="fl_cannon_link"/>
-    <origin xyz="0 0 -0.60" rpy="0 0 0"/><axis xyz="0 1 0"/>
+    <origin xyz="0 0 -0.36" rpy="0 0 0"/><axis xyz="0 1 0"/>
     <limit lower="-2.0" upper="2.0" effort="100" velocity="6.0"/>
     <dynamics damping="1.0" friction="0.1"/>
@@ -209,11 +209,11 @@
       <inertia ixx="0.00026" iyy="0.00026" izz="0.00026" ixy="0" ixz="0" iyz="0"/></inertial>
     <visual><origin xyz="0 0 0" rpy="0 0 0"/>
-      <geometry><sphere radius="0.06"/></geometry><material name="black"/></visual>
+      <geometry><sphere radius="0.05"/></geometry><material name="black"/></visual>
     <collision><origin xyz="0 0 0" rpy="0 0 0"/>
-      <geometry><sphere radius="0.06"/></geometry></collision>
+      <geometry><sphere radius="0.05"/></geometry></collision>
   </link>
   <joint name="fl_foot_joint" type="fixed">
     <parent link="fl_cannon_link"/><child link="fl_foot_link"/>
-    <origin xyz="0 0 -0.35" rpy="0 0 0"/>
+    <origin xyz="0 0 -0.25" rpy="0 0 0"/>
   </joint>
   <gazebo reference="fl_foot_link">
@@ -226,12 +226,12 @@
     <inertial><mass value="4.0"/><origin xyz="0 0 0" rpy="0 0 0"/>
       <inertia ixx="0.012" iyy="0.012" izz="0.007" ixy="0" ixz="0" iyz="0"/></inertial>
-    <visual><origin xyz="0 0 -0.08" rpy="0 0 0"/>
-      <geometry><cylinder radius="0.06" length="0.16"/></geometry><material name="silver"/></visual>
-    <collision><origin xyz="0 0 -0.07" rpy="0 0 0">
-      </origin><geometry><cylinder radius="0.04" length="0.14"/></geometry></collision>
+    <visual><origin xyz="0 0 -0.06" rpy="0 0 0"/>
+      <geometry><cylinder radius="0.05" length="0.12"/></geometry><material name="silver"/></visual>
+    <collision><origin xyz="0 0 -0.05" rpy="0 0 0">
+      </origin><geometry><cylinder radius="0.04" length="0.10"/></geometry></collision>
   </link>
   <joint name="fr_hip_joint" type="revolute">
     <parent link="base_link"/><child link="fr_hip_link"/>
-    <origin xyz="0.55 -0.28 -0.08" rpy="0 0 0"/>
+    <origin xyz="0.43 -0.19 -0.22" rpy="0 0 0"/>
     <axis xyz="0 0 1"/>
     <limit lower="-0.35" upper="0.35" effort="200" velocity="2.0"/>
@@ -242,15 +242,15 @@
     <inertial><mass value="5.5"/><origin xyz="0 0 -0.30" rpy="0 0 0"/>
       <inertia ixx="0.170" iyy="0.170" izz="0.010" ixy="0" ixz="0" iyz="0"/></inertial>
-    <visual><origin xyz="0 0 -0.30" rpy="0 0 0">
-      </origin><geometry><box size="0.06 0.06 0.60"/></geometry><material name="orange"/></visual>
+    <visual><origin xyz="0 0 -0.19" rpy="0 0 0">
+      </origin><geometry><box size="0.055 0.055 0.38"/></geometry><material name="orange"/></visual>
     <!-- Ballscrew actuator tube -->
-    <visual><origin xyz="0.04 0 -0.30" rpy="0 0 0"/>
-      <geometry><cylinder radius="0.022" length="0.40"/></geometry><material name="silver"/></visual>
-    <collision><origin xyz="0 0 -0.30" rpy="0 0 0">
-      </origin><geometry><box size="0.06 0.06 0.60"/></geometry></collision>
+    <visual><origin xyz="0.035 0 -0.19" rpy="0 0 0"/>
+      <geometry><cylinder radius="0.018" length="0.25"/></geometry><material name="silver"/></visual>
+    <collision><origin xyz="0 0 -0.19" rpy="0 0 0">
+      </origin><geometry><box size="0.055 0.055 0.38"/></geometry></collision>
   </link>
   <joint name="fr_thigh_joint" type="revolute">
     <parent link="fr_hip_link"/><child link="fr_thigh_link"/>
-    <origin xyz="0 0 -0.13" rpy="0 0 0"/><axis xyz="0 1 0"/>
+    <origin xyz="0 0 -0.10" rpy="0 0 0"/><axis xyz="0 1 0"/>
     <limit lower="-1.8" upper="1.8" effort="500" velocity="3.0"/>
     <dynamics damping="2.5" friction="0.3"/>
@@ -260,12 +260,12 @@
     <inertial><mass value="4.0"/><origin xyz="0 0 -0.30" rpy="0 0 0"/>
       <inertia ixx="0.122" iyy="0.122" izz="0.004" ixy="0" ixz="0" iyz="0"/></inertial>
-    <visual><origin xyz="0 0 -0.30" rpy="0 0 0">
-      </origin><geometry><box size="0.050 0.050 0.60"/></geometry><material name="dark_grey"/></visual>
-    <collision><origin xyz="0 0 -0.19" rpy="0 0 0">
-      </origin><geometry><box size="0.04 0.04 0.60"/></geometry></collision>
+    <visual><origin xyz="0 0 -0.18" rpy="0 0 0">
+      </origin><geometry><box size="0.045 0.045 0.36"/></geometry><material name="dark_grey"/></visual>
+    <collision><origin xyz="0 0 -0.18" rpy="0 0 0">
+      </origin><geometry><box size="0.04 0.04 0.36"/></geometry></collision>
   </link>
   <joint name="fr_knee_joint" type="revolute">
     <parent link="fr_thigh_link"/><child link="fr_shank_link"/>
-    <origin xyz="0 0 -0.60" rpy="0 0 0"/><axis xyz="0 1 0"/>
+    <origin xyz="0 0 -0.38" rpy="0 0 0"/><axis xyz="0 1 0"/>
     <limit lower="-1.8" upper="2.0" effort="800" velocity="5.0"/>
     <dynamics damping="3.5" friction="0.3"/>
@@ -274,14 +274,14 @@
   <!-- Cannon bone (metatarsal/metacarpal): pantograph-kept near vertical -->
   <link name="fr_cannon_link">
-    <inertial><mass value="1.5"/><origin xyz="0 0 -0.175" rpy="0 0 0"/>
-      <inertia ixx="0.0155" iyy="0.0155" izz="0.0003" ixy="0" ixz="0" iyz="0"/></inertial>
-    <visual><origin xyz="0 0 -0.175" rpy="0 0 0"/>
-      <geometry><cylinder radius="0.018" length="0.35"/></geometry><material name="dark_grey"/></visual>
-    <collision><origin xyz="0 0 -0.175" rpy="0 0 0"/>
-      <geometry><cylinder radius="0.014" length="0.35"/></geometry></collision>
+    <inertial><mass value="1.0"/><origin xyz="0 0 -0.125" rpy="0 0 0"/>
+      <inertia ixx="0.0053" iyy="0.0053" izz="0.0001" ixy="0" ixz="0" iyz="0"/></inertial>
+    <visual><origin xyz="0 0 -0.125" rpy="0 0 0"/>
+      <geometry><cylinder radius="0.015" length="0.25"/></geometry><material name="dark_grey"/></visual>
+    <collision><origin xyz="0 0 -0.125" rpy="0 0 0"/>
+      <geometry><cylinder radius="0.012" length="0.25"/></geometry></collision>
   </link>
   <joint name="fr_cannon_joint" type="revolute">
     <parent link="fr_shank_link"/><child link="fr_cannon_link"/>
-    <origin xyz="0 0 -0.60" rpy="0 0 0"/><axis xyz="0 1 0"/>
+    <origin xyz="0 0 -0.36" rpy="0 0 0"/><axis xyz="0 1 0"/>
     <limit lower="-2.0" upper="2.0" effort="100" velocity="6.0"/>
     <dynamics damping="1.0" friction="0.1"/>
@@ -292,11 +292,11 @@
       <inertia ixx="0.00026" iyy="0.00026" izz="0.00026" ixy="0" ixz="0" iyz="0"/></inertial>
     <visual><origin xyz="0 0 0" rpy="0 0 0"/>
-      <geometry><sphere radius="0.06"/></geometry><material name="black"/></visual>
+      <geometry><sphere radius="0.05"/></geometry><material name="black"/></visual>
     <collision><origin xyz="0 0 0" rpy="0 0 0"/>
-      <geometry><sphere radius="0.06"/></geometry></collision>
+      <geometry><sphere radius="0.05"/></geometry></collision>
   </link>
   <joint name="fr_foot_joint" type="fixed">
     <parent link="fr_cannon_link"/><child link="fr_foot_link"/>
-    <origin xyz="0 0 -0.35" rpy="0 0 0"/>
+    <origin xyz="0 0 -0.25" rpy="0 0 0"/>
   </joint>
   <gazebo reference="fr_foot_link">
@@ -308,12 +308,12 @@
     <inertial><mass value="4.0"/><origin xyz="0 0 0" rpy="0 0 0"/>
       <inertia ixx="0.012" iyy="0.012" izz="0.007" ixy="0" ixz="0" iyz="0"/></inertial>
-    <visual><origin xyz="0 0 -0.08" rpy="0 0 0"/>
-      <geometry><cylinder radius="0.06" length="0.16"/></geometry><material name="silver"/></visual>
-    <collision><origin xyz="0 0 -0.07" rpy="0 0 0">
-      </origin><geometry><cylinder radius="0.04" length="0.14"/></geometry></collision>
+    <visual><origin xyz="0 0 -0.06" rpy="0 0 0"/>
+      <geometry><cylinder radius="0.05" length="0.12"/></geometry><material name="silver"/></visual>
+    <collision><origin xyz="0 0 -0.05" rpy="0 0 0">
+      </origin><geometry><cylinder radius="0.04" length="0.10"/></geometry></collision>
   </link>
   <joint name="rl_hip_joint" type="revolute">
     <parent link="base_link"/><child link="rl_hip_link"/>
-    <origin xyz="-0.55 0.28 -0.08" rpy="0 0 0"/>
+    <origin xyz="-0.43 0.19 -0.22" rpy="0 0 0"/>
     <axis xyz="0 0 1"/>
     <limit lower="-0.35" upper="0.35" effort="200" velocity="2.0"/>
@@ -324,15 +324,15 @@
     <inertial><mass value="5.5"/><origin xyz="0 0 -0.30" rpy="0 0 0"/>
       <inertia ixx="0.170" iyy="0.170" izz="0.010" ixy="0" ixz="0" iyz="0"/></inertial>
-    <visual><origin xyz="0 0 -0.30" rpy="0 0 0">
-      </origin><geometry><box size="0.06 0.06 0.60"/></geometry><material name="orange"/></visual>
+    <visual><origin xyz="0 0 -0.19" rpy="0 0 0">
+      </origin><geometry><box size="0.055 0.055 0.38"/></geometry><material name="orange"/></visual>
     <!-- Ballscrew actuator tube -->
-    <visual><origin xyz="0.04 0 -0.30" rpy="0 0 0"/>
-      <geometry><cylinder radius="0.022" length="0.40"/></geometry><material name="silver"/></visual>
-    <collision><origin xyz="0 0 -0.30" rpy="0 0 0">
-      </origin><geometry><box size="0.06 0.06 0.60"/></geometry></collision>
+    <visual><origin xyz="0.035 0 -0.19" rpy="0 0 0"/>
+      <geometry><cylinder radius="0.018" length="0.25"/></geometry><material name="silver"/></visual>
+    <collision><origin xyz="0 0 -0.19" rpy="0 0 0">
+      </origin><geometry><box size="0.055 0.055 0.38"/></geometry></collision>
   </link>
   <joint name="rl_thigh_joint" type="revolute">
     <parent link="rl_hip_link"/><child link="rl_thigh_link"/>
-    <origin xyz="0 0 -0.13" rpy="0 0 0"/><axis xyz="0 1 0"/>
+    <origin xyz="0 0 -0.10" rpy="0 0 0"/><axis xyz="0 1 0"/>
     <limit lower="-1.8" upper="1.8" effort="500" velocity="3.0"/>
     <dynamics damping="2.5" friction="0.3"/>
@@ -342,12 +342,12 @@
     <inertial><mass value="4.0"/><origin xyz="0 0 -0.30" rpy="0 0 0"/>
       <inertia ixx="0.122" iyy="0.122" izz="0.004" ixy="0" ixz="0" iyz="0"/></inertial>
-    <visual><origin xyz="0 0 -0.30" rpy="0 0 0">
-      </origin><geometry><box size="0.050 0.050 0.60"/></geometry><material name="dark_grey"/></visual>
-    <collision><origin xyz="0 0 -0.19" rpy="0 0 0">
-      </origin><geometry><box size="0.04 0.04 0.60"/></geometry></collision>
+    <visual><origin xyz="0 0 -0.18" rpy="0 0 0">
+      </origin><geometry><box size="0.045 0.045 0.36"/></geometry><material name="dark_grey"/></visual>
+    <collision><origin xyz="0 0 -0.18" rpy="0 0 0">
+      </origin><geometry><box size="0.04 0.04 0.36"/></geometry></collision>
   </link>
   <joint name="rl_knee_joint" type="revolute">
     <parent link="rl_thigh_link"/><child link="rl_shank_link"/>
-    <origin xyz="0 0 -0.60" rpy="0 0 0"/><axis xyz="0 1 0"/>
+    <origin xyz="0 0 -0.38" rpy="0 0 0"/><axis xyz="0 1 0"/>
     <limit lower="-1.8" upper="2.0" effort="800" velocity="5.0"/>
     <dynamics damping="3.5" friction="0.3"/>
@@ -356,14 +356,14 @@
   <!-- Cannon bone (metatarsal/metacarpal): pantograph-kept near vertical -->
   <link name="rl_cannon_link">
-    <inertial><mass value="1.5"/><origin xyz="0 0 -0.175" rpy="0 0 0"/>
-      <inertia ixx="0.0155" iyy="0.0155" izz="0.0003" ixy="0" ixz="0" iyz="0"/></inertial>
-    <visual><origin xyz="0 0 -0.175" rpy="0 0 0"/>
-      <geometry><cylinder radius="0.018" length="0.35"/></geometry><material name="dark_grey"/></visual>
-    <collision><origin xyz="0 0 -0.175" rpy="0 0 0"/>
-      <geometry><cylinder radius="0.014" length="0.35"/></geometry></collision>
+    <inertial><mass value="1.0"/><origin xyz="0 0 -0.125" rpy="0 0 0"/>
+      <inertia ixx="0.0053" iyy="0.0053" izz="0.0001" ixy="0" ixz="0" iyz="0"/></inertial>
+    <visual><origin xyz="0 0 -0.125" rpy="0 0 0"/>
+      <geometry><cylinder radius="0.015" length="0.25"/></geometry><material name="dark_grey"/></visual>
+    <collision><origin xyz="0 0 -0.125" rpy="0 0 0"/>
+      <geometry><cylinder radius="0.012" length="0.25"/></geometry></collision>
   </link>
   <joint name="rl_cannon_joint" type="revolute">
     <parent link="rl_shank_link"/><child link="rl_cannon_link"/>
-    <origin xyz="0 0 -0.60" rpy="0 0 0"/><axis xyz="0 1 0"/>
+    <origin xyz="0 0 -0.36" rpy="0 0 0"/><axis xyz="0 1 0"/>
     <limit lower="-2.0" upper="2.0" effort="100" velocity="6.0"/>
     <dynamics damping="1.0" friction="0.1"/>
@@ -374,11 +374,11 @@
       <inertia ixx="0.00026" iyy="0.00026" izz="0.00026" ixy="0" ixz="0" iyz="0"/></inertial>
     <visual><origin xyz="0 0 0" rpy="0 0 0"/>
-      <geometry><sphere radius="0.06"/></geometry><material name="black"/></visual>
+      <geometry><sphere radius="0.05"/></geometry><material name="black"/></visual>
     <collision><origin xyz="0 0 0" rpy="0 0 0"/>
-      <geometry><sphere radius="0.06"/></geometry></collision>
+      <geometry><sphere radius="0.05"/></geometry></collision>
   </link>
   <joint name="rl_foot_joint" type="fixed">
     <parent link="rl_cannon_link"/><child link="rl_foot_link"/>
-    <origin xyz="0 0 -0.35" rpy="0 0 0"/>
+    <origin xyz="0 0 -0.25" rpy="0 0 0"/>
   </joint>
   <gazebo reference="rl_foot_link">
@@ -390,12 +390,12 @@
     <inertial><mass value="4.0"/><origin xyz="0 0 0" rpy="0 0 0"/>
       <inertia ixx="0.012" iyy="0.012" izz="0.007" ixy="0" ixz="0" iyz="0"/></inertial>
-    <visual><origin xyz="0 0 -0.08" rpy="0 0 0"/>
-      <geometry><cylinder radius="0.06" length="0.16"/></geometry><material name="silver"/></visual>
-    <collision><origin xyz="0 0 -0.07" rpy="0 0 0">
-      </origin><geometry><cylinder radius="0.04" length="0.14"/></geometry></collision>
+    <visual><origin xyz="0 0 -0.06" rpy="0 0 0"/>
+      <geometry><cylinder radius="0.05" length="0.12"/></geometry><material name="silver"/></visual>
+    <collision><origin xyz="0 0 -0.05" rpy="0 0 0">
+      </origin><geometry><cylinder radius="0.04" length="0.10"/></geometry></collision>
   </link>
   <joint name="rr_hip_joint" type="revolute">
     <parent link="base_link"/><child link="rr_hip_link"/>
-    <origin xyz="-0.55 -0.28 -0.08" rpy="0 0 0"/>
+    <origin xyz="-0.43 -0.19 -0.22" rpy="0 0 0"/>
     <axis xyz="0 0 1"/>
     <limit lower="-0.35" upper="0.35" effort="200" velocity="2.0"/>
@@ -406,15 +406,15 @@
     <inertial><mass value="5.5"/><origin xyz="0 0 -0.30" rpy="0 0 0"/>
       <inertia ixx="0.170" iyy="0.170" izz="0.010" ixy="0" ixz="0" iyz="0"/></inertial>
-    <visual><origin xyz="0 0 -0.30" rpy="0 0 0">
-      </origin><geometry><box size="0.06 0.06 0.60"/></geometry><material name="orange"/></visual>
+    <visual><origin xyz="0 0 -0.19" rpy="0 0 0">
+      </origin><geometry><box size="0.055 0.055 0.38"/></geometry><material name="orange"/></visual>
     <!-- Ballscrew actuator tube -->
-    <visual><origin xyz="0.04 0 -0.30" rpy="0 0 0"/>
-      <geometry><cylinder radius="0.022" length="0.40"/></geometry><material name="silver"/></visual>
-    <collision><origin xyz="0 0 -0.30" rpy="0 0 0">
-      </origin><geometry><box size="0.06 0.06 0.60"/></geometry></collision>
+    <visual><origin xyz="0.035 0 -0.19" rpy="0 0 0"/>
+      <geometry><cylinder radius="0.018" length="0.25"/></geometry><material name="silver"/></visual>
+    <collision><origin xyz="0 0 -0.19" rpy="0 0 0">
+      </origin><geometry><box size="0.055 0.055 0.38"/></geometry></collision>
   </link>
   <joint name="rr_thigh_joint" type="revolute">
     <parent link="rr_hip_link"/><child link="rr_thigh_link"/>
-    <origin xyz="0 0 -0.13" rpy="0 0 0"/><axis xyz="0 1 0"/>
+    <origin xyz="0 0 -0.10" rpy="0 0 0"/><axis xyz="0 1 0"/>
     <limit lower="-1.8" upper="1.8" effort="500" velocity="3.0"/>
     <dynamics damping="2.5" friction="0.3"/>
@@ -424,12 +424,12 @@
     <inertial><mass value="4.0"/><origin xyz="0 0 -0.30" rpy="0 0 0"/>
       <inertia ixx="0.122" iyy="0.122" izz="0.004" ixy="0" ixz="0" iyz="0"/></inertial>
-    <visual><origin xyz="0 0 -0.30" rpy="0 0 0">
-      </origin><geometry><box size="0.050 0.050 0.60"/></geometry><material name="dark_grey"/></visual>
-    <collision><origin xyz="0 0 -0.19" rpy="0 0 0">
-      </origin><geometry><box size="0.04 0.04 0.60"/></geometry></collision>
+    <visual><origin xyz="0 0 -0.18" rpy="0 0 0">
+      </origin><geometry><box size="0.045 0.045 0.36"/></geometry><material name="dark_grey"/></visual>
+    <collision><origin xyz="0 0 -0.18" rpy="0 0 0">
+      </origin><geometry><box size="0.04 0.04 0.36"/></geometry></collision>
   </link>
   <joint name="rr_knee_joint" type="revolute">
     <parent link="rr_thigh_link"/><child link="rr_shank_link"/>
-    <origin xyz="0 0 -0.60" rpy="0 0 0"/><axis xyz="0 1 0"/>
+    <origin xyz="0 0 -0.38" rpy="0 0 0"/><axis xyz="0 1 0"/>
     <limit lower="-1.8" upper="2.0" effort="800" velocity="5.0"/>
     <dynamics damping="3.5" friction="0.3"/>
@@ -438,14 +438,14 @@
   <!-- Cannon bone (metatarsal/metacarpal): pantograph-kept near vertical -->
   <link name="rr_cannon_link">
-    <inertial><mass value="1.5"/><origin xyz="0 0 -0.175" rpy="0 0 0"/>
-      <inertia ixx="0.0155" iyy="0.0155" izz="0.0003" ixy="0" ixz="0" iyz="0"/></inertial>
-    <visual><origin xyz="0 0 -0.175" rpy="0 0 0"/>
-      <geometry><cylinder radius="0.018" length="0.35"/></geometry><material name="dark_grey"/></visual>
-    <collision><origin xyz="0 0 -0.175" rpy="0 0 0"/>
-      <geometry><cylinder radius="0.014" length="0.35"/></geometry></collision>
+    <inertial><mass value="1.0"/><origin xyz="0 0 -0.125" rpy="0 0 0"/>
+      <inertia ixx="0.0053" iyy="0.0053" izz="0.0001" ixy="0" ixz="0" iyz="0"/></inertial>
+    <visual><origin xyz="0 0 -0.125" rpy="0 0 0"/>
+      <geometry><cylinder radius="0.015" length="0.25"/></geometry><material name="dark_grey"/></visual>
+    <collision><origin xyz="0 0 -0.125" rpy="0 0 0"/>
+      <geometry><cylinder radius="0.012" length="0.25"/></geometry></collision>
   </link>
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