Commit message: Add cart with anti-roll arms: VW Up sized carriage + 1m wheels + shaft collar
- cart_base is now the root link (replaces freestanding horse)
- VW Up sized carriage body: 3.2 x 1.4 x 0.7m, mass=350kg
- Four 1m-diameter wheels (r=0.5m), mu=0.85, continuous joints
- Two shaft arms (2.5m, span ±0.25m) connect cart to horse collar
- cart_to_shaft_steer: passive Z-revolute ±35° - lets horse steer cart
- shaft_to_collar: passive Y-revolute ±12° - lets horse pitch over bumps
- collar_to_horse: FIXED joint - no X rotation = roll mechanically prevented
- Collar sits at horse haunch (0.30m behind body center), matching real harness
- Spawn at (-4.4, 0, 0.90): horse base_link settles at ~(0, 0, 1.27) world
- Cart joints are passive (not in ros2_control); all 16 horse joints unchanged

Co-authored-by: Copilot <223556219+Copilot@users.noreply.github.com>

File: ros2_ws/src/robotic_horse_description/urdf/robotic_horse.urdf.xacro (robot description, xacro)
@@ -62,4 +62,220 @@
   </gazebo>
   <!-- ═══════════════════════════════════════════════════════
+       CART  —  Root link. Acts as stabilising chassis for the elk.
+       VW-Up size: 3.2m L x 1.4m W x 0.7m H body, 1.0m-diameter wheels.
+       Two parallel shaft arms connect to a wide collar that prevents
+       the horse from rolling left/right (only yaw + limited pitch free).
+       Horse is a FIXED child of the collar — no X-axis freedom = no roll.
+  ═══════════════════════════════════════════════════════ -->
+  <!-- Cart body (root link — entire robot tree starts here) -->
+  <link name="cart_base">
+    <inertial>
+      <mass value="350.0"/>
+      <origin xyz="0 0 0" rpy="0 0 0"/>
+      <!-- 3.2×1.4×0.7m box: Ixx=m(y²+z²)/12, Iyy=m(x²+z²)/12, Izz=m(x²+y²)/12 -->
+      <inertia ixx="71.5" iyy="313.0" izz="355.8" ixy="0" ixz="0" iyz="0"/>
+    </inertial>
+    <!-- Main carriage box -->
+    <visual>
+      <origin xyz="0 0 0" rpy="0 0 0"/>
+      <geometry><box size="3.2 1.4 0.7"/></geometry>
+      <material name="wood"/>
+    </visual>
+    <!-- Roof panel -->
+    <visual>
+      <origin xyz="0.20 0 0.35" rpy="0 0 0"/>
+      <geometry><box size="2.6 1.35 0.05"/></geometry>
+      <material name="dark_grey"/>
+    </visual>
+    <!-- Front fascia -->
+    <visual>
+      <origin xyz="1.58 0 0.10" rpy="0 0 0"/>
+      <geometry><box size="0.06 1.35 0.50"/></geometry>
+      <material name="dark_grey"/>
+    </visual>
+    <collision>
+      <origin xyz="0 0 0" rpy="0 0 0"/>
+      <geometry><box size="3.2 1.4 0.7"/></geometry>
+    </collision>
+  </link>
+  <gazebo reference="cart_base">
+    <material>Gazebo/WoodPallet</material>
+  </gazebo>
+  <!-- ── CART WHEELS (1.0m diameter, continuous) ──────────────────── -->
+  <link name="cart_fl_wheel_link">
+    <inertial>
+      <mass value="8.0"/>
+      <origin xyz="0 0 0" rpy="0 0 0"/>
+      <!-- Solid cylinder: Ixx=Izz=m(3r²+l²)/12, Iyy=mr²/2 -->
+      <inertia ixx="0.515" iyy="1.000" izz="0.515" ixy="0" ixz="0" iyz="0"/>
+    </inertial>
+    <visual>
+      <origin xyz="0 0 0" rpy="1.5708 0 0"/>
+      <geometry><cylinder radius="0.50" length="0.15"/></geometry>
+      <material name="black"/>
+    </visual>
+    <collision>
+      <origin xyz="0 0 0" rpy="1.5708 0 0"/>
+      <geometry><cylinder radius="0.50" length="0.15"/></geometry>
+    </collision>
+  </link>
+  <joint name="cart_fl_wheel_joint" type="continuous">
+    <parent link="cart_base"/><child link="cart_fl_wheel_link"/>
+    <origin xyz="1.2 0.72 -0.35" rpy="0 0 0"/>
+    <axis xyz="0 1 0"/>
+    <dynamics damping="0.4" friction="0.5"/>
+  </joint>
+  <gazebo reference="cart_fl_wheel_link">
+    <material>Gazebo/FlatBlack</material>
+    <mu1>0.85</mu1><mu2>0.85</mu2><kp>1000000</kp><kd>80</kd>
+  </gazebo>
+  <link name="cart_fr_wheel_link">
+    <inertial><mass value="8.0"/><origin xyz="0 0 0" rpy="0 0 0"/>
+      <inertia ixx="0.515" iyy="1.000" izz="0.515" ixy="0" ixz="0" iyz="0"/></inertial>
+    <visual><origin xyz="0 0 0" rpy="1.5708 0 0"/>
+      <geometry><cylinder radius="0.50" length="0.15"/></geometry><material name="black"/></visual>
+    <collision><origin xyz="0 0 0" rpy="1.5708 0 0"/>
+      <geometry><cylinder radius="0.50" length="0.15"/></geometry></collision>
+  </link>
+  <joint name="cart_fr_wheel_joint" type="continuous">
+    <parent link="cart_base"/><child link="cart_fr_wheel_link"/>
+    <origin xyz="1.2 -0.72 -0.35" rpy="0 0 0"/>
+    <axis xyz="0 1 0"/>
+    <dynamics damping="0.4" friction="0.5"/>
+  </joint>
+  <gazebo reference="cart_fr_wheel_link">
+    <material>Gazebo/FlatBlack</material>
+    <mu1>0.85</mu1><mu2>0.85</mu2><kp>1000000</kp><kd>80</kd>
+  </gazebo>
+  <link name="cart_rl_wheel_link">
+    <inertial><mass value="8.0"/><origin xyz="0 0 0" rpy="0 0 0"/>
+      <inertia ixx="0.515" iyy="1.000" izz="0.515" ixy="0" ixz="0" iyz="0"/></inertial>
+    <visual><origin xyz="0 0 0" rpy="1.5708 0 0"/>
+      <geometry><cylinder radius="0.50" length="0.15"/></geometry><material name="black"/></visual>
+    <collision><origin xyz="0 0 0" rpy="1.5708 0 0">
+      </origin><geometry><cylinder radius="0.50" length="0.15"/></geometry></collision>
+  </link>
+  <joint name="cart_rl_wheel_joint" type="continuous">
+    <parent link="cart_base"/><child link="cart_rl_wheel_link"/>
+    <origin xyz="-1.2 0.72 -0.35" rpy="0 0 0"/>
+    <axis xyz="0 1 0"/>
+    <dynamics damping="0.4" friction="0.5"/>
+  </joint>
+  <gazebo reference="cart_rl_wheel_link">
+    <material>Gazebo/FlatBlack</material>
+    <mu1>0.85</mu1><mu2>0.85</mu2><kp>1000000</kp><kd>80</kd>
+  </gazebo>
+  <link name="cart_rr_wheel_link">
+    <inertial><mass value="8.0"/><origin xyz="0 0 0" rpy="0 0 0"/>
+      <inertia ixx="0.515" iyy="1.000" izz="0.515" ixy="0" ixz="0" iyz="0"/></inertial>
+    <visual><origin xyz="0 0 0" rpy="1.5708 0 0"/>
+      <geometry><cylinder radius="0.50" length="0.15"/></geometry><material name="black"/></visual>
+    <collision><origin xyz="0 0 0" rpy="1.5708 0 0">
+      </origin><geometry><cylinder radius="0.50" length="0.15"/></geometry></collision>
+  </link>
+  <joint name="cart_rr_wheel_joint" type="continuous">
+    <parent link="cart_base"/><child link="cart_rr_wheel_link"/>
+    <origin xyz="-1.2 -0.72 -0.35" rpy="0 0 0"/>
+    <axis xyz="0 1 0"/>
+    <dynamics damping="0.4" friction="0.5"/>
+  </joint>
+  <gazebo reference="cart_rr_wheel_link">
+    <material>Gazebo/FlatBlack</material>
+    <mu1>0.85</mu1><mu2>0.85</mu2><kp>1000000</kp><kd>80</kd>
+  </gazebo>
+  <!-- ── SHAFT ARMS  —  two parallel poles running alongside the horse ─── -->
+  <!-- Pivot (cart_to_shaft_steer) is at cart front at horse-body height.   -->
+  <!-- Arms spread to ±0.25m spanning the horse body (0.38m wide).         -->
+  <!-- This wide stance mechanically prevents roll via geometry.            -->
+  <link name="shaft_steer_link">
+    <inertial>
+      <mass value="8.0"/>
+      <origin xyz="1.25 0 0" rpy="0 0 0"/>
+      <inertia ixx="0.040" iyy="1.680" izz="1.680" ixy="0" ixz="0" iyz="0"/>
+    </inertial>
+    <!-- Left shaft arm -->
+    <visual>
+      <origin xyz="1.25 0.25 0" rpy="0 0 0"/>
+      <geometry><box size="2.50 0.06 0.06"/></geometry>
+      <material name="iron"/>
+    </visual>
+    <!-- Right shaft arm -->
+    <visual>
+      <origin xyz="1.25 -0.25 0" rpy="0 0 0"/>
+      <geometry><box size="2.50 0.06 0.06"/></geometry>
+      <material name="iron"/>
+    </visual>
+    <!-- Cross brace at pivot end -->
+    <visual>
+      <origin xyz="0.04 0 0" rpy="0 0 0"/>
+      <geometry><box size="0.08 0.56 0.06"/></geometry>
+      <material name="iron"/>
+    </visual>
+    <!-- Cross brace at collar end -->
+    <visual>
+      <origin xyz="2.46 0 0" rpy="0 0 0"/>
+      <geometry><box size="0.08 0.56 0.06"/></geometry>
+      <material name="iron"/>
+    </visual>
+    <collision>
+      <origin xyz="1.25 0 0" rpy="0 0 0"/>
+      <geometry><box size="2.50 0.56 0.08"/></geometry>
+    </collision>
+  </link>
+  <!-- cart_to_shaft_steer: PASSIVE yaw joint — horse turns, pulls cart around. -->
+  <!-- Limits ±35° so horse can turn tightly without jackknifing the cart.     -->
+  <joint name="cart_to_shaft_steer" type="revolute">
+    <parent link="cart_base"/><child link="shaft_steer_link"/>
+    <origin xyz="1.6 0 0.42" rpy="0 0 0"/>
+    <axis xyz="0 0 1"/>
+    <limit lower="-0.61" upper="0.61" effort="200" velocity="2.0"/>
+    <dynamics damping="15.0" friction="3.0"/>
+  </joint>
+  <gazebo reference="shaft_steer_link"><material>Gazebo/Grey</material></gazebo>
+  <!-- ── COLLAR  —  wide yoke that prevents horse rolling L/R ─────────── -->
+  <!-- collar_to_horse is FIXED — no X rotation possible = roll prevented.  -->
+  <!-- Only freedoms are: Z-yaw (cart_to_shaft_steer) + Y-pitch (here).    -->
+  <link name="horse_collar_link">
+    <inertial>
+      <mass value="3.0"/>
+      <origin xyz="0 0 0" rpy="0 0 0"/>
+      <inertia ixx="0.060" iyy="0.010" izz="0.062" ixy="0" ixz="0" iyz="0"/>
+    </inertial>
+    <!-- Wide collar bar spanning both sides of horse body -->
+    <visual>
+      <origin xyz="0 0 0" rpy="0 0 0"/>
+      <geometry><box size="0.06 0.58 0.32"/></geometry>
+      <material name="iron"/>
+    </visual>
+    <!-- Side attachment brackets (show the connection points on horse sides) -->
+    <visual>
+      <origin xyz="0 0.29 0" rpy="0 0 0"/>
+      <geometry><cylinder radius="0.04" length="0.10"/></geometry>
+      <material name="silver"/>
+    </visual>
+    <visual>
+      <origin xyz="0 -0.29 0" rpy="0 0 0"/>
+      <geometry><cylinder radius="0.04" length="0.10"/></geometry>
+      <material name="silver"/>
+    </visual>
+    <!-- NO collision geometry — collar is fixed to horse body, no contact needed -->
+  </link>
+  <!-- shaft_to_collar: PASSIVE pitch joint — horse pitches over bumps. -->
+  <!-- Tight limits ±12° + high damping keeps horse level while gait runs.  -->
+  <joint name="shaft_to_collar" type="revolute">
+    <parent link="shaft_steer_link"/><child link="horse_collar_link"/>
+    <origin xyz="2.50 0 0" rpy="0 0 0"/>
+    <axis xyz="0 1 0"/>
+    <limit lower="-0.21" upper="0.21" effort="500" velocity="2.0"/>
+    <dynamics damping="50.0" friction="10.0"/>
+  </joint>
+  <gazebo reference="horse_collar_link"><material>Gazebo/Grey</material></gazebo>
+  <!-- FIXED: horse body is rigidly attached to collar. Collar is 0.30m behind
+       horse center so arms connect at haunch area (like real carriage harness). -->
+  <joint name="collar_to_horse" type="fixed">
+    <parent link="horse_collar_link"/><child link="base_link"/>
+    <origin xyz="0.30 0 0" rpy="0 0 0"/>
+  </joint>
+  <!-- ═══════════════════════════════════════════════════════
        BASE LINK
   ═══════════════════════════════════════════════════════ -->
