Commit message: Percheron proportions + free-standing horse + rope cart
Animal rationale:
- Current Red Deer (narrow, tall) unstable for robot gait
- Recommended Percheron Draft Horse: historic carriage horse with
  compact, wide, heavy proportions that match Spot-like robot kinematics

Structural changes:
- Horse (base_link) is now FREE-STANDING root link again
- Cart removed from rigid kinematic chain
- Cart reattached via 2.5m rope: 4 passive revolute joints (2 universal
  joints = yaw+pitch at each end) let rope swing in any direction
- Horse pulls cart naturally; cart cannot prevent horse rolling

Percheron geometry (FK-verified: hip=0.7189m, target 0.72m):
  L1=0.28m, L2=0.26m, L3=0.16m, FOOT_R=0.04m
  Body: 1.10x0.55x0.48m (wider, lower), mass=160kg
  Hip stance: y=+-0.25m (was +-0.19m), z=-0.20m (was -0.22m)
  Neutral: thigh=+-0.25, knee=-+0.55, cannon=+-0.40/-0.20

PID gains: p_thigh=1200, p_knee=1800 (heavier body needs stronger hold)
Step heights: walk=0.15, trot=0.25, gallop=0.40m (scaled for shorter legs)
Spawn z=1.02m (horse freestanding), cart follows at ~-4.65m via rope

Co-authored-by: Copilot <223556219+Copilot@users.noreply.github.com>

File: ros2_ws/src/robotic_horse_description/urdf/robotic_horse.urdf.xacro (robot description, xacro)
@@ -62,220 +62,4 @@
   </gazebo>
   <!-- ═══════════════════════════════════════════════════════
-       CART  —  Root link. Acts as stabilising chassis for the elk.
-       VW-Up size: 3.2m L x 1.4m W x 0.7m H body, 1.0m-diameter wheels.
-       Two parallel shaft arms connect to a wide collar that prevents
-       the horse from rolling left/right (only yaw + limited pitch free).
-       Horse is a FIXED child of the collar — no X-axis freedom = no roll.
-  ═══════════════════════════════════════════════════════ -->
-  <!-- Cart body (root link — entire robot tree starts here) -->
-  <link name="cart_base">
-    <inertial>
-      <mass value="350.0"/>
-      <origin xyz="0 0 0" rpy="0 0 0"/>
-      <!-- 3.2×1.4×0.7m box: Ixx=m(y²+z²)/12, Iyy=m(x²+z²)/12, Izz=m(x²+y²)/12 -->
-      <inertia ixx="71.5" iyy="313.0" izz="355.8" ixy="0" ixz="0" iyz="0"/>
-    </inertial>
-    <!-- Main carriage box -->
-    <visual>
-      <origin xyz="0 0 0" rpy="0 0 0"/>
-      <geometry><box size="3.2 1.4 0.7"/></geometry>
-      <material name="wood"/>
-    </visual>
-    <!-- Roof panel -->
-    <visual>
-      <origin xyz="0.20 0 0.35" rpy="0 0 0"/>
-      <geometry><box size="2.6 1.35 0.05"/></geometry>
-      <material name="dark_grey"/>
-    </visual>
-    <!-- Front fascia -->
-    <visual>
-      <origin xyz="1.58 0 0.10" rpy="0 0 0"/>
-      <geometry><box size="0.06 1.35 0.50"/></geometry>
-      <material name="dark_grey"/>
-    </visual>
-    <collision>
-      <origin xyz="0 0 0" rpy="0 0 0"/>
-      <geometry><box size="3.2 1.4 0.7"/></geometry>
-    </collision>
-  </link>
-  <gazebo reference="cart_base">
-    <material>Gazebo/WoodPallet</material>
-  </gazebo>
-  <!-- ── CART WHEELS (1.0m diameter, continuous) ──────────────────── -->
-  <link name="cart_fl_wheel_link">
-    <inertial>
-      <mass value="8.0"/>
-      <origin xyz="0 0 0" rpy="0 0 0"/>
-      <!-- Solid cylinder: Ixx=Izz=m(3r²+l²)/12, Iyy=mr²/2 -->
-      <inertia ixx="0.515" iyy="1.000" izz="0.515" ixy="0" ixz="0" iyz="0"/>
-    </inertial>
-    <visual>
-      <origin xyz="0 0 0" rpy="1.5708 0 0"/>
-      <geometry><cylinder radius="0.50" length="0.15"/></geometry>
-      <material name="black"/>
-    </visual>
-    <collision>
-      <origin xyz="0 0 0" rpy="1.5708 0 0"/>
-      <geometry><cylinder radius="0.50" length="0.15"/></geometry>
-    </collision>
-  </link>
-  <joint name="cart_fl_wheel_joint" type="continuous">
-    <parent link="cart_base"/><child link="cart_fl_wheel_link"/>
-    <origin xyz="1.2 0.72 -0.35" rpy="0 0 0"/>
-    <axis xyz="0 1 0"/>
-    <dynamics damping="0.4" friction="0.5"/>
-  </joint>
-  <gazebo reference="cart_fl_wheel_link">
-    <material>Gazebo/FlatBlack</material>
-    <mu1>0.85</mu1><mu2>0.85</mu2><kp>1000000</kp><kd>80</kd>
-  </gazebo>
-  <link name="cart_fr_wheel_link">
-    <inertial><mass value="8.0"/><origin xyz="0 0 0" rpy="0 0 0"/>
-      <inertia ixx="0.515" iyy="1.000" izz="0.515" ixy="0" ixz="0" iyz="0"/></inertial>
-    <visual><origin xyz="0 0 0" rpy="1.5708 0 0"/>
-      <geometry><cylinder radius="0.50" length="0.15"/></geometry><material name="black"/></visual>
-    <collision><origin xyz="0 0 0" rpy="1.5708 0 0"/>
-      <geometry><cylinder radius="0.50" length="0.15"/></geometry></collision>
-  </link>
-  <joint name="cart_fr_wheel_joint" type="continuous">
-    <parent link="cart_base"/><child link="cart_fr_wheel_link"/>
-    <origin xyz="1.2 -0.72 -0.35" rpy="0 0 0"/>
-    <axis xyz="0 1 0"/>
-    <dynamics damping="0.4" friction="0.5"/>
-  </joint>
-  <gazebo reference="cart_fr_wheel_link">
-    <material>Gazebo/FlatBlack</material>
-    <mu1>0.85</mu1><mu2>0.85</mu2><kp>1000000</kp><kd>80</kd>
-  </gazebo>
-  <link name="cart_rl_wheel_link">
-    <inertial><mass value="8.0"/><origin xyz="0 0 0" rpy="0 0 0"/>
-      <inertia ixx="0.515" iyy="1.000" izz="0.515" ixy="0" ixz="0" iyz="0"/></inertial>
-    <visual><origin xyz="0 0 0" rpy="1.5708 0 0"/>
-      <geometry><cylinder radius="0.50" length="0.15"/></geometry><material name="black"/></visual>
-    <collision><origin xyz="0 0 0" rpy="1.5708 0 0">
-      </origin><geometry><cylinder radius="0.50" length="0.15"/></geometry></collision>
-  </link>
-  <joint name="cart_rl_wheel_joint" type="continuous">
-    <parent link="cart_base"/><child link="cart_rl_wheel_link"/>
-    <origin xyz="-1.2 0.72 -0.35" rpy="0 0 0"/>
-    <axis xyz="0 1 0"/>
-    <dynamics damping="0.4" friction="0.5"/>
-  </joint>
-  <gazebo reference="cart_rl_wheel_link">
-    <material>Gazebo/FlatBlack</material>
-    <mu1>0.85</mu1><mu2>0.85</mu2><kp>1000000</kp><kd>80</kd>
-  </gazebo>
-  <link name="cart_rr_wheel_link">
-    <inertial><mass value="8.0"/><origin xyz="0 0 0" rpy="0 0 0"/>
-      <inertia ixx="0.515" iyy="1.000" izz="0.515" ixy="0" ixz="0" iyz="0"/></inertial>
-    <visual><origin xyz="0 0 0" rpy="1.5708 0 0"/>
-      <geometry><cylinder radius="0.50" length="0.15"/></geometry><material name="black"/></visual>
-    <collision><origin xyz="0 0 0" rpy="1.5708 0 0">
-      </origin><geometry><cylinder radius="0.50" length="0.15"/></geometry></collision>
-  </link>
-  <joint name="cart_rr_wheel_joint" type="continuous">
-    <parent link="cart_base"/><child link="cart_rr_wheel_link"/>
-    <origin xyz="-1.2 -0.72 -0.35" rpy="0 0 0"/>
-    <axis xyz="0 1 0"/>
-    <dynamics damping="0.4" friction="0.5"/>
-  </joint>
-  <gazebo reference="cart_rr_wheel_link">
-    <material>Gazebo/FlatBlack</material>
-    <mu1>0.85</mu1><mu2>0.85</mu2><kp>1000000</kp><kd>80</kd>
-  </gazebo>
-  <!-- ── SHAFT ARMS  —  two parallel poles running alongside the horse ─── -->
-  <!-- Pivot (cart_to_shaft_steer) is at cart front at horse-body height.   -->
-  <!-- Arms spread to ±0.25m spanning the horse body (0.38m wide).         -->
-  <!-- This wide stance mechanically prevents roll via geometry.            -->
-  <link name="shaft_steer_link">
-    <inertial>
-      <mass value="8.0"/>
-      <origin xyz="1.25 0 0" rpy="0 0 0"/>
-      <inertia ixx="0.040" iyy="1.680" izz="1.680" ixy="0" ixz="0" iyz="0"/>
-    </inertial>
-    <!-- Left shaft arm -->
-    <visual>
-      <origin xyz="1.25 0.25 0" rpy="0 0 0"/>
-      <geometry><box size="2.50 0.06 0.06"/></geometry>
-      <material name="iron"/>
-    </visual>
-    <!-- Right shaft arm -->
-    <visual>
-      <origin xyz="1.25 -0.25 0" rpy="0 0 0"/>
-      <geometry><box size="2.50 0.06 0.06"/></geometry>
-      <material name="iron"/>
-    </visual>
-    <!-- Cross brace at pivot end -->
-    <visual>
-      <origin xyz="0.04 0 0" rpy="0 0 0"/>
-      <geometry><box size="0.08 0.56 0.06"/></geometry>
-      <material name="iron"/>
-    </visual>
-    <!-- Cross brace at collar end -->
-    <visual>
-      <origin xyz="2.46 0 0" rpy="0 0 0"/>
-      <geometry><box size="0.08 0.56 0.06"/></geometry>
-      <material name="iron"/>
-    </visual>
-    <collision>
-      <origin xyz="1.25 0 0" rpy="0 0 0"/>
-      <geometry><box size="2.50 0.56 0.08"/></geometry>
-    </collision>
-  </link>
-  <!-- cart_to_shaft_steer: PASSIVE yaw joint — horse turns, pulls cart around. -->
-  <!-- Limits ±35° so horse can turn tightly without jackknifing the cart.     -->
-  <joint name="cart_to_shaft_steer" type="revolute">
-    <parent link="cart_base"/><child link="shaft_steer_link"/>
-    <origin xyz="1.6 0 0.42" rpy="0 0 0"/>
-    <axis xyz="0 0 1"/>
-    <limit lower="-0.61" upper="0.61" effort="200" velocity="2.0"/>
-    <dynamics damping="15.0" friction="3.0"/>
-  </joint>
-  <gazebo reference="shaft_steer_link"><material>Gazebo/Grey</material></gazebo>
-  <!-- ── COLLAR  —  wide yoke that prevents horse rolling L/R ─────────── -->
-  <!-- collar_to_horse is FIXED — no X rotation possible = roll prevented.  -->
-  <!-- Only freedoms are: Z-yaw (cart_to_shaft_steer) + Y-pitch (here).    -->
-  <link name="horse_collar_link">
-    <inertial>
-      <mass value="3.0"/>
-      <origin xyz="0 0 0" rpy="0 0 0"/>
-      <inertia ixx="0.060" iyy="0.010" izz="0.062" ixy="0" ixz="0" iyz="0"/>
-    </inertial>
-    <!-- Wide collar bar spanning both sides of horse body -->
-    <visual>
-      <origin xyz="0 0 0" rpy="0 0 0"/>
-      <geometry><box size="0.06 0.58 0.32"/></geometry>
-      <material name="iron"/>
-    </visual>
-    <!-- Side attachment brackets (show the connection points on horse sides) -->
-    <visual>
-      <origin xyz="0 0.29 0" rpy="0 0 0"/>
-      <geometry><cylinder radius="0.04" length="0.10"/></geometry>
-      <material name="silver"/>
-    </visual>
-    <visual>
-      <origin xyz="0 -0.29 0" rpy="0 0 0"/>
-      <geometry><cylinder radius="0.04" length="0.10"/></geometry>
-      <material name="silver"/>
-    </visual>
-    <!-- NO collision geometry — collar is fixed to horse body, no contact needed -->
-  </link>
-  <!-- shaft_to_collar: PASSIVE pitch joint — horse pitches over bumps. -->
-  <!-- Tight limits ±12° + high damping keeps horse level while gait runs.  -->
-  <joint name="shaft_to_collar" type="revolute">
-    <parent link="shaft_steer_link"/><child link="horse_collar_link"/>
-    <origin xyz="2.50 0 0" rpy="0 0 0"/>
-    <axis xyz="0 1 0"/>
-    <limit lower="-0.21" upper="0.21" effort="500" velocity="2.0"/>
-    <dynamics damping="50.0" friction="10.0"/>
-  </joint>
-  <gazebo reference="horse_collar_link"><material>Gazebo/Grey</material></gazebo>
-  <!-- FIXED: horse body is rigidly attached to collar. Collar is 0.30m behind
-       horse center so arms connect at haunch area (like real carriage harness). -->
-  <joint name="collar_to_horse" type="fixed">
-    <parent link="horse_collar_link"/><child link="base_link"/>
-    <origin xyz="0.30 0 0" rpy="0 0 0"/>
-  </joint>
-  <!-- ═══════════════════════════════════════════════════════
        BASE LINK
   ═══════════════════════════════════════════════════════ -->
@@ -284,17 +68,17 @@
   <link name="base_link">
     <inertial>
-      <mass value="60.0"/>
-      <origin xyz="-0.10 0 0" rpy="0 0 0"/>
-      <inertia ixx="2.234" iyy="7.563" izz="6.772" ixy="0" ixz="0" iyz="0"/>
+      <mass value="160.0"/>
+      <origin xyz="-0.08 0 0" rpy="0 0 0"/>
+      <inertia ixx="7.105" iyy="19.21" izz="20.17" ixy="0" ixz="0" iyz="0"/>
     </inertial>
     <!-- Main body panel -->
     <visual>
       <origin xyz="0 0 0" rpy="0 0 0"/>
-      <geometry><box size="1.10 0.38 0.55"/></geometry>
+      <geometry><box size="1.10 0.55 0.48"/></geometry>
       <material name="body_panel"/>
     </visual>
     <!-- Top saddle plate -->
     <visual>
-      <origin xyz="-0.06 0 0.275" rpy="0 0 0"/>
+      <origin xyz="-0.06 0 0.24" rpy="0 0 0"/>
       <geometry><box size="0.70 0.32 0.04"/></geometry>
       <material name="silver"/>
@@ -302,5 +86,5 @@
     <collision>
       <origin xyz="0 0 0" rpy="0 0 0"/>
-      <geometry><box size="1.10 0.45 0.55"/></geometry>
+      <geometry><box size="1.10 0.62 0.48"/></geometry>
     </collision>
   </link>
@@ -323,5 +107,5 @@
   <joint name="neck_joint" type="fixed">
     <parent link="base_link"/><child link="neck_link"/>
-    <origin xyz="0.52 0 0.265" rpy="0 -0.698 0"/>
+    <origin xyz="0.52 0 0.24" rpy="0 -0.698 0"/>
   </joint>
   <gazebo reference="neck_link"><material>Gazebo/Brown</material></gazebo>
@@ -366,5 +150,5 @@
   <joint name="fl_hip_joint" type="revolute">
     <parent link="base_link"/><child link="fl_hip_link"/>
-    <origin xyz="0.43 0.19 -0.22" rpy="0 0 0"/>
+    <origin xyz="0.43 0.25 -0.20" rpy="0 0 0"/>
     <axis xyz="0 0 1"/>
     <limit lower="-0.35" upper="0.35" effort="200" velocity="2.0"/>
@@ -373,13 +157,13 @@
   <gazebo reference="fl_hip_link"><material>Gazebo/Grey</material></gazebo>
   <link name="fl_thigh_link">
-    <inertial><mass value="5.5"/><origin xyz="0 0 -0.30" rpy="0 0 0"/>
-      <inertia ixx="0.170" iyy="0.170" izz="0.010" ixy="0" ixz="0" iyz="0"/></inertial>
-    <visual><origin xyz="0 0 -0.19" rpy="0 0 0"/>
-      <geometry><box size="0.055 0.055 0.38"/></geometry><material name="orange"/></visual>
+    <inertial><mass value="5.0"/><origin xyz="0 0 -0.14" rpy="0 0 0"/>
+      <inertia ixx="0.034" iyy="0.034" izz="0.003" ixy="0" ixz="0" iyz="0"/></inertial>
+    <visual><origin xyz="0 0 -0.14" rpy="0 0 0"/>
+      <geometry><box size="0.060 0.060 0.28"/></geometry><material name="orange"/></visual>
     <!-- Ballscrew actuator tube -->
-    <visual><origin xyz="0.035 0 -0.19" rpy="0 0 0"/>
-      <geometry><cylinder radius="0.018" length="0.25"/></geometry><material name="silver"/></visual>
-    <collision><origin xyz="0 0 -0.19" rpy="0 0 0">
-      </origin><geometry><box size="0.055 0.055 0.38"/></geometry></collision>
+    <visual><origin xyz="0.035 0 -0.14" rpy="0 0 0"/>
+      <geometry><cylinder radius="0.018" length="0.18"/></geometry><material name="silver"/></visual>
+    <collision><origin xyz="0 0 -0.14" rpy="0 0 0">
+      </origin><geometry><box size="0.060 0.060 0.28"/></geometry></collision>
   </link>
   <joint name="fl_thigh_joint" type="revolute">
@@ -391,14 +175,14 @@
   <gazebo reference="fl_thigh_link"><material>Gazebo/Orange</material></gazebo>
   <link name="fl_shank_link">
-    <inertial><mass value="4.0"/><origin xyz="0 0 -0.30" rpy="0 0 0"/>
-      <inertia ixx="0.122" iyy="0.122" izz="0.004" ixy="0" ixz="0" iyz="0"/></inertial>
-    <visual><origin xyz="0 0 -0.18" rpy="0 0 0">
-      </origin><geometry><box size="0.045 0.045 0.36"/></geometry><material name="dark_grey"/></visual>
-    <collision><origin xyz="0 0 -0.18" rpy="0 0 0">
-      </origin><geometry><box size="0.04 0.04 0.36"/></geometry></collision>
+    <inertial><mass value="4.0"/><origin xyz="0 0 -0.13" rpy="0 0 0"/>
+      <inertia ixx="0.023" iyy="0.023" izz="0.001" ixy="0" ixz="0" iyz="0"/></inertial>
+    <visual><origin xyz="0 0 -0.13" rpy="0 0 0">
+      </origin><geometry><box size="0.045 0.045 0.26"/></geometry><material name="dark_grey"/></visual>
+    <collision><origin xyz="0 0 -0.13" rpy="0 0 0">
+      </origin><geometry><box size="0.04 0.04 0.26"/></geometry></collision>
   </link>
   <joint name="fl_knee_joint" type="revolute">
     <parent link="fl_thigh_link"/><child link="fl_shank_link"/>
-    <origin xyz="0 0 -0.38" rpy="0 0 0"/><axis xyz="0 1 0"/>
+    <origin xyz="0 0 -0.28" rpy="0 0 0"/><axis xyz="0 1 0"/>
     <limit lower="-1.8" upper="2.0" effort="800" velocity="5.0"/>
     <dynamics damping="3.5" friction="0.3"/>
@@ -407,14 +191,14 @@
   <!-- Cannon bone (metatarsal/metacarpal): pantograph-kept near vertical -->
   <link name="fl_cannon_link">
-    <inertial><mass value="1.0"/><origin xyz="0 0 -0.125" rpy="0 0 0"/>
-      <inertia ixx="0.0053" iyy="0.0053" izz="0.0001" ixy="0" ixz="0" iyz="0"/></inertial>
-    <visual><origin xyz="0 0 -0.125" rpy="0 0 0"/>
-      <geometry><cylinder radius="0.015" length="0.25"/></geometry><material name="dark_grey"/></visual>
-    <collision><origin xyz="0 0 -0.125" rpy="0 0 0"/>
-      <geometry><cylinder radius="0.012" length="0.25"/></geometry></collision>
+    <inertial><mass value="1.0"/><origin xyz="0 0 -0.08" rpy="0 0 0"/>
+      <inertia ixx="0.0022" iyy="0.0022" izz="0.0001" ixy="0" ixz="0" iyz="0"/></inertial>
+    <visual><origin xyz="0 0 -0.08" rpy="0 0 0"/>
+      <geometry><cylinder radius="0.015" length="0.16"/></geometry><material name="dark_grey"/></visual>
+    <collision><origin xyz="0 0 -0.08" rpy="0 0 0"/>
+      <geometry><cylinder radius="0.012" length="0.16"/></geometry></collision>
   </link>
   <joint name="fl_cannon_joint" type="revolute">
     <parent link="fl_shank_link"/><child link="fl_cannon_link"/>
-    <origin xyz="0 0 -0.36" rpy="0 0 0"/><axis xyz="0 1 0"/>
+    <origin xyz="0 0 -0.26" rpy="0 0 0"/><axis xyz="0 1 0"/>
     <limit lower="-2.0" upper="2.0" effort="100" velocity="6.0"/>
     <dynamics damping="1.0" friction="0.1"/>
@@ -425,11 +209,11 @@
       <inertia ixx="0.00026" iyy="0.00026" izz="0.00026" ixy="0" ixz="0" iyz="0"/></inertial>
     <visual><origin xyz="0 0 0" rpy="0 0 0"/>
-      <geometry><sphere radius="0.05"/></geometry><material name="black"/></visual>
+      <geometry><sphere radius="0.04"/></geometry><material name="black"/></visual>
     <collision><origin xyz="0 0 0" rpy="0 0 0"/>
-      <geometry><sphere radius="0.05"/></geometry></collision>
+      <geometry><sphere radius="0.04"/></geometry></collision>
   </link>
   <joint name="fl_foot_joint" type="fixed">
     <parent link="fl_cannon_link"/><child link="fl_foot_link"/>
-    <origin xyz="0 0 -0.25" rpy="0 0 0"/>
+    <origin xyz="0 0 -0.16" rpy="0 0 0"/>
   </joint>
   <gazebo reference="fl_foot_link">
@@ -449,5 +233,5 @@
   <joint name="fr_hip_joint" type="revolute">
     <parent link="base_link"/><child link="fr_hip_link"/>
-    <origin xyz="0.43 -0.19 -0.22" rpy="0 0 0"/>
+    <origin xyz="0.43 -0.25 -0.20" rpy="0 0 0"/>
     <axis xyz="0 0 1"/>
     <limit lower="-0.35" upper="0.35" effort="200" velocity="2.0"/>
@@ -456,13 +240,13 @@
   <gazebo reference="fr_hip_link"><material>Gazebo/Grey</material></gazebo>
   <link name="fr_thigh_link">
-    <inertial><mass value="5.5"/><origin xyz="0 0 -0.30" rpy="0 0 0"/>
-      <inertia ixx="0.170" iyy="0.170" izz="0.010" ixy="0" ixz="0" iyz="0"/></inertial>
-    <visual><origin xyz="0 0 -0.19" rpy="0 0 0">
-      </origin><geometry><box size="0.055 0.055 0.38"/></geometry><material name="orange"/></visual>
+    <inertial><mass value="5.0"/><origin xyz="0 0 -0.14" rpy="0 0 0"/>
+      <inertia ixx="0.034" iyy="0.034" izz="0.003" ixy="0" ixz="0" iyz="0"/></inertial>
+    <visual><origin xyz="0 0 -0.14" rpy="0 0 0">
+      </origin><geometry><box size="0.060 0.060 0.28"/></geometry><material name="orange"/></visual>
     <!-- Ballscrew actuator tube -->
-    <visual><origin xyz="0.035 0 -0.19" rpy="0 0 0"/>
-      <geometry><cylinder radius="0.018" length="0.25"/></geometry><material name="silver"/></visual>
-    <collision><origin xyz="0 0 -0.19" rpy="0 0 0">
-      </origin><geometry><box size="0.055 0.055 0.38"/></geometry></collision>
+    <visual><origin xyz="0.035 0 -0.14" rpy="0 0 0"/>
+      <geometry><cylinder radius="0.018" length="0.18"/></geometry><material name="silver"/></visual>
+    <collision><origin xyz="0 0 -0.14" rpy="0 0 0">
+      </origin><geometry><box size="0.060 0.060 0.28"/></geometry></collision>
   </link>
   <joint name="fr_thigh_joint" type="revolute">
@@ -474,14 +258,14 @@
   <gazebo reference="fr_thigh_link"><material>Gazebo/Orange</material></gazebo>
   <link name="fr_shank_link">
-    <inertial><mass value="4.0"/><origin xyz="0 0 -0.30" rpy="0 0 0"/>
-      <inertia ixx="0.122" iyy="0.122" izz="0.004" ixy="0" ixz="0" iyz="0"/></inertial>
-    <visual><origin xyz="0 0 -0.18" rpy="0 0 0">
-      </origin><geometry><box size="0.045 0.045 0.36"/></geometry><material name="dark_grey"/></visual>
-    <collision><origin xyz="0 0 -0.18" rpy="0 0 0">
-      </origin><geometry><box size="0.04 0.04 0.36"/></geometry></collision>
+    <inertial><mass value="4.0"/><origin xyz="0 0 -0.13" rpy="0 0 0"/>
+      <inertia ixx="0.023" iyy="0.023" izz="0.001" ixy="0" ixz="0" iyz="0"/></inertial>
+    <visual><origin xyz="0 0 -0.13" rpy="0 0 0">
+      </origin><geometry><box size="0.045 0.045 0.26"/></geometry><material name="dark_grey"/></visual>
+    <collision><origin xyz="0 0 -0.13" rpy="0 0 0">
+      </origin><geometry><box size="0.04 0.04 0.26"/></geometry></collision>
   </link>
   <joint name="fr_knee_joint" type="revolute">
     <parent link="fr_thigh_link"/><child link="fr_shank_link"/>
-    <origin xyz="0 0 -0.38" rpy="0 0 0"/><axis xyz="0 1 0"/>
+    <origin xyz="0 0 -0.28" rpy="0 0 0"/><axis xyz="0 1 0"/>
     <limit lower="-1.8" upper="2.0" effort="800" velocity="5.0"/>
     <dynamics damping="3.5" friction="0.3"/>
@@ -490,14 +274,14 @@
   <!-- Cannon bone (metatarsal/metacarpal): pantograph-kept near vertical -->
   <link name="fr_cannon_link">
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