Commit message: Fix forward-falling: deep crouch stance, realistic 100kg mass, bounded strides
Root cause: ANKLE_HEIGHT (0.366m) was nearly equal to L1+L2 (0.38m), leaving
only ~0.10m horizontal reach. MAX_STEP=0.45m forced constant IK clamping →
legs fully extended, zero compliance, robot faceplanted immediately.

Changes:
- Neutral stance: thigh 0.25→0.55, knee -0.55→-1.10 (deeper crouch)
  ANKLE_HEIGHT: 0.366→0.324m, horizontal reach: 0.10→0.179m
- MAX_STEP: 0.45→0.14m (within actual leg reach at all times)
- Body mass: 400kg→100kg (motors 48kg + frame 24kg + electronics 8kg +
  decoration 35kg + legs 5kg). Inertia recalculated accordingly.
- Body inertia: Ixx 17.33→4.33, Iyy 70.67→17.67, Izz 77.33→19.33 kg·m²
- WALK: period 2.2→1.5s, swing_frac 0.22→0.30, step_height 0.16→0.10m,
  min_stride 0.22→0.04m, speed 0.8→0.30 m/s
- TROT: swing_frac 0.35→0.40, step_height 0.22→0.11m, min_stride 0.28→0.05m,
  speed 1.8→0.65 m/s, period 0.9→0.8s
- TROT_THRESHOLD: 1.5→0.48 (between new WALK=0.30 and TROT=0.65)
- spawn_z: 0.77→0.72m (FK: 0.464 + 0.16 + 0.10 = 0.724m)
- Initial joint values updated in URDF to match new neutral stance
- Teleop WALK/TROT speeds updated to match blendspace constants

Co-authored-by: Copilot <223556219+Copilot@users.noreply.github.com>

File: ros2_ws/src/robotic_horse_description/urdf/robotic_horse.urdf.xacro (robot description, xacro)
@@ -64,10 +64,11 @@
        BASE LINK
   ═══════════════════════════════════════════════════════ -->
-  <!-- Highland Cow body: 400kg, 1.40x0.60x0.40m. Low CoM for stability. -->
+  <!-- Body mass ~100 kg: motors(48)+frame(24)+electronics(8)+decoration(35)+legs(5).
+       Inertia (100 kg, 1.40x0.60x0.40 m box): Ixx=4.33, Iyy=17.67, Izz=19.33 kg·m² -->
   <link name="base_link">
     <inertial>
-      <mass value="400.0"/>
+      <mass value="100.0"/>
       <origin xyz="0 0 0" rpy="0 0 0"/>
-      <inertia ixx="17.33" iyy="70.67" izz="77.33" ixy="0" ixz="0" iyz="0"/>
+      <inertia ixx="4.33" iyy="17.67" izz="19.33" ixy="0" ixz="0" iyz="0"/>
     </inertial>
     <!-- Main body panel -->
@@ -622,5 +623,5 @@
       </command_interface>
       <state_interface name="position">
-        <param name="initial_value">0.25</param>
+        <param name="initial_value">0.55</param>
       </state_interface>
       <state_interface name="velocity"/>
@@ -632,5 +633,5 @@
       </command_interface>
       <state_interface name="position">
-        <param name="initial_value">-0.55</param>
+        <param name="initial_value">-1.10</param>
       </state_interface>
       <state_interface name="velocity"/>
@@ -642,5 +643,5 @@
       </command_interface>
       <state_interface name="position">
-        <param name="initial_value">0.38</param>
+        <param name="initial_value">0.63</param>
       </state_interface>
       <state_interface name="velocity"/>
@@ -663,5 +664,5 @@
       </command_interface>
       <state_interface name="position">
-        <param name="initial_value">0.25</param>
+        <param name="initial_value">0.55</param>
       </state_interface>
       <state_interface name="velocity"/>
@@ -673,5 +674,5 @@
       </command_interface>
       <state_interface name="position">
-        <param name="initial_value">-0.55</param>
+        <param name="initial_value">-1.10</param>
       </state_interface>
       <state_interface name="velocity"/>
@@ -683,5 +684,5 @@
       </command_interface>
       <state_interface name="position">
-        <param name="initial_value">0.38</param>
+        <param name="initial_value">0.63</param>
       </state_interface>
       <state_interface name="velocity"/>
@@ -704,5 +705,5 @@
       </command_interface>
       <state_interface name="position">
-        <param name="initial_value">-0.25</param>
+        <param name="initial_value">-0.55</param>
       </state_interface>
       <state_interface name="velocity"/>
@@ -714,5 +715,5 @@
       </command_interface>
       <state_interface name="position">
-        <param name="initial_value">0.55</param>
+        <param name="initial_value">1.10</param>
       </state_interface>
       <state_interface name="velocity"/>
@@ -724,5 +725,5 @@
       </command_interface>
       <state_interface name="position">
-        <param name="initial_value">-0.22</param>
+        <param name="initial_value">-0.47</param>
       </state_interface>
       <state_interface name="velocity"/>
@@ -745,5 +746,5 @@
       </command_interface>
       <state_interface name="position">
-        <param name="initial_value">-0.25</param>
+        <param name="initial_value">-0.55</param>
       </state_interface>
       <state_interface name="velocity"/>
@@ -755,5 +756,5 @@
       </command_interface>
       <state_interface name="position">
-        <param name="initial_value">0.55</param>
+        <param name="initial_value">1.10</param>
       </state_interface>
       <state_interface name="velocity"/>
@@ -765,5 +766,5 @@
       </command_interface>
       <state_interface name="position">
-        <param name="initial_value">-0.22</param>
+        <param name="initial_value">-0.47</param>
       </state_interface>
       <state_interface name="velocity"/>
