Commit message: Redesign carriage: vis-à-vis body, U-shaped shaft, driver, fix spawn height
- Spawn height: 0.72→1.08m (feet on ground at neutral stance)
- Carriage: vis-à-vis style with facing bench seats, curved panels, lanterns
- Shaft: U-shaped fork 2.35m, continuous yaw (infinite turn angle)
- Hitch: 50cm fwd + 37cm above front wheel center
- Wheels: ⌀85cm front, ⌀105cm rear, 145cm track, 205cm wheelbase
- Carriage body: 250×110×110cm sitting ~60cm off ground
- Driver: 85kg figure on front bench
- Updated build plan with accurate carriage mass budget

Co-authored-by: Copilot <223556219+Copilot@users.noreply.github.com>

File: ros2_ws/src/robotic_horse_description/urdf/robotic_horse.urdf.xacro (robot description, xacro)
@@ -36,4 +36,5 @@
   <material name="wood">       <color rgba="0.55 0.35 0.15 1"/></material>
   <material name="iron">       <color rgba="0.28 0.28 0.28 1"/></material>
+  <material name="red_velvet"> <color rgba="0.60 0.05 0.05 1"/></material>
   <!-- ═══════════════════════════════════════════════════════
        IMU SENSOR  — provides body orientation for self-balance
@@ -566,92 +567,175 @@
   </gazebo>
   <!-- ═══════════════════════════════════════════════════════
-       CARRIAGE — hitched behind the horse
-       Total carriage mass ≈ 64 kg (+ 30 kg payload)
-       Front wheels ⌀ 85 cm, Rear wheels ⌀ 105 cm
-       Track width 205 cm, Wheelbase 140 cm
+       CARRIAGE — vis-à-vis style, hitched to bovine robot
+       Real measurements from owner's carriage:
+         Front wheels ⌀ 85 cm,  Rear wheels ⌀ 105 cm
+         Wheelbase 205 cm,  Track 145 cm
+         Shaft 235 cm long, U-shaped, 85→70 cm wide
+         Hitch: 50 cm fwd + 37 cm above front wheel center
+         Body: 250 × 110 × 110 cm, ~60 cm off ground
+         Driver: ~85 kg on front bench
+       Total carriage mass ≈ 105 kg + 85 kg driver = 190 kg
   ═══════════════════════════════════════════════════════ -->
-  <!-- Hitch yaw joint (base_link → hitch_link) -->
-  <joint name="horse_hitch_joint" type="revolute">
-    <parent link="base_link"/><child link="hitch_link"/>
-    <origin xyz="-0.70 0 -0.10" rpy="0 0 0"/>
+  <!-- Shaft yaw joint (base_link → shaft) — continuous rotation (infinite turn angle) -->
+  <joint name="shaft_yaw_joint" type="continuous">
+    <parent link="base_link"/><child link="shaft_link"/>
+    <origin xyz="0.0 0 -0.30" rpy="0 0 0"/>
+    <axis xyz="0 0 1"/>
+    <dynamics damping="5.0" friction="0.5"/>
+  </joint>
+  <!-- Shaft — U-shaped wooden fork, 2.35m long -->
+  <link name="shaft_link">
+    <inertial><mass value="15.0"/><origin xyz="-1.175 0 0" rpy="0 0 0"/>
+      <inertia ixx="0.10" iyy="6.93" izz="6.95" ixy="0" ixz="0" iyz="0"/></inertial>
+    <!-- Left shaft bar -->
+    <visual><origin xyz="-1.175 0.39 0" rpy="0 0 0"/>
+      <geometry><box size="2.35 0.05 0.05"/></geometry><material name="wood"/></visual>
+    <collision><origin xyz="-1.175 0.39 0" rpy="0 0 0"/>
+      <geometry><box size="2.35 0.05 0.05"/></geometry></collision>
+    <!-- Right shaft bar -->
+    <visual><origin xyz="-1.175 -0.39 0" rpy="0 0 0"/>
+      <geometry><box size="2.35 0.05 0.05"/></geometry><material name="wood"/></visual>
+    <collision><origin xyz="-1.175 -0.39 0" rpy="0 0 0"/>
+      <geometry><box size="2.35 0.05 0.05"/></geometry></collision>
+    <!-- Cross piece at carriage end -->
+    <visual><origin xyz="-2.30 0 0" rpy="0 0 0"/>
+      <geometry><box size="0.05 0.70 0.05"/></geometry><material name="wood"/></visual>
+    <collision><origin xyz="-2.30 0 0" rpy="0 0 0"/>
+      <geometry><box size="0.05 0.70 0.05"/></geometry></collision>
+  </link>
+  <!-- Shaft pitch joint — allows carriage to pitch on uneven ground -->
+  <joint name="shaft_pitch_joint" type="revolute">
+    <parent link="shaft_link"/><child link="cart_hitch_link"/>
+    <origin xyz="-2.35 0 0.015" rpy="0 0 0"/>
+    <axis xyz="0 1 0"/>
+    <limit lower="-0.20" upper="0.20" effort="0" velocity="2.0"/>
+    <dynamics damping="15.0" friction="0.5"/>
+  </joint>
+  <!-- Hitch pin (small connector) -->
+  <link name="cart_hitch_link">
+    <inertial><mass value="2.0"/><origin xyz="0 0 0" rpy="0 0 0"/>
+      <inertia ixx="0.002" iyy="0.002" izz="0.001" ixy="0" ixz="0" iyz="0"/></inertial>
+    <visual><origin xyz="0 0 0" rpy="0 0 0"/>
+      <geometry><cylinder radius="0.04" length="0.12"/></geometry><material name="iron"/></visual>
+    <collision><origin xyz="0 0 0" rpy="0 0 0"/>
+      <geometry><cylinder radius="0.04" length="0.12"/></geometry></collision>
+  </link>
+  <!-- Cart body (fixed to hitch) — vis-à-vis carriage -->
+  <joint name="cart_body_joint" type="fixed">
+    <parent link="cart_hitch_link"/><child link="cart_body_link"/>
+    <origin xyz="0 0 0" rpy="0 0 0"/>
+  </joint>
+  <!-- Cart body — 250×110×110 cm wooden carriage body
+       Body center at (-1.525, 0, +0.355) from hitch
+       Driver (85 kg) seated on front bench at (-0.90, 0, +0.80) from hitch -->
+  <link name="cart_body_link">
+    <!-- Combined inertia: carriage structure 55 kg + driver 85 kg = 140 kg
+         Approximate as box 2.50×1.10×1.10 at combined COM -->
+    <inertial><mass value="140.0"/><origin xyz="-1.40 0 0.42" rpy="0 0 0"/>
+      <inertia ixx="25.0" iyy="95.0" izz="85.0" ixy="0" ixz="0" iyz="0"/></inertial>
+    <!-- Main body floor/deck -->
+    <visual><origin xyz="-1.525 0 0.16" rpy="0 0 0"/>
+      <geometry><box size="2.50 1.10 0.06"/></geometry><material name="wood"/></visual>
+    <collision><origin xyz="-1.525 0 0.16" rpy="0 0 0"/>
+      <geometry><box size="2.50 1.10 0.06"/></geometry></collision>
+    <!-- Left side panel (curved in real life — approximated with box) -->
+    <visual><origin xyz="-1.525 0.52 0.55" rpy="0 0 0"/>
+      <geometry><box size="2.20 0.06 0.72"/></geometry><material name="wood"/></visual>
+    <collision><origin xyz="-1.525 0.52 0.55" rpy="0 0 0"/>
+      <geometry><box size="2.20 0.06 0.72"/></geometry></collision>
+    <!-- Right side panel -->
+    <visual><origin xyz="-1.525 -0.52 0.55" rpy="0 0 0"/>
+      <geometry><box size="2.20 0.06 0.72"/></geometry><material name="wood"/></visual>
+    <collision><origin xyz="-1.525 -0.52 0.55" rpy="0 0 0"/>
+      <geometry><box size="2.20 0.06 0.72"/></geometry></collision>
+    <!-- Front panel (driver side, with kick board — black leather) -->
+    <visual><origin xyz="-0.45 0 0.50" rpy="0 0 0"/>
+      <geometry><box size="0.06 1.00 0.62"/></geometry><material name="dark_grey"/></visual>
+    <!-- Rear panel -->
+    <visual><origin xyz="-2.60 0 0.50" rpy="0 0 0"/>
+      <geometry><box size="0.06 1.00 0.62"/></geometry><material name="dark_grey"/></visual>
+    <!-- Center divider panel -->
+    <visual><origin xyz="-1.525 0 0.50" rpy="0 0 0"/>
+      <geometry><box size="0.06 0.90 0.50"/></geometry><material name="dark_grey"/></visual>
+    <!-- Front bench seat (driver sits here, facing backward) -->
+    <visual><origin xyz="-0.80 0 0.46" rpy="0 0 0"/>
+      <geometry><box size="0.45 0.90 0.08"/></geometry><material name="red_velvet"/></visual>
+    <!-- Front seat backrest -->
+    <visual><origin xyz="-0.58 0 0.68" rpy="0 0 0"/>
+      <geometry><box size="0.06 0.90 0.36"/></geometry><material name="wood"/></visual>
+    <!-- Rear bench seat (passengers, facing forward) -->
+    <visual><origin xyz="-2.25 0 0.46" rpy="0 0 0"/>
+      <geometry><box size="0.45 0.90 0.08"/></geometry><material name="red_velvet"/></visual>
+    <!-- Rear seat backrest -->
+    <visual><origin xyz="-2.47 0 0.68" rpy="0 0 0"/>
+      <geometry><box size="0.06 0.90 0.36"/></geometry><material name="wood"/></visual>
+    <!-- Driver figure (85 kg, seated on front bench) -->
+    <!-- Torso -->
+    <visual><origin xyz="-0.80 0 0.82" rpy="0 0 0"/>
+      <geometry><box size="0.30 0.40 0.55"/></geometry><material name="dark_grey"/></visual>
+    <!-- Head -->
+    <visual><origin xyz="-0.80 0 1.17" rpy="0 0 0"/>
+      <geometry><sphere radius="0.12"/></geometry><material name="light_grey"/></visual>
+    <!-- Left mudguard / fender (over rear wheels) -->
+    <visual><origin xyz="-2.35 0.58 0.10" rpy="0 0 0"/>
+      <geometry><box size="0.70 0.12 0.06"/></geometry><material name="wood"/></visual>
+    <!-- Right mudguard -->
+    <visual><origin xyz="-2.35 -0.58 0.10" rpy="0 0 0"/>
+      <geometry><box size="0.70 0.12 0.06"/></geometry><material name="wood"/></visual>
+    <!-- Iron underframe / chassis rail (left) -->
+    <visual><origin xyz="-1.525 0.40 -0.05" rpy="0 0 0"/>
+      <geometry><box size="2.60 0.04 0.04"/></geometry><material name="iron"/></visual>
+    <!-- Iron underframe / chassis rail (right) -->
+    <visual><origin xyz="-1.525 -0.40 -0.05" rpy="0 0 0"/>
+      <geometry><box size="2.60 0.04 0.04"/></geometry><material name="iron"/></visual>
+    <!-- Left carriage lamp bracket -->
+    <visual><origin xyz="-0.35 0.50 0.95" rpy="0 0 0"/>
+      <geometry><cylinder radius="0.02" length="0.25"/></geometry><material name="iron"/></visual>
+    <!-- Left lamp housing -->
+    <visual><origin xyz="-0.35 0.54 1.10" rpy="0 0 0"/>
+      <geometry><box size="0.10 0.10 0.15"/></geometry><material name="iron"/></visual>
+    <!-- Right carriage lamp bracket -->
+    <visual><origin xyz="-0.35 -0.50 0.95" rpy="0 0 0"/>
+      <geometry><cylinder radius="0.02" length="0.25"/></geometry><material name="iron"/></visual>
+    <!-- Right lamp housing -->
+    <visual><origin xyz="-0.35 -0.54 1.10" rpy="0 0 0"/>
+      <geometry><box size="0.10 0.10 0.15"/></geometry><material name="iron"/></visual>
+    <!-- Folding hood frame (rear, collapsed) -->
+    <visual><origin xyz="-2.55 0 1.00" rpy="0 0 0"/>
+      <geometry><box size="0.08 0.95 0.15"/></geometry><material name="wood"/></visual>
+  </link>
+  <!-- ── Front axle (steering) ── -->
+  <joint name="front_axle_joint" type="revolute">
+    <parent link="cart_body_link"/><child link="front_axle_link"/>
+    <origin xyz="-0.50 0 -0.37" rpy="0 0 0"/>
     <axis xyz="0 0 1"/>
     <limit lower="-0.5" upper="0.5" effort="0" velocity="2.0"/>
-    <dynamics damping="5.0" friction="0.1"/>
-  </joint>
-  <link name="hitch_link">
-    <inertial><mass value="1.0"/><origin xyz="0 0 0" rpy="0 0 0"/>
-      <inertia ixx="0.001" iyy="0.001" izz="0.0005" ixy="0" ixz="0" iyz="0"/></inertial>
+    <dynamics damping="20.0" friction="0.5"/>
+  </joint>
+  <link name="front_axle_link">
+    <inertial><mass value="6.0"/><origin xyz="0 0 0" rpy="0 0 0"/>
+      <inertia ixx="0.53" iyy="0.003" izz="0.53" ixy="0" ixz="0" iyz="0"/></inertial>
     <visual><origin xyz="0 0 0" rpy="0 0 0"/>
-      <geometry><cylinder radius="0.03" length="0.10"/></geometry><material name="iron"/></visual>
+      <geometry><box size="0.06 1.40 0.06"/></geometry><material name="iron"/></visual>
     <collision><origin xyz="0 0 0" rpy="0 0 0"/>
-      <geometry><cylinder radius="0.03" length="0.10"/></geometry></collision>
-  </link>
-  <!-- Hitch pitch joint (hitch_link → tongue_link) -->
-  <joint name="hitch_pitch_joint" type="revolute">
-    <parent link="hitch_link"/><child link="tongue_link"/>
-    <origin xyz="0 0 0" rpy="0 0 0"/>
-    <axis xyz="0 1 0"/>
-    <limit lower="-0.3" upper="0.3" effort="0" velocity="2.0"/>
-    <dynamics damping="10.0" friction="0.1"/>
-  </joint>
-  <link name="tongue_link">
-    <inertial><mass value="5.0"/><origin xyz="-0.40 0 0" rpy="0 0 0"/>
-      <inertia ixx="0.001" iyy="0.027" izz="0.027" ixy="0" ixz="0" iyz="0"/></inertial>
-    <visual><origin xyz="-0.40 0 0" rpy="0 0 0"/>
-      <geometry><box size="0.80 0.06 0.04"/></geometry><material name="wood"/></visual>
-    <collision><origin xyz="-0.40 0 0" rpy="0 0 0"/>
-      <geometry><box size="0.80 0.06 0.04"/></geometry></collision>
-  </link>
-  <!-- Cart base (tongue_link → cart_base_link) -->
-  <joint name="cart_base_joint" type="fixed">
-    <parent link="tongue_link"/><child link="cart_base_link"/>
-    <origin xyz="-0.80 0 0.10" rpy="0 0 0"/>
-  </joint>
-  <link name="cart_base_link">
-    <inertial><mass value="34.0"/><origin xyz="-0.60 0 0" rpy="0 0 0"/>
-      <inertia ixx="1.82" iyy="4.08" izz="5.90" ixy="0" ixz="0" iyz="0"/></inertial>
-    <visual><origin xyz="-0.60 0 0" rpy="0 0 0"/>
-      <geometry><box size="1.20 0.80 0.05"/></geometry><material name="wood"/></visual>
-    <collision><origin xyz="-0.60 0 0" rpy="0 0 0"/>
-      <geometry><box size="1.20 0.80 0.05"/></geometry></collision>
-    <!-- Bench / seat -->
-    <visual><origin xyz="-0.80 0 0.175" rpy="0 0 0"/>
-      <geometry><box size="0.40 0.70 0.30"/></geometry><material name="wood"/></visual>
-    <collision><origin xyz="-0.80 0 0.175" rpy="0 0 0"/>
-      <geometry><box size="0.40 0.70 0.30"/></geometry></collision>
-  </link>
-  <!-- Front axle (steering) -->
-  <joint name="front_axle_joint" type="revolute">
-    <parent link="cart_base_link"/><child link="front_axle_link"/>
-    <origin xyz="-0.10 0 -0.05" rpy="0 0 0"/>
-    <axis xyz="0 0 1"/>
-    <limit lower="-0.4" upper="0.4" effort="0" velocity="2.0"/>
-    <dynamics damping="20.0" friction="0.1"/>
-  </joint>
-  <link name="front_axle_link">
-    <inertial><mass value="3.0"/><origin xyz="0 0 0" rpy="0 0 0"/>
-      <inertia ixx="0.423" iyy="0.001" izz="0.423" ixy="0" ixz="0" iyz="0"/></inertial>
+      <geometry><box size="0.06 1.40 0.06"/></geometry></collision>
+  </link>
+  <!-- ── Rear axle (fixed) ── -->
+  <joint name="rear_axle_joint" type="fixed">
+    <parent link="cart_body_link"/><child link="rear_axle_link"/>
+    <origin xyz="-2.55 0 -0.27" rpy="0 0 0"/>
+  </joint>
+  <link name="rear_axle_link">
+    <inertial><mass value="6.0"/><origin xyz="0 0 0" rpy="0 0 0"/>
+      <inertia ixx="0.53" iyy="0.003" izz="0.53" ixy="0" ixz="0" iyz="0"/></inertial>
     <visual><origin xyz="0 0 0" rpy="0 0 0"/>
-      <geometry><box size="0.06 2.00 0.06"/></geometry><material name="iron"/></visual>
+      <geometry><box size="0.06 1.40 0.06"/></geometry><material name="iron"/></visual>
     <collision><origin xyz="0 0 0" rpy="0 0 0"/>
-      <geometry><box size="0.06 2.00 0.06"/></geometry></collision>
-  </link>
-  <!-- Rear axle (fixed) -->
-  <joint name="rear_axle_joint" type="fixed">
-    <parent link="cart_base_link"/><child link="rear_axle_link"/>
-    <origin xyz="-0.90 0 -0.05" rpy="0 0 0"/>
-  </joint>
-  <link name="rear_axle_link">
-    <inertial><mass value="3.0"/><origin xyz="0 0 0" rpy="0 0 0"/>
-      <inertia ixx="0.423" iyy="0.001" izz="0.423" ixy="0" ixz="0" iyz="0"/></inertial>
-    <visual><origin xyz="0 0 0" rpy="0 0 0"/>
-      <geometry><box size="0.06 2.00 0.06"/></geometry><material name="iron"/></visual>
-    <collision><origin xyz="0 0 0" rpy="0 0 0"/>
-      <geometry><box size="0.06 2.00 0.06"/></geometry></collision>
-  </link>
-  <!-- ── Front-Left Wheel ── -->
+      <geometry><box size="0.06 1.40 0.06"/></geometry></collision>
+  </link>
+  <!-- ── Front-Left Wheel (⌀85cm) ── -->
   <joint name="cart_fl_wheel_joint" type="continuous">
     <parent link="front_axle_link"/><child link="cart_fl_wheel_link"/>
-    <origin xyz="0 1.025 0" rpy="0 0 0"/>
+    <origin xyz="0 0.725 0" rpy="0 0 0"/>
     <axis xyz="0 1 0"/>
     <dynamics damping="0.5" friction="0.1"/>
@@ -659,14 +743,17 @@
   <link name="cart_fl_wheel_link">
     <inertial><mass value="4.0"/><origin xyz="0 0 0" rpy="0 0 0"/>
-      <inertia ixx="0.182" iyy="0.361" izz="0.182" ixy="0" ixz="0" iyz="0"/></inertial>
+      <inertia ixx="0.091" iyy="0.181" izz="0.091" ixy="0" ixz="0" iyz="0"/></inertial>
     <visual><origin xyz="0 0 0" rpy="1.5708 0 0"/>
-      <geometry><cylinder radius="0.425" length="0.06"/></geometry><material name="dark_grey"/></visual>
+      <geometry><cylinder radius="0.425" length="0.05"/></geometry><material name="wood"/></visual>
     <collision><origin xyz="0 0 0" rpy="1.5708 0 0"/>
-      <geometry><cylinder radius="0.425" length="0.06"/></geometry></collision>
-  </link>
-  <!-- ── Front-Right Wheel ── -->
+      <geometry><cylinder radius="0.425" length="0.05"/></geometry></collision>
+    <!-- Wheel hub -->
+    <visual><origin xyz="0 0.03 0" rpy="1.5708 0 0"/>
+      <geometry><cylinder radius="0.06" length="0.08"/></geometry><material name="iron"/></visual>
+  </link>
+  <!-- ── Front-Right Wheel (⌀85cm) ── -->
   <joint name="cart_fr_wheel_joint" type="continuous">
     <parent link="front_axle_link"/><child link="cart_fr_wheel_link"/>
-    <origin xyz="0 -1.025 0" rpy="0 0 0"/>
+    <origin xyz="0 -0.725 0" rpy="0 0 0"/>
     <axis xyz="0 1 0"/>
     <dynamics damping="0.5" friction="0.1"/>
@@ -674,14 +761,16 @@
   <link name="cart_fr_wheel_link">
     <inertial><mass value="4.0"/><origin xyz="0 0 0" rpy="0 0 0"/>
-      <inertia ixx="0.182" iyy="0.361" izz="0.182" ixy="0" ixz="0" iyz="0"/></inertial>
+      <inertia ixx="0.091" iyy="0.181" izz="0.091" ixy="0" ixz="0" iyz="0"/></inertial>
     <visual><origin xyz="0 0 0" rpy="1.5708 0 0"/>
-      <geometry><cylinder radius="0.425" length="0.06"/></geometry><material name="dark_grey"/></visual>
+      <geometry><cylinder radius="0.425" length="0.05"/></geometry><material name="wood"/></visual>
     <collision><origin xyz="0 0 0" rpy="1.5708 0 0"/>
-      <geometry><cylinder radius="0.425" length="0.06"/></geometry></collision>
-  </link>
-  <!-- ── Rear-Left Wheel ── -->
+      <geometry><cylinder radius="0.425" length="0.05"/></geometry></collision>
+    <visual><origin xyz="0 -0.03 0" rpy="1.5708 0 0"/>
+      <geometry><cylinder radius="0.06" length="0.08"/></geometry><material name="iron"/></visual>
+  </link>
+  <!-- ── Rear-Left Wheel (⌀105cm) ── -->
   <joint name="cart_rl_wheel_joint" type="continuous">
     <parent link="rear_axle_link"/><child link="cart_rl_wheel_link"/>
-    <origin xyz="0 1.025 0" rpy="0 0 0"/>
+    <origin xyz="0 0.725 0" rpy="0 0 0"/>
     <axis xyz="0 1 0"/>
     <dynamics damping="0.5" friction="0.1"/>
@@ -689,14 +778,16 @@
   <link name="cart_rl_wheel_link">
     <inertial><mass value="5.0"/><origin xyz="0 0 0" rpy="0 0 0"/>
-      <inertia ixx="0.347" iyy="0.689" izz="0.347" ixy="0" ixz="0" iyz="0"/></inertial>
+      <inertia ixx="0.174" iyy="0.345" izz="0.174" ixy="0" ixz="0" iyz="0"/></inertial>
     <visual><origin xyz="0 0 0" rpy="1.5708 0 0"/>
-      <geometry><cylinder radius="0.525" length="0.08"/></geometry><material name="dark_grey"/></visual>
+      <geometry><cylinder radius="0.525" length="0.06"/></geometry><material name="wood"/></visual>
     <collision><origin xyz="0 0 0" rpy="1.5708 0 0"/>
-      <geometry><cylinder radius="0.525" length="0.08"/></geometry></collision>
-  </link>
-  <!-- ── Rear-Right Wheel ── -->
+      <geometry><cylinder radius="0.525" length="0.06"/></geometry></collision>
+    <visual><origin xyz="0 0.04 0" rpy="1.5708 0 0"/>
+      <geometry><cylinder radius="0.06" length="0.10"/></geometry><material name="iron"/></visual>
+  </link>
+  <!-- ── Rear-Right Wheel (⌀105cm) ── -->
   <joint name="cart_rr_wheel_joint" type="continuous">
     <parent link="rear_axle_link"/><child link="cart_rr_wheel_link"/>
-    <origin xyz="0 -1.025 0" rpy="0 0 0"/>
+    <origin xyz="0 -0.725 0" rpy="0 0 0"/>
     <axis xyz="0 1 0"/>
     <dynamics damping="0.5" friction="0.1"/>
@@ -704,17 +795,20 @@
   <link name="cart_rr_wheel_link">
     <inertial><mass value="5.0"/><origin xyz="0 0 0" rpy="0 0 0"/>
-      <inertia ixx="0.347" iyy="0.689" izz="0.347" ixy="0" ixz="0" iyz="0"/></inertial>
+      <inertia ixx="0.174" iyy="0.345" izz="0.174" ixy="0" ixz="0" iyz="0"/></inertial>
     <visual><origin xyz="0 0 0" rpy="1.5708 0 0"/>
-      <geometry><cylinder radius="0.525" length="0.08"/></geometry><material name="dark_grey"/></visual>
+      <geometry><cylinder radius="0.525" length="0.06"/></geometry><material name="wood"/></visual>
     <collision><origin xyz="0 0 0" rpy="1.5708 0 0"/>
-      <geometry><cylinder radius="0.525" length="0.08"/></geometry></collision>
+      <geometry><cylinder radius="0.525" length="0.06"/></geometry></collision>
+    <visual><origin xyz="0 -0.04 0" rpy="1.5708 0 0"/>
+      <geometry><cylinder radius="0.06" length="0.10"/></geometry><material name="iron"/></visual>
   </link>
   <!-- ── Gazebo contact/material for carriage ── -->
-  <gazebo reference="tongue_link"><material>Gazebo/Wood</material></gazebo>
-  <gazebo reference="cart_base_link"><material>Gazebo/Wood</material></gazebo>
+  <gazebo reference="shaft_link"><material>Gazebo/Wood</material></gazebo>
+  <gazebo reference="cart_hitch_link"><material>Gazebo/Grey</material></gazebo>
+  <gazebo reference="cart_body_link"><material>Gazebo/Wood</material></gazebo>
   <gazebo reference="front_axle_link"><material>Gazebo/Grey</material></gazebo>
   <gazebo reference="rear_axle_link"><material>Gazebo/Grey</material></gazebo>
   <gazebo reference="cart_fl_wheel_link">
-    <material>Gazebo/DarkGrey</material>
+    <material>Gazebo/Wood</material>
     <kp>1000000.0</kp><kd>100.0</kd>
     <mu1>1.0</mu1><mu2>1.0</mu2>
@@ -722,5 +816,5 @@
   </gazebo>
   <gazebo reference="cart_fr_wheel_link">
-    <material>Gazebo/DarkGrey</material>
+    <material>Gazebo/Wood</material>
     <kp>1000000.0</kp><kd>100.0</kd>
     <mu1>1.0</mu1><mu2>1.0</mu2>
@@ -728,5 +822,5 @@
   </gazebo>
   <gazebo reference="cart_rl_wheel_link">
-    <material>Gazebo/DarkGrey</material>
+    <material>Gazebo/Wood</material>
     <kp>1000000.0</kp><kd>100.0</kd>
     <mu1>1.0</mu1><mu2>1.0</mu2>
@@ -734,5 +828,5 @@
   </gazebo>
   <gazebo reference="cart_rr_wheel_link">
-    <material>Gazebo/DarkGrey</material>
+    <material>Gazebo/Wood</material>
     <kp>1000000.0</kp><kd>100.0</kd>
     <mu1>1.0</mu1><mu2>1.0</mu2>
