Commit message: Fix carriage bouncing, lower body height, toggle A/D steering
Hitch compliance (anti-bounce):
- shaft_yaw damping: 5.0 -> 0.2 (cow can sway without jostling carriage)
- shaft_pitch damping: 15.0 -> 1.5, range +/-0.35 rad (was +/-0.20)
- turntable_yaw damping: 25.0 -> 4.0 (smooth turning, less resistance)
- Carriage inertia (140kg) naturally dampens any remaining oscillation

Cart body height corrected:
- All visual z-positions shifted down 0.355m
- Body floor now at ~60cm off ground (was ~95cm)
- Matches user's measured carriage dimensions

Teleop steering rewrite:
- A/D changed from ramp/decay to toggle: press A = turn left,
  press A again = go straight. Same for D = right.
- Fixed turn rate of 0.6 rad/s (clean, predictable steering)
- Space bar now also resets steering direction

Co-authored-by: Copilot <223556219+Copilot@users.noreply.github.com>

File: ros2_ws/src/robotic_horse_description/urdf/robotic_horse.urdf.xacro (robot description, xacro)
@@ -591,10 +591,12 @@
        Total carriage mass ≈ 105 kg + 85 kg driver = 190 kg
   ═══════════════════════════════════════════════════════ -->
-  <!-- Shaft yaw joint (base_link → shaft) — continuous rotation (infinite turn angle) -->
+  <!-- Shaft yaw joint (base_link → shaft) — continuous rotation (infinite turn angle)
+       Very low damping: cow can sway laterally without jostling the carriage.
+       In reality, the shaft hangs via leather harness straps with lots of compliance. -->
   <joint name="shaft_yaw_joint" type="continuous">
     <parent link="base_link"/><child link="shaft_link"/>
     <origin xyz="0.0 0 -0.30" rpy="0 0 0"/>
     <axis xyz="0 0 1"/>
-    <dynamics damping="5.0" friction="0.5"/>
+    <dynamics damping="0.2" friction="0.05"/>
   </joint>
   <!-- Shaft — U-shaped wooden fork, 2.35m long -->
@@ -618,11 +620,12 @@
       <geometry><box size="0.05 0.70 0.05"/></geometry></collision>
   </link>
-  <!-- Shaft pitch joint — perch pivot at front of front axle assembly -->
+  <!-- Shaft pitch joint — perch pivot at front of front axle assembly
+       Moderate damping: allows free pitch motion over bumps without oscillation. -->
   <joint name="shaft_pitch_joint" type="revolute">
     <parent link="shaft_link"/><child link="front_assembly_link"/>
     <origin xyz="-2.35 0 0.015" rpy="0 0 0"/>
     <axis xyz="0 1 0"/>
-    <limit lower="-0.20" upper="0.20" effort="0" velocity="2.0"/>
-    <dynamics damping="15.0" friction="0.5"/>
+    <limit lower="-0.35" upper="0.35" effort="0" velocity="2.0"/>
+    <dynamics damping="1.5" friction="0.2"/>
   </joint>
   <!-- Front assembly (perch beam + front axle + turntable pin) ~8 kg -->
@@ -681,5 +684,7 @@
       <geometry><cylinder radius="0.06" length="0.08"/></geometry><material name="iron"/></visual>
   </link>
-  <!-- Turntable yaw joint — cart body rotates relative to front axle assembly -->
+  <!-- Turntable yaw joint — cart body rotates relative to front axle assembly
+       Moderate damping: enough to prevent oscillation but allows smooth turning.
+       The cart body's inertia (140 kg) provides natural stability. -->
   <joint name="turntable_yaw_joint" type="revolute">
     <parent link="front_assembly_link"/><child link="cart_body_link"/>
@@ -687,84 +692,85 @@
     <axis xyz="0 0 1"/>
     <limit lower="-0.785" upper="0.785" effort="0" velocity="2.0"/>
-    <dynamics damping="25.0" friction="1.0"/>
+    <dynamics damping="4.0" friction="0.3"/>
   </joint>
   <!-- Cart body — 250×110×110 cm wooden carriage body
        Origin at turntable center (directly above front wheel center)
-       All visual offsets are relative to this origin (shifted +0.50m x vs old hitch-based origin)
+       Visuals shifted down so body floor sits at ~60cm off ground
+       (turntable origin at z≈0.795m abs → floor at -0.195 rel = 0.60m abs)
        Driver (85 kg) seated on front bench -->
   <link name="cart_body_link">
     <!-- Combined inertia: carriage structure 55 kg + driver 85 kg = 140 kg
-         Approximate as box 2.50×1.10×1.10 at combined COM -->
-    <inertial><mass value="140.0"/><origin xyz="-0.90 0 0.42" rpy="0 0 0"/>
+         COM shifted down to match lowered body position -->
+    <inertial><mass value="140.0"/><origin xyz="-0.90 0 0.07" rpy="0 0 0"/>
       <inertia ixx="25.0" iyy="95.0" izz="85.0" ixy="0" ixz="0" iyz="0"/></inertial>
-    <!-- Main body floor/deck -->
-    <visual><origin xyz="-1.025 0 0.16" rpy="0 0 0"/>
+    <!-- Main body floor/deck — abs z ≈ 0.60m -->
+    <visual><origin xyz="-1.025 0 -0.195" rpy="0 0 0"/>
       <geometry><box size="2.50 1.10 0.06"/></geometry><material name="wood"/></visual>
-    <collision><origin xyz="-1.025 0 0.16" rpy="0 0 0"/>
+    <collision><origin xyz="-1.025 0 -0.195" rpy="0 0 0"/>
       <geometry><box size="2.50 1.10 0.06"/></geometry></collision>
-    <!-- Left side panel (curved in real life — approximated with box) -->
-    <visual><origin xyz="-1.025 0.52 0.55" rpy="0 0 0"/>
+    <!-- Left side panel -->
+    <visual><origin xyz="-1.025 0.52 0.195" rpy="0 0 0"/>
       <geometry><box size="2.20 0.06 0.72"/></geometry><material name="wood"/></visual>
-    <collision><origin xyz="-1.025 0.52 0.55" rpy="0 0 0"/>
+    <collision><origin xyz="-1.025 0.52 0.195" rpy="0 0 0"/>
       <geometry><box size="2.20 0.06 0.72"/></geometry></collision>
     <!-- Right side panel -->
-    <visual><origin xyz="-1.025 -0.52 0.55" rpy="0 0 0"/>
+    <visual><origin xyz="-1.025 -0.52 0.195" rpy="0 0 0"/>
       <geometry><box size="2.20 0.06 0.72"/></geometry><material name="wood"/></visual>
-    <collision><origin xyz="-1.025 -0.52 0.55" rpy="0 0 0"/>
+    <collision><origin xyz="-1.025 -0.52 0.195" rpy="0 0 0"/>
       <geometry><box size="2.20 0.06 0.72"/></geometry></collision>
-    <!-- Front panel (driver side, with kick board — black leather) -->
-    <visual><origin xyz="0.05 0 0.50" rpy="0 0 0"/>
+    <!-- Front panel (driver side, kick board) -->
+    <visual><origin xyz="0.05 0 0.145" rpy="0 0 0"/>
       <geometry><box size="0.06 1.00 0.62"/></geometry><material name="dark_grey"/></visual>
     <!-- Rear panel -->
-    <visual><origin xyz="-2.10 0 0.50" rpy="0 0 0"/>
+    <visual><origin xyz="-2.10 0 0.145" rpy="0 0 0"/>
       <geometry><box size="0.06 1.00 0.62"/></geometry><material name="dark_grey"/></visual>
     <!-- Center divider panel -->
-    <visual><origin xyz="-1.025 0 0.50" rpy="0 0 0"/>
+    <visual><origin xyz="-1.025 0 0.145" rpy="0 0 0"/>
       <geometry><box size="0.06 0.90 0.50"/></geometry><material name="dark_grey"/></visual>
-    <!-- Front bench seat (driver sits here, facing backward) -->
-    <visual><origin xyz="-0.30 0 0.46" rpy="0 0 0"/>
+    <!-- Front bench seat -->
+    <visual><origin xyz="-0.30 0 0.105" rpy="0 0 0"/>
       <geometry><box size="0.45 0.90 0.08"/></geometry><material name="red_velvet"/></visual>
     <!-- Front seat backrest -->
-    <visual><origin xyz="-0.08 0 0.68" rpy="0 0 0"/>
+    <visual><origin xyz="-0.08 0 0.325" rpy="0 0 0"/>
       <geometry><box size="0.06 0.90 0.36"/></geometry><material name="wood"/></visual>
-    <!-- Rear bench seat (passengers, facing forward) -->
-    <visual><origin xyz="-1.75 0 0.46" rpy="0 0 0"/>
+    <!-- Rear bench seat -->
+    <visual><origin xyz="-1.75 0 0.105" rpy="0 0 0"/>
       <geometry><box size="0.45 0.90 0.08"/></geometry><material name="red_velvet"/></visual>
     <!-- Rear seat backrest -->
-    <visual><origin xyz="-1.97 0 0.68" rpy="0 0 0"/>
+    <visual><origin xyz="-1.97 0 0.325" rpy="0 0 0"/>
       <geometry><box size="0.06 0.90 0.36"/></geometry><material name="wood"/></visual>
     <!-- Driver figure (85 kg, seated on front bench) -->
     <!-- Torso -->
-    <visual><origin xyz="-0.30 0 0.82" rpy="0 0 0"/>
+    <visual><origin xyz="-0.30 0 0.465" rpy="0 0 0"/>
       <geometry><box size="0.30 0.40 0.55"/></geometry><material name="dark_grey"/></visual>
     <!-- Head -->
-    <visual><origin xyz="-0.30 0 1.17" rpy="0 0 0"/>
+    <visual><origin xyz="-0.30 0 0.815" rpy="0 0 0"/>
       <geometry><sphere radius="0.12"/></geometry><material name="light_grey"/></visual>
     <!-- Left mudguard / fender (over rear wheels) -->
-    <visual><origin xyz="-1.85 0.58 0.10" rpy="0 0 0"/>
+    <visual><origin xyz="-1.85 0.58 -0.245" rpy="0 0 0"/>
       <geometry><box size="0.70 0.12 0.06"/></geometry><material name="wood"/></visual>
     <!-- Right mudguard -->
-    <visual><origin xyz="-1.85 -0.58 0.10" rpy="0 0 0"/>
+    <visual><origin xyz="-1.85 -0.58 -0.245" rpy="0 0 0"/>
       <geometry><box size="0.70 0.12 0.06"/></geometry><material name="wood"/></visual>
     <!-- Iron underframe / chassis rail (left) -->
-    <visual><origin xyz="-1.025 0.40 -0.05" rpy="0 0 0"/>
+    <visual><origin xyz="-1.025 0.40 -0.405" rpy="0 0 0"/>
       <geometry><box size="2.60 0.04 0.04"/></geometry><material name="iron"/></visual>
     <!-- Iron underframe / chassis rail (right) -->
-    <visual><origin xyz="-1.025 -0.40 -0.05" rpy="0 0 0"/>
+    <visual><origin xyz="-1.025 -0.40 -0.405" rpy="0 0 0"/>
       <geometry><box size="2.60 0.04 0.04"/></geometry><material name="iron"/></visual>
     <!-- Left carriage lamp bracket -->
-    <visual><origin xyz="0.15 0.50 0.95" rpy="0 0 0"/>
+    <visual><origin xyz="0.15 0.50 0.595" rpy="0 0 0"/>
       <geometry><cylinder radius="0.02" length="0.25"/></geometry><material name="iron"/></visual>
     <!-- Left lamp housing -->
-    <visual><origin xyz="0.15 0.54 1.10" rpy="0 0 0"/>
+    <visual><origin xyz="0.15 0.54 0.745" rpy="0 0 0"/>
       <geometry><box size="0.10 0.10 0.15"/></geometry><material name="iron"/></visual>
     <!-- Right carriage lamp bracket -->
-    <visual><origin xyz="0.15 -0.50 0.95" rpy="0 0 0"/>
+    <visual><origin xyz="0.15 -0.50 0.595" rpy="0 0 0"/>
       <geometry><cylinder radius="0.02" length="0.25"/></geometry><material name="iron"/></visual>
     <!-- Right lamp housing -->
-    <visual><origin xyz="0.15 -0.54 1.10" rpy="0 0 0"/>
+    <visual><origin xyz="0.15 -0.54 0.745" rpy="0 0 0"/>
       <geometry><box size="0.10 0.10 0.15"/></geometry><material name="iron"/></visual>
     <!-- Folding hood frame (rear, collapsed) -->
-    <visual><origin xyz="-2.05 0 1.00" rpy="0 0 0"/>
+    <visual><origin xyz="-2.05 0 0.645" rpy="0 0 0"/>
       <geometry><box size="0.08 0.95 0.15"/></geometry><material name="wood"/></visual>
   </link>

Commit message: Widen shaft, add roll joint (ball joint), raise spawn, bigger strides
Shaft clearance:
- Bars widened from +/-0.39m to +/-0.50m (1.0m apart)
- Clears 0.88m cow body with 6cm margin per side
- Cross piece at carriage end widened to 0.85m

Ball-joint hitch (3 DOF):
- Added shaft_yaw_link + shaft_roll_joint (revolute, x, +/-0.25 rad)
- Chain: base_link -> yaw(z) -> roll(x) -> shaft -> pitch(y) -> front_assembly
- Simulates leather harness flexibility around barrel
- Cow can sway, roll, and pitch without jostling carriage

Spawn height:
- Raised 1.08m -> 1.12m (4cm clearance for settling under gravity)
- Prevents feet/wheels clipping into ground at spawn

Stride increase (~30%):
- WALK stride: 0.50 -> 0.65m (half=0.325m)
- TROT stride: 0.65 -> 0.85m (half=0.425m, within 0.453m front reach at trot lift)
- MAX_STEP: 0.35 -> 0.45m
- Walk min_stride: 0.12 -> 0.15m, Trot min_stride: 0.18 -> 0.22m

Co-authored-by: Copilot <223556219+Copilot@users.noreply.github.com>

File: ros2_ws/src/robotic_horse_description/urdf/robotic_horse.urdf.xacro (robot description, xacro)
@@ -571,19 +571,25 @@
        Correct kinematic chain (real carriage):
          base_link → shaft_yaw (continuous, z)
-           → shaft_link (U-fork, 2.35m)
-             → shaft_pitch (revolute, y, at perch)
-               → front_assembly_link (perch + front axle + turntable)
-                 ├─ cart_fl_wheel_joint (continuous)
-                 ├─ cart_fr_wheel_joint (continuous)
-                 └─ turntable_yaw_joint (revolute, z, ±45°)
-                    → cart_body_link (body, driver, etc.)
-                      → rear_axle_joint (fixed)
-                        → rear_axle_link
-                          ├─ cart_rl_wheel_joint (continuous)
-                          └─ cart_rr_wheel_joint (continuous)
+           → shaft_yaw_link (dummy)
+             → shaft_roll (revolute, x, ±0.20 rad)
+               → shaft_link (U-fork, 2.35m, bars at ±0.50m to clear body)
+                 → shaft_pitch (revolute, y, at perch)
+                   → front_assembly_link (perch + front axle + turntable)
+                     ├─ cart_fl_wheel_joint (continuous)
+                     ├─ cart_fr_wheel_joint (continuous)
+                     └─ turntable_yaw_joint (revolute, z, ±45°)
+                        → cart_body_link (body, driver, etc.)
+                          → rear_axle_joint (fixed)
+                            → rear_axle_link
+                              ├─ cart_rl_wheel_joint (continuous)
+                              └─ cart_rr_wheel_joint (continuous)
+       Ball-joint at cow: yaw (z) + roll (x) = 2 DOF
+       Pitch at carriage end: 1 DOF
+       Total: 3 rotational DOF ≈ ball joint
+       Shaft bars at ±0.50m (1.0m apart) clear 0.88m body width
        Real measurements from owner's carriage:
          Front wheels ⌀ 85 cm,  Rear wheels ⌀ 105 cm
          Wheelbase 205 cm,  Track 145 cm
-         Shaft 235 cm long, U-shaped, 85→70 cm wide
+         Shaft 235 cm long, U-shaped
          Perch: shaft connects to front axle assembly 50cm fwd of wheel center
          Body: 250 × 110 × 110 cm, ~60 cm off ground
@@ -591,32 +597,46 @@
        Total carriage mass ≈ 105 kg + 85 kg driver = 190 kg
   ═══════════════════════════════════════════════════════ -->
-  <!-- Shaft yaw joint (base_link → shaft) — continuous rotation (infinite turn angle)
-       Very low damping: cow can sway laterally without jostling the carriage.
-       In reality, the shaft hangs via leather harness straps with lots of compliance. -->
+  <!-- Shaft yaw joint — free yaw rotation (harness strap compliance)
+       Very low damping: cow can sway without jostling carriage -->
   <joint name="shaft_yaw_joint" type="continuous">
-    <parent link="base_link"/><child link="shaft_link"/>
+    <parent link="base_link"/><child link="shaft_yaw_link"/>
     <origin xyz="0.0 0 -0.30" rpy="0 0 0"/>
     <axis xyz="0 0 1"/>
     <dynamics damping="0.2" friction="0.05"/>
   </joint>
-  <!-- Shaft — U-shaped wooden fork, 2.35m long -->
+  <!-- Dummy link between yaw and roll joints -->
+  <link name="shaft_yaw_link">
+    <inertial><mass value="0.5"/><origin xyz="0 0 0" rpy="0 0 0"/>
+      <inertia ixx="0.001" iyy="0.001" izz="0.001" ixy="0" ixz="0" iyz="0"/></inertial>
+  </link>
+  <!-- Shaft roll joint — allows body roll without transferring to carriage
+       Simulates leather harness flexibility around the barrel -->
+  <joint name="shaft_roll_joint" type="revolute">
+    <parent link="shaft_yaw_link"/><child link="shaft_link"/>
+    <origin xyz="0 0 0" rpy="0 0 0"/>
+    <axis xyz="1 0 0"/>
+    <limit lower="-0.25" upper="0.25" effort="0" velocity="2.0"/>
+    <dynamics damping="0.3" friction="0.05"/>
+  </joint>
+  <!-- Shaft — U-shaped wooden fork, 2.35m long
+       Bars at ±0.50m (1.0m apart) to clear 0.88m body width -->
   <link name="shaft_link">
     <inertial><mass value="15.0"/><origin xyz="-1.175 0 0" rpy="0 0 0"/>
-      <inertia ixx="0.10" iyy="6.93" izz="6.95" ixy="0" ixz="0" iyz="0"/></inertial>
+      <inertia ixx="0.15" iyy="6.93" izz="7.00" ixy="0" ixz="0" iyz="0"/></inertial>
     <!-- Left shaft bar -->
-    <visual><origin xyz="-1.175 0.39 0" rpy="0 0 0"/>
+    <visual><origin xyz="-1.175 0.50 0" rpy="0 0 0"/>
       <geometry><box size="2.35 0.05 0.05"/></geometry><material name="wood"/></visual>
-    <collision><origin xyz="-1.175 0.39 0" rpy="0 0 0"/>
+    <collision><origin xyz="-1.175 0.50 0" rpy="0 0 0"/>
       <geometry><box size="2.35 0.05 0.05"/></geometry></collision>
     <!-- Right shaft bar -->
-    <visual><origin xyz="-1.175 -0.39 0" rpy="0 0 0"/>
+    <visual><origin xyz="-1.175 -0.50 0" rpy="0 0 0"/>
       <geometry><box size="2.35 0.05 0.05"/></geometry><material name="wood"/></visual>
-    <collision><origin xyz="-1.175 -0.39 0" rpy="0 0 0"/>
+    <collision><origin xyz="-1.175 -0.50 0" rpy="0 0 0"/>
       <geometry><box size="2.35 0.05 0.05"/></geometry></collision>
-    <!-- Cross piece at carriage end -->
+    <!-- Cross piece at carriage end (tapers to ~0.85m) -->
     <visual><origin xyz="-2.30 0 0" rpy="0 0 0"/>
-      <geometry><box size="0.05 0.70 0.05"/></geometry><material name="wood"/></visual>
+      <geometry><box size="0.05 0.85 0.05"/></geometry><material name="wood"/></visual>
     <collision><origin xyz="-2.30 0 0" rpy="0 0 0"/>
-      <geometry><box size="0.05 0.70 0.05"/></geometry></collision>
+      <geometry><box size="0.05 0.85 0.05"/></geometry></collision>
   </link>
   <!-- Shaft pitch joint — perch pivot at front of front axle assembly
@@ -823,4 +843,5 @@
   </link>
   <!-- ── Gazebo contact/material for carriage ── -->
+  <gazebo reference="shaft_yaw_link"/>
   <gazebo reference="shaft_link"><material>Gazebo/Wood</material></gazebo>
   <gazebo reference="front_assembly_link"><material>Gazebo/Grey</material></gazebo>
