Commit message: Add spine articulation, overhaul gait to match bovine biomechanics
Spine articulation:
- Split body into rear (base_link, 48kg) and front (front_body_link, 59kg)
- spine_yaw_joint (revolute, z, ±0.30rad) between them for turning
- FL/FR legs and head reparented to front_body_link
- Spine controlled proportionally to angular velocity (SPINE_TURN_GAIN=0.35)
- PID gains: p=2000, d=120 for smooth, strong spine control

Bovine gait overhaul (from biomechanics research):
- Walk: stride 0.65m→1.10m, swing_frac 0.30→0.40 (60% stance like real cattle)
- Walk: speed 0.80→1.00 m/s, step_height 0.10/0.08→0.12/0.10
- Trot: stride 0.85m→1.50m, swing_frac stays 0.50
- Trot: speed 1.50→2.00 m/s, period 0.70→0.75s, step_height 0.14/0.12→0.16/0.14
- MAX_STEP 0.45→0.60m, MAX_SHOULDER 0.20→0.25rad
- Speed ramp tuned for smoother acceleration

17 joints total (was 16): spine + 4 legs × 4 joints each.

Co-authored-by: Copilot <223556219+Copilot@users.noreply.github.com>

File: ros2_ws/src/robotic_horse_description/urdf/robotic_horse.urdf.xacro (robot description, xacro)
@@ -12,5 +12,6 @@
       |        |
       RL –––– RR
-  Controlled joints (16 total, QDD actuated):
+  Controlled joints (17 total, QDD actuated):
+      spine_yaw_joint              — spine lateral bend       (position ctrl)
       {fl,fr,rl,rr}_hip_joint     — lateral hip yaw          (position ctrl)
       {fl,fr,rl,rr}_thigh_joint   — hip flexion/extension    (position ctrl)
@@ -69,17 +70,63 @@
        Inertia (107 kg, 1.80x0.88x0.85 m box): Ixx=13.35, Iyy=35.33, Izz=35.80 kg·m²
        Scaled 1.36× from real Highland cow (110cm withers → 150cm) -->
+  <!-- base_link = REAR body half (haunches/lumbar).
+       Rear legs (RL/RR) and carriage hitch attach here.
+       IMU stays on base_link for balance sensing. -->
   <link name="base_link">
     <inertial>
-      <mass value="107.0"/>
-      <origin xyz="0 0 0" rpy="0 0 0"/>
-      <inertia ixx="13.35" iyy="35.33" izz="35.80" ixy="0" ixz="0" iyz="0"/>
+      <mass value="48.0"/>
+      <origin xyz="0.45 0 0" rpy="0 0 0"/>
+      <inertia ixx="6.0" iyy="6.1" izz="6.3" ixy="0" ixz="0" iyz="0"/>
     </inertial>
-    <!-- Main barrel (ribcage/abdomen) — 1.36× scaled: 75cm tall, 88cm wide -->
+    <!-- Rear barrel half -->
     <visual>
-      <origin xyz="0 0 0" rpy="0 0 0"/>
-      <geometry><box size="1.80 0.88 0.75"/></geometry>
+      <origin xyz="0.45 0 0" rpy="0 0 0"/>
+      <geometry><box size="0.90 0.88 0.75"/></geometry>
       <material name="body_panel"/>
     </visual>
-    <!-- Withers rise (front — now at -X since robot faces -X) -->
+    <!-- Rump (back — at +X) -->
+    <visual>
+      <origin xyz="0.55 0 0.425" rpy="0 0 0"/>
+      <geometry><box size="0.40 0.76 0.10"/></geometry>
+      <material name="body_panel"/>
+    </visual>
+    <collision>
+      <origin xyz="0.45 0 0" rpy="0 0 0"/>
+      <geometry><box size="0.90 0.88 0.85"/></geometry>
+    </collision>
+  </link>
+  <gazebo reference="base_link">
+    <material>Gazebo/DarkGrey</material>
+  </gazebo>
+  <!-- ═══════════════════════════════════════════════════════
+       SPINE YAW JOINT — articulated spine for turning
+       Connects rear body (base_link) to front body (front_body_link).
+       Z-axis rotation allows lateral bending like a real quadruped.
+       This is the PRIMARY turning mechanism — combined with
+       differential stride length for smooth, natural turns.
+  ═══════════════════════════════════════════════════════ -->
+  <joint name="spine_yaw_joint" type="revolute">
+    <parent link="base_link"/><child link="front_body_link"/>
+    <origin xyz="0 0 0" rpy="0 0 0"/>
+    <axis xyz="0 0 1"/>
+    <limit lower="-0.30" upper="0.30" effort="500" velocity="1.5"/>
+    <dynamics damping="12.0" friction="1.0"/>
+  </joint>
+  <!-- front_body_link = FRONT body half (thorax/shoulders).
+       Front legs (FL/FR) and head/neck attach here.
+       55% of body mass (bovine weight distribution). -->
+  <link name="front_body_link">
+    <inertial>
+      <mass value="59.0"/>
+      <origin xyz="-0.45 0 0" rpy="0 0 0"/>
+      <inertia ixx="7.4" iyy="7.5" izz="7.8" ixy="0" ixz="0" iyz="0"/>
+    </inertial>
+    <!-- Front barrel half -->
+    <visual>
+      <origin xyz="-0.45 0 0" rpy="0 0 0"/>
+      <geometry><box size="0.90 0.88 0.75"/></geometry>
+      <material name="body_panel"/>
+    </visual>
+    <!-- Withers rise (front shoulder hump) -->
     <visual>
       <origin xyz="-0.50 0 0.475" rpy="0 0 0"/>
@@ -93,16 +140,10 @@
       <material name="body_panel"/>
     </visual>
-    <!-- Rump (back — now at +X) -->
-    <visual>
-      <origin xyz="0.55 0 0.425" rpy="0 0 0"/>
-      <geometry><box size="0.40 0.76 0.10"/></geometry>
-      <material name="body_panel"/>
-    </visual>
     <collision>
-      <origin xyz="0 0 0" rpy="0 0 0"/>
-      <geometry><box size="1.80 0.88 0.85"/></geometry>
+      <origin xyz="-0.45 0 0" rpy="0 0 0"/>
+      <geometry><box size="0.90 0.88 0.85"/></geometry>
     </collision>
   </link>
-  <gazebo reference="base_link">
+  <gazebo reference="front_body_link">
     <material>Gazebo/DarkGrey</material>
   </gazebo>
@@ -110,5 +151,6 @@
   <!-- Neck: yaw + pitch joints for head motion
        Head: jaw (open/close), eyes (left/right pan)
-       Small servos — total head assembly ~6.5 kg -->
+       Small servos — total head assembly ~6.5 kg
+       Attached to front_body_link (thorax) -->
   <!-- Neck yaw — swivel left/right (head faces -X direction of travel) -->
   <link name="neck_yaw_link">
@@ -117,5 +159,5 @@
   </link>
   <joint name="neck_yaw_joint" type="revolute">
-    <parent link="base_link"/><child link="neck_yaw_link"/>
+    <parent link="front_body_link"/><child link="neck_yaw_link"/>
     <origin xyz="-0.85 0 0.42" rpy="0 0 3.14159"/>
     <axis xyz="0 0 1"/>
@@ -260,5 +302,5 @@
   </link>
   <joint name="fl_hip_joint" type="revolute">
-    <parent link="base_link"/><child link="fl_hip_link"/>
+    <parent link="front_body_link"/><child link="fl_hip_link"/>
     <origin xyz="0.65 0.44 -0.15" rpy="0 0 0"/>
     <axis xyz="0 0 1"/>
@@ -341,5 +383,5 @@
   </link>
   <joint name="fr_hip_joint" type="revolute">
-    <parent link="base_link"/><child link="fr_hip_link"/>
+    <parent link="front_body_link"/><child link="fr_hip_link"/>
     <origin xyz="0.65 -0.44 -0.15" rpy="0 0 0"/>
     <axis xyz="0 0 1"/>
@@ -867,5 +909,5 @@
   <!-- ═══════════════════════════════════════════════════════
        ROS2 CONTROL — hardware interface
-       16 commanded joints: 4x hip(Z) + 4x thigh(Y) + 4x knee(Y) + 4x cannon(Y)
+       17 commanded joints: spine(Z) + 4x hip(Z) + 4x thigh(Y) + 4x knee(Y) + 4x cannon(Y)
        Carriage wheels are passive — not included in ros2_control.
   ═══════════════════════════════════════════════════════ -->
@@ -874,4 +916,15 @@
       <plugin>gz_ros2_control/GazeboSimSystem</plugin>
     </hardware>
+    <!-- Spine yaw — articulated spine for turning -->
+    <joint name="spine_yaw_joint">
+      <command_interface name="position">
+        <param name="min">-0.30</param><param name="max">0.30</param>
+      </command_interface>
+      <state_interface name="position">
+        <param name="initial_value">0.0</param>
+      </state_interface>
+      <state_interface name="velocity"/>
+      <state_interface name="effort"/>
+    </joint>
     <!-- Front-left -->
     <joint name="fl_hip_joint">

Commit message: Fix front-leg buckling: stiffer joints, stance push, shorter strides
Problem: Front legs buckled under forward momentum during walking.
The 107kg body + dynamic loading exceeded the PID tracking ability,
causing knees to collapse and the robot to tip forward.

Multi-layer fix (inspired by MIT Cheetah / ANYmal approaches):

1. PID gains (ros2_control.yaml):
   - Controller update rate: 100 → 200 Hz (better tracking)
   - Front thigh P: 3000 → 6000, knee P: 4500 → 8000
   - Rear thigh P: 3000 → 5000, knee P: 4500 → 7000
   - Added I-gains on all leg joints for gravity compensation
   - Increased D-gains for damping during dynamic motion

2. URDF joint physics:
   - Front knee effort: 800 → 1200 Nm (matches dynamic load)
   - Front thigh effort: 500 → 800 Nm
   - All joint damping increased 1.5-2x (resists sudden collapse)
   - Rear joints also moderately increased

3. Gait parameters (blendspace_node.py):
   - Walk stride: 1.10 → 0.90m (less overreach)
   - Trot stride: 1.50 → 1.20m
   - Walk swing: 40% → 35% (longer stance = more stable)
   - Trot swing: 50% → 45%
   - Walk speed: 1.00 → 0.80 m/s
   - Trot speed: 2.00 → 1.60 m/s
   - Front step height: 0.12 → 0.14m (better clearance)

4. Virtual spring stance model (new):
   - Sinusoidal ground penetration profile during stance
   - Base 4cm + peak 5cm push at mid-stance
   - Front legs push 2cm deeper (55% weight distribution)
   - Replaces flat 2cm penetration that was too shallow

5. Stronger balance correction:
   - BALANCE_FOOT_GAIN: 0.40 → 0.50
   - MIN_STEP_HEIGHT: 0.04 → 0.05m

Co-authored-by: Copilot <223556219+Copilot@users.noreply.github.com>

File: ros2_ws/src/robotic_horse_description/urdf/robotic_horse.urdf.xacro (robot description, xacro)
@@ -305,6 +305,6 @@
     <origin xyz="0.65 0.44 -0.15" rpy="0 0 0"/>
     <axis xyz="0 0 1"/>
-    <limit lower="-0.35" upper="0.35" effort="200" velocity="2.0"/>
-    <dynamics damping="2.5" friction="0.3"/>
+    <limit lower="-0.35" upper="0.35" effort="300" velocity="2.0"/>
+    <dynamics damping="4.0" friction="0.5"/>
   </joint>
   <gazebo reference="fl_hip_link"><material>Gazebo/Grey</material></gazebo>
@@ -320,6 +320,6 @@
     <parent link="fl_hip_link"/><child link="fl_thigh_link"/>
     <origin xyz="0 0 -0.10" rpy="0 0 0"/><axis xyz="0 1 0"/>
-    <limit lower="-0.30" upper="1.20" effort="500" velocity="3.0"/>
-    <dynamics damping="2.5" friction="0.3"/>
+    <limit lower="-0.30" upper="1.20" effort="800" velocity="3.0"/>
+    <dynamics damping="5.0" friction="0.5"/>
   </joint>
   <gazebo reference="fl_thigh_link"><material>Gazebo/Orange</material></gazebo>
@@ -335,6 +335,6 @@
     <parent link="fl_thigh_link"/><child link="fl_shank_link"/>
     <origin xyz="0 0 -0.38" rpy="0 0 0"/><axis xyz="0 1 0"/>
-    <limit lower="-1.80" upper="-0.10" effort="800" velocity="5.0"/>
-    <dynamics damping="3.5" friction="0.3"/>
+    <limit lower="-1.80" upper="-0.10" effort="1200" velocity="5.0"/>
+    <dynamics damping="6.0" friction="0.5"/>
   </joint>
   <gazebo reference="fl_shank_link"><material>Gazebo/DarkGrey</material></gazebo>
@@ -351,6 +351,6 @@
     <parent link="fl_shank_link"/><child link="fl_cannon_link"/>
     <origin xyz="0 0 -0.34" rpy="0 0 0"/><axis xyz="0 1 0"/>
-    <limit lower="-2.0" upper="2.0" effort="100" velocity="6.0"/>
-    <dynamics damping="1.0" friction="0.1"/>
+    <limit lower="-2.0" upper="2.0" effort="200" velocity="6.0"/>
+    <dynamics damping="2.0" friction="0.2"/>
   </joint>
   <gazebo reference="fl_cannon_link"><material>Gazebo/DarkGrey</material></gazebo>
@@ -386,6 +386,6 @@
     <origin xyz="0.65 -0.44 -0.15" rpy="0 0 0"/>
     <axis xyz="0 0 1"/>
-    <limit lower="-0.35" upper="0.35" effort="200" velocity="2.0"/>
-    <dynamics damping="2.5" friction="0.3"/>
+    <limit lower="-0.35" upper="0.35" effort="300" velocity="2.0"/>
+    <dynamics damping="4.0" friction="0.5"/>
   </joint>
   <gazebo reference="fr_hip_link"><material>Gazebo/Grey</material></gazebo>
@@ -401,6 +401,6 @@
     <parent link="fr_hip_link"/><child link="fr_thigh_link"/>
     <origin xyz="0 0 -0.10" rpy="0 0 0"/><axis xyz="0 1 0"/>
-    <limit lower="-0.30" upper="1.20" effort="500" velocity="3.0"/>
-    <dynamics damping="2.5" friction="0.3"/>
+    <limit lower="-0.30" upper="1.20" effort="800" velocity="3.0"/>
+    <dynamics damping="5.0" friction="0.5"/>
   </joint>
   <gazebo reference="fr_thigh_link"><material>Gazebo/Orange</material></gazebo>
@@ -416,6 +416,6 @@
     <parent link="fr_thigh_link"/><child link="fr_shank_link"/>
     <origin xyz="0 0 -0.38" rpy="0 0 0"/><axis xyz="0 1 0"/>
-    <limit lower="-1.80" upper="-0.10" effort="800" velocity="5.0"/>
-    <dynamics damping="3.5" friction="0.3"/>
+    <limit lower="-1.80" upper="-0.10" effort="1200" velocity="5.0"/>
+    <dynamics damping="6.0" friction="0.5"/>
   </joint>
   <gazebo reference="fr_shank_link"><material>Gazebo/DarkGrey</material></gazebo>
@@ -432,6 +432,6 @@
     <parent link="fr_shank_link"/><child link="fr_cannon_link"/>
     <origin xyz="0 0 -0.34" rpy="0 0 0"/><axis xyz="0 1 0"/>
-    <limit lower="-2.0" upper="2.0" effort="100" velocity="6.0"/>
-    <dynamics damping="1.0" friction="0.1"/>
+    <limit lower="-2.0" upper="2.0" effort="200" velocity="6.0"/>
+    <dynamics damping="2.0" friction="0.2"/>
   </joint>
   <gazebo reference="fr_cannon_link"><material>Gazebo/DarkGrey</material></gazebo>
@@ -467,6 +467,6 @@
     <origin xyz="-0.65 0.40 0.12" rpy="0 0 0"/>
     <axis xyz="0 0 1"/>
-    <limit lower="-0.35" upper="0.35" effort="200" velocity="2.0"/>
-    <dynamics damping="2.5" friction="0.3"/>
+    <limit lower="-0.35" upper="0.35" effort="250" velocity="2.0"/>
+    <dynamics damping="3.5" friction="0.4"/>
   </joint>
   <gazebo reference="rl_hip_link"><material>Gazebo/Grey</material></gazebo>
@@ -482,6 +482,6 @@
     <parent link="rl_hip_link"/><child link="rl_thigh_link"/>
     <origin xyz="0 0 -0.10" rpy="0 0 0"/><axis xyz="0 1 0"/>
-    <limit lower="-1.20" upper="0.30" effort="500" velocity="3.0"/>
-    <dynamics damping="2.5" friction="0.3"/>
+    <limit lower="-1.20" upper="0.30" effort="700" velocity="3.0"/>
+    <dynamics damping="4.5" friction="0.4"/>
   </joint>
   <gazebo reference="rl_thigh_link"><material>Gazebo/Orange</material></gazebo>
@@ -497,6 +497,6 @@
     <parent link="rl_thigh_link"/><child link="rl_shank_link"/>
     <origin xyz="0 0 -0.50" rpy="0 0 0"/><axis xyz="0 1 0"/>
-    <limit lower="0.10" upper="1.80" effort="800" velocity="5.0"/>
-    <dynamics damping="3.5" friction="0.3"/>
+    <limit lower="0.10" upper="1.80" effort="1000" velocity="5.0"/>
+    <dynamics damping="5.0" friction="0.4"/>
   </joint>
   <gazebo reference="rl_shank_link"><material>Gazebo/DarkGrey</material></gazebo>
@@ -513,6 +513,6 @@
     <parent link="rl_shank_link"/><child link="rl_cannon_link"/>
     <origin xyz="0 0 -0.45" rpy="0 0 0"/><axis xyz="0 1 0"/>
-    <limit lower="-2.0" upper="2.0" effort="100" velocity="6.0"/>
-    <dynamics damping="1.0" friction="0.1"/>
+    <limit lower="-2.0" upper="2.0" effort="150" velocity="6.0"/>
+    <dynamics damping="1.5" friction="0.2"/>
   </joint>
   <gazebo reference="rl_cannon_link"><material>Gazebo/DarkGrey</material></gazebo>
@@ -548,6 +548,6 @@
     <origin xyz="-0.65 -0.40 0.12" rpy="0 0 0"/>
     <axis xyz="0 0 1"/>
-    <limit lower="-0.35" upper="0.35" effort="200" velocity="2.0"/>
-    <dynamics damping="2.5" friction="0.3"/>
+    <limit lower="-0.35" upper="0.35" effort="250" velocity="2.0"/>
+    <dynamics damping="3.5" friction="0.4"/>
   </joint>
   <gazebo reference="rr_hip_link"><material>Gazebo/Grey</material></gazebo>
@@ -563,6 +563,6 @@
     <parent link="rr_hip_link"/><child link="rr_thigh_link"/>
     <origin xyz="0 0 -0.10" rpy="0 0 0"/><axis xyz="0 1 0"/>
-    <limit lower="-1.20" upper="0.30" effort="500" velocity="3.0"/>
-    <dynamics damping="2.5" friction="0.3"/>
+    <limit lower="-1.20" upper="0.30" effort="700" velocity="3.0"/>
+    <dynamics damping="4.5" friction="0.4"/>
   </joint>
   <gazebo reference="rr_thigh_link"><material>Gazebo/Orange</material></gazebo>
@@ -578,6 +578,6 @@
     <parent link="rr_thigh_link"/><child link="rr_shank_link"/>
     <origin xyz="0 0 -0.50" rpy="0 0 0"/><axis xyz="0 1 0"/>
-    <limit lower="0.10" upper="1.80" effort="800" velocity="5.0"/>
-    <dynamics damping="3.5" friction="0.3"/>
+    <limit lower="0.10" upper="1.80" effort="1000" velocity="5.0"/>
+    <dynamics damping="5.0" friction="0.4"/>
   </joint>
   <gazebo reference="rr_shank_link"><material>Gazebo/DarkGrey</material></gazebo>
@@ -594,6 +594,6 @@
     <parent link="rr_shank_link"/><child link="rr_cannon_link"/>
     <origin xyz="0 0 -0.45" rpy="0 0 0"/><axis xyz="0 1 0"/>
-    <limit lower="-2.0" upper="2.0" effort="100" velocity="6.0"/>
-    <dynamics damping="1.0" friction="0.1"/>
+    <limit lower="-2.0" upper="2.0" effort="150" velocity="6.0"/>
+    <dynamics damping="1.5" friction="0.2"/>
   </joint>
   <gazebo reference="rr_cannon_link"><material>Gazebo/DarkGrey</material></gazebo>
